File: hard/led_matrix.kicad_pcb (KiCad board)
At the start: 2 copper layers, 160 x 110 mm, 1355 parts, among them J1 MicroXNJ, J2 PJ-3062-CO, M1 IRLML6402TRPBF, M10 2N7002,215, M11 IRLML6402TRPBF, M12 2N7002,215, M13 IRLML6402TRPBF, M14 2N7002,215, M15 IRLML6402TRPBF, M16 2N7002,215, M17 IRLML6402TRPBF, M18 2N7002,215, M19 IRLML6402TRPBF, M2 2N7002,215, M20 2N7002,215, M21 IRLML6402TRPBF, M22 2N7002,215, M23 IRLML6402TRPBF, M24 2N7002,215, M25 IRLML6402TRPBF, M26 2N7002,215, M27 IRLML6402TRPBF, M28 2N7002,215, M29 IRLML6402TRPBF, M3 IRLML6402TRPBF, M30 2N7002,215, M31 IRLML6402TRPBF, M32 2N7002,215, M33 IRLML6402TRPBF, M34 2N7002,215, M35 IRLML6402TRPBF, M36 2N7002,215, M37 IRLML6402TRPBF, M38 2N7002,215, M39 IRLML6402TRPBF, M4 2N7002,215, M40 2N7002,215, M41 IRLML6402TRPBF, M42 2N7002,215, M43 IRLML6402TRPBF, M44 2N7002,215, M45 IRLML6402TRPBF, M46 2N7002,215, M47 IRLML6402TRPBF, M48 2N7002,215, M49 IRLML6402TRPBF, M5 IRLML6402TRPBF, M50 2N7002,215, M51 IRLML6402TRPBF, M52 2N7002,215, M53 IRLML6402TRPBF, M54 2N7002,215, M55 IRLML6402TRPBF, M56 2N7002,215, M57 IRLML6402TRPBF, M58 2N7002,215, M59 IRLML6402TRPBF, M6 2N7002,215, M60 2N7002,215, M61 IRLML6402TRPBF, M62 2N7002,215, M63 IRLML6402TRPBF, M64 2N7002,215, M65 IRLML0030TRPBF, M66 IRLML0030TRPBF, M67 IRLML0030TRPBF, M68 IRLML0030TRPBF, M69 IRLML0030TRPBF, M7 IRLML6402TRPBF, M70 IRLML0030TRPBF, M71 IRLML0030TRPBF, M72 IRLML0030TRPBF, M73 IRLML0030TRPBF, M74 IRLML0030TRPBF, M75 IRLML0030TRPBF, M76 IRLML0030TRPBF, M77 IRLML0030TRPBF, M78 IRLML0030TRPBF, M79 IRLML0030TRPBF, M8 2N7002,215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

Commit message: layouting update
Parts:
- removed G***: LOGO, led_matrix:logo2
- removed G***: LOGO, led_matrix:logo
- R1, R10, R101, R102, R104, R105, R107, R108, R110, R111, R113, R114, R116, R117, R119, R12, R120, R122, R123, R125, R126, R128, R129, R13, R131, R132, R134, R135, R137, R138, R140, R141, R143, R144, R146, R147, R149, R15, R150, R152, R153, R155, R156, R158, R159, R16, R161, R162, R164, R165, R167, R168, R170, R171, R173, R174, R176, R177, R179, R18, R180, R182, R183, R185, R186, R188, R189, R19, R191, R192, R21, R22, R24, R25, R27, R28, R3, R30, R31, R33, R34, R36, R37, R39, R4, R40, R42, R43, R45, R46, R48, R49, R51, R52, R54, R55, R57, R58, R6, R60, R61, R63, R64, R66, R67, R69, R7, R70, R72, R73, R75, R76, R78, R79, R81, R82, R84, R85, R87, R88, R9, R90, R91, R93, R94, R96, R98, R99: footprint Resistor_SMD:R_0603_1608Metric -> Resistor_SMD:R_0402_1005Metric
- R100, R103, R106, R109, R11, R112, R115, R118, R121, R124, R127, R130, R133, R136, R139, R14, R142, R145, R148, R151, R154, R157, R160, R163, R166, R169, R17, R172, R175, R178, R181, R184, R187, R190, R2, R20, R23, R26, R29, R32, R35, R38, R41, R44, R47, R5, R50, R53, R56, R59, R62, R65, R68, R71, R74, R77, R8, R80, R83, R86, R89, R92, R95, R97: footprint Resistor_SMD:R_0603_1608Metric -> Resistor_SMD:R_1210_3225Metric
- moved R104 268.2 mm to (40.2, 115.0), turned to 270 degrees
- moved R105 266.2 mm to (41.8, 115.0), turned to 270 degrees
- moved M67 262.3 mm to (41.0, 111.5), turned to 90 degrees
- moved R103 260.4 mm to (41.0, 106.5), turned to 270 degrees
- moved R101 253.6 mm to (37.2, 115.0), turned to 270 degrees
- moved R102 251.6 mm to (38.8, 115.0), turned to 270 degrees
- moved M66 247.8 mm to (38.0, 111.5), turned to 90 degrees
- moved R100 246.2 mm to (38.0, 106.5), turned to 270 degrees
- moved R2 237.7 mm to (21.0, -8.00)
- moved R1 236.5 mm to (26.2, -8.00), turned to 270 degrees
- moved M2 232.7 mm to (25.5, -5.00), turned to 90 degrees
- moved R3 230.1 mm to (24.8, -8.00), turned to 90 degrees
- moved M65 227.1 mm to (22.1, 115.9)
- moved R97 227.1 mm to (26.3, 114.9)
- moved R98 227.1 mm to (21.9, 119.4)
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
Commit message: driver nmos update
Parts:
- moved R15 211.3 mm to (21.5, 18.5), turned to 90 degrees
- moved M10 205.3 mm to (19.0, 19.8), turned to 270 degrees
- moved M9 204.7 mm to (24.0, 19.8), turned to 180 degrees
- moved R13 203.3 mm to (21.5, 21.0), turned to 270 degrees
- moved R14 200.8 mm to (28.5, 19.8)
- moved R101 119.0 mm to (39.2, -4.00), turned to 0 degrees
- moved R102 119.0 mm to (36.8, -4.00), turned to 180 degrees
- moved R5 118.3 mm to (139.2, 12.8), turned to 180 degrees
- moved M66 112.5 mm to (38.0, -1.00), turned to 270 degrees
- moved R6 110.8 mm to (135.5, 12.8), turned to 270 degrees
- moved M4 109.3 mm to (134.8, 9.75), turned to 270 degrees
- moved R4 107.8 mm to (134.0, 12.8), turned to 90 degrees
- moved R100 103.0 mm to (38.0, 3.50), turned to 90 degrees
- moved M3 101.3 mm to (130.8, 11.8), turned to 270 degrees
- moved M6 37.8 mm to (17.5, 13.8), turned to 270 degrees
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Connections:
- M1 pad 2: /led matrix/common anode/ANODES -> Net-(M1-Pad2)
- M1 pad 3: Net-(M1-Pad3) -> +5V
- M11 pad 2: /led matrix/sheetA341C380/ANODES -> Net-(M11-Pad2)
- M11 pad 3: Net-(M11-Pad3) -> +5V
- M13 pad 2: /led matrix/sheetA3FD3BF7/ANODES -> Net-(M13-Pad2)
- M13 pad 3: Net-(M13-Pad3) -> +5V
- M15 pad 2: /led matrix/sheetA3FD3BF8/ANODES -> Net-(M15-Pad2)
- M15 pad 3: Net-(M15-Pad3) -> +5V
- M17 pad 2: /led matrix/sheetA4B98B86/ANODES -> Net-(M17-Pad2)
- M17 pad 3: Net-(M17-Pad3) -> +5V
- M19 pad 2: /led matrix/sheetA4B98B87/ANODES -> Net-(M19-Pad2)
- M19 pad 3: Net-(M19-Pad3) -> +5V
- M21 pad 2: /led matrix/sheetA4B98B88/ANODES -> Net-(M21-Pad2)
- M21 pad 3: Net-(M21-Pad3) -> +5V
- M23 pad 2: /led matrix/sheetA4B98B89/ANODES -> Net-(M23-Pad2)
- M23 pad 3: Net-(M23-Pad3) -> +5V
- M25 pad 2: /led matrix/sheetA4B98B8A/ANODES -> Net-(M25-Pad2)
- M25 pad 3: Net-(M25-Pad3) -> +5V
- M27 pad 2: /led matrix/sheetA4B98B8B/ANODES -> Net-(M27-Pad2)
- M27 pad 3: Net-(M27-Pad3) -> +5V
- M29 pad 2: /led matrix/sheetA4B98B8C/ANODES -> Net-(M29-Pad2)
- M29 pad 3: Net-(M29-Pad3) -> +5V
- M3 pad 2: /led matrix/sheet9E2197FD/ANODES -> Net-(M3-Pad2)
- M3 pad 3: Net-(M3-Pad3) -> +5V
- M31 pad 2: /led matrix/sheetA4B98B8D/ANODES -> Net-(M31-Pad2)
- M31 pad 3: Net-(M31-Pad3) -> +5V
- M33 pad 2: /led matrix/sheetA575BE8D/ANODES -> Net-(M33-Pad2)
- M33 pad 3: Net-(M33-Pad3) -> +5V
- M35 pad 2: /led matrix/sheetA575BE8E/ANODES -> Net-(M35-Pad2)
- M35 pad 3: Net-(M35-Pad3) -> +5V
- M37 pad 2: /led matrix/sheetA575BE8F/ANODES -> Net-(M37-Pad2)
- M37 pad 3: Net-(M37-Pad3) -> +5V
- M39 pad 2: /led matrix/sheetA575BE90/ANODES -> Net-(M39-Pad2)
- M39 pad 3: Net-(M39-Pad3) -> +5V
- M41 pad 2: /led matrix/sheetA575BE91/ANODES -> Net-(M41-Pad2)
- M41 pad 3: Net-(M41-Pad3) -> +5V
- M43 pad 2: /led matrix/sheetA575BE92/ANODES -> Net-(M43-Pad2)
- M43 pad 3: Net-(M43-Pad3) -> +5V
- M45 pad 2: /led matrix/sheetA575BE93/ANODES -> Net-(M45-Pad2)
- M45 pad 3: Net-(M45-Pad3) -> +5V
- M47 pad 2: /led matrix/sheetA575BE94/ANODES -> Net-(M47-Pad2)
- M47 pad 3: Net-(M47-Pad3) -> +5V
- M49 pad 2: /led matrix/sheetA575BE95/ANODES -> Net-(M49-Pad2)
- M49 pad 3: Net-(M49-Pad3) -> +5V
- M5 pad 2: /led matrix/sheetA10E8493/ANODES -> Net-(M5-Pad2)
- M5 pad 3: Net-(M5-Pad3) -> +5V
- M51 pad 2: /led matrix/sheetA575BE96/ANODES -> Net-(M51-Pad2)
- M51 pad 3: Net-(M51-Pad3) -> +5V
- M53 pad 2: /led matrix/sheetA575BE97/ANODES -> Net-(M53-Pad2)
- M53 pad 3: Net-(M53-Pad3) -> +5V
- M55 pad 2: /led matrix/sheetA575BE98/ANODES -> Net-(M55-Pad2)
- M55 pad 3: Net-(M55-Pad3) -> +5V
- M57 pad 2: /led matrix/sheetA575BE99/ANODES -> Net-(M57-Pad2)
- M57 pad 3: Net-(M57-Pad3) -> +5V
- M59 pad 2: /led matrix/sheetA575BE9A/ANODES -> Net-(M59-Pad2)
- M59 pad 3: Net-(M59-Pad3) -> +5V
- M61 pad 2: /led matrix/sheetA575BE9B/ANODES -> Net-(M61-Pad2)
- M61 pad 3: Net-(M61-Pad3) -> +5V
- M63 pad 2: /led matrix/sheetA575BE9C/ANODES -> Net-(M63-Pad2)
- M63 pad 3: Net-(M63-Pad3) -> +5V
- M7 pad 2: /led matrix/sheetA10E8494/ANODES -> Net-(M7-Pad2)
- M7 pad 3: Net-(M7-Pad3) -> +5V
- M9 pad 2: /led matrix/sheetA341C37F/ANODES -> Net-(M9-Pad2)
- M9 pad 3: Net-(M9-Pad3) -> +5V
- R11 pad 1: +5V -> Net-(M7-Pad2)
- R11 pad 2: Net-(M7-Pad3) -> /led matrix/sheetA10E8494/ANODES
- R14 pad 1: +5V -> Net-(M9-Pad2)
- R14 pad 2: Net-(M9-Pad3) -> /led matrix/sheetA341C37F/ANODES
- R17 pad 1: +5V -> Net-(M11-Pad2)
- R17 pad 2: Net-(M11-Pad3) -> /led matrix/sheetA341C380/ANODES
- R2 pad 1: +5V -> Net-(M1-Pad2)
- R2 pad 2: Net-(M1-Pad3) -> /led matrix/common anode/ANODES
- R20 pad 1: +5V -> Net-(M13-Pad2)
- R20 pad 2: Net-(M13-Pad3) -> /led matrix/sheetA3FD3BF7/ANODES
- R23 pad 1: +5V -> Net-(M15-Pad2)
- R23 pad 2: Net-(M15-Pad3) -> /led matrix/sheetA3FD3BF8/ANODES
- R26 pad 1: +5V -> Net-(M17-Pad2)
- R26 pad 2: Net-(M17-Pad3) -> /led matrix/sheetA4B98B86/ANODES
- R29 pad 1: +5V -> Net-(M19-Pad2)
- R29 pad 2: Net-(M19-Pad3) -> /led matrix/sheetA4B98B87/ANODES
- R32 pad 1: +5V -> Net-(M21-Pad2)
- R32 pad 2: Net-(M21-Pad3) -> /led matrix/sheetA4B98B88/ANODES
- R35 pad 1: +5V -> Net-(M23-Pad2)
- R35 pad 2: Net-(M23-Pad3) -> /led matrix/sheetA4B98B89/ANODES
- R38 pad 1: +5V -> Net-(M25-Pad2)
- R38 pad 2: Net-(M25-Pad3) -> /led matrix/sheetA4B98B8A/ANODES
- R41 pad 1: +5V -> Net-(M27-Pad2)
- R41 pad 2: Net-(M27-Pad3) -> /led matrix/sheetA4B98B8B/ANODES
- R44 pad 1: +5V -> Net-(M29-Pad2)
- R44 pad 2: Net-(M29-Pad3) -> /led matrix/sheetA4B98B8C/ANODES
- R47 pad 1: +5V -> Net-(M31-Pad2)
- R47 pad 2: Net-(M31-Pad3) -> /led matrix/sheetA4B98B8D/ANODES
- R5 pad 1: +5V -> Net-(M3-Pad2)
- R5 pad 2: Net-(M3-Pad3) -> /led matrix/sheet9E2197FD/ANODES
- R50 pad 1: +5V -> Net-(M33-Pad2)
- R50 pad 2: Net-(M33-Pad3) -> /led matrix/sheetA575BE8D/ANODES
- R53 pad 1: +5V -> Net-(M35-Pad2)
- R53 pad 2: Net-(M35-Pad3) -> /led matrix/sheetA575BE8E/ANODES
- R56 pad 1: +5V -> Net-(M37-Pad2)
- R56 pad 2: Net-(M37-Pad3) -> /led matrix/sheetA575BE8F/ANODES
- R59 pad 1: +5V -> Net-(M39-Pad2)
- R59 pad 2: Net-(M39-Pad3) -> /led matrix/sheetA575BE90/ANODES
- R62 pad 1: +5V -> Net-(M41-Pad2)
- R62 pad 2: Net-(M41-Pad3) -> /led matrix/sheetA575BE91/ANODES
- R65 pad 1: +5V -> Net-(M43-Pad2)
- R65 pad 2: Net-(M43-Pad3) -> /led matrix/sheetA575BE92/ANODES
- R68 pad 1: +5V -> Net-(M45-Pad2)
- R68 pad 2: Net-(M45-Pad3) -> /led matrix/sheetA575BE93/ANODES
- R71 pad 1: +5V -> Net-(M47-Pad2)
- R71 pad 2: Net-(M47-Pad3) -> /led matrix/sheetA575BE94/ANODES
- R74 pad 1: +5V -> Net-(M49-Pad2)
- R74 pad 2: Net-(M49-Pad3) -> /led matrix/sheetA575BE95/ANODES
- R77 pad 1: +5V -> Net-(M51-Pad2)
- R77 pad 2: Net-(M51-Pad3) -> /led matrix/sheetA575BE96/ANODES
- R8 pad 1: +5V -> Net-(M5-Pad2)
- R8 pad 2: Net-(M5-Pad3) -> /led matrix/sheetA10E8493/ANODES
- R80 pad 1: +5V -> Net-(M53-Pad2)
- R80 pad 2: Net-(M53-Pad3) -> /led matrix/sheetA575BE97/ANODES
- R83 pad 1: +5V -> Net-(M55-Pad2)
- R83 pad 2: Net-(M55-Pad3) -> /led matrix/sheetA575BE98/ANODES
- R86 pad 1: +5V -> Net-(M57-Pad2)
- R86 pad 2: Net-(M57-Pad3) -> /led matrix/sheetA575BE99/ANODES
- R89 pad 1: +5V -> Net-(M59-Pad2)
- R89 pad 2: Net-(M59-Pad3) -> /led matrix/sheetA575BE9A/ANODES
- R92 pad 1: +5V -> Net-(M61-Pad2)
- R92 pad 2: Net-(M61-Pad3) -> /led matrix/sheetA575BE9B/ANODES
- R95 pad 1: +5V -> Net-(M63-Pad2)
- R95 pad 2: Net-(M63-Pad3) -> /led matrix/sheetA575BE9C/ANODES
Routing:
- net /led matrix/sheetD7D8B720/CATHODES: track 128.9 -> 133.9 mm, vias 32 -> 33
- net Net-(M66-Pad1): track 0.00 -> 4.94 mm
- net /led matrix/sheetD89BE98B/CATHODES: track 128.9 -> 131.9 mm, vias 32 -> 33
- net /led matrix/common cathode/CATHODES: track 128.9 -> 131.9 mm, vias 32 -> 33
- net GND: track 0.00 -> 1.76 mm, vias 0 -> 2
- net Net-(M66-Pad3): track 0.00 -> 1.66 mm
- net (no net): track 0.00 -> 0.74 mm, vias 0 -> 1

Commit message: Backup LEDdriver progress
Parts:
- added C26: 1u/6V3, Capacitor_SMD:C_0805_2012Metric, F.Cu at (-8.87, 71.0)
- added C27: 0u1/6V3, Capacitor_SMD:C_0402_1005Metric, F.Cu at (-3.84, 72.5)
- added C5: 0u1/6V3, Capacitor_SMD:C_0402_1005Metric, F.Cu at (-6.75, 75.5)
- added J3: Conn_01x06, Connector_PinHeader_2.54mm:PinHeader_1x06_P2.54mm_Horizontal, F.Cu at (-22.2, 71.8)
- added R198: 22R, Resistor_SMD:R_0402_1005Metric, F.Cu at (-9.64, 73.5)
- added R199: 22R, Resistor_SMD:R_0402_1005Metric, F.Cu at (-5.19, 70.5)
- added R200: 22R, Resistor_SMD:R_0402_1005Metric, F.Cu at (-9.64, 75.5)
- added R201: 22R, Resistor_SMD:R_0402_1005Metric, F.Cu at (-6.73, 73.5)
- added R202: 470R, Resistor_SMD:R_0402_1005Metric, F.Cu at (-2.28, 70.5)
- added R203: 10K, Resistor_SMD:R_0402_1005Metric, F.Cu at (-9.64, 77.5)
- C2, C3: value 1u/6V3 -> 4u7/6V3
- moved R91 254.4 mm to (21.2, 99.0)
- moved M62 252.6 mm to (18.2, 97.8)
- moved R93 243.9 mm to (21.2, 96.6)
- moved M61 242.6 mm to (24.2, 97.8), turned to 180 degrees
- moved R92 241.1 mm to (28.5, 97.8)
- moved R67 232.1 mm to (21.2, 75.0)
- moved R79 227.6 mm to (21.3, 87.0)
- moved M46 226.1 mm to (18.2, 73.8)
- moved R69 225.9 mm to (21.2, 72.5)
- moved M45 224.6 mm to (24.2, 73.8), turned to 180 degrees
- moved R27 222.9 mm to (21.2, 30.5)
- moved R39 222.7 mm to (21.2, 42.5)
- moved M18 221.6 mm to (18.2, 31.8)
- moved M54 221.6 mm to (18.2, 85.8)
- moved M53 220.1 mm to (24.2, 85.8), turned to 180 degrees
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Connections:
- C6 pad 1: (no net) -> GND
- C6 pad 2: (no net) -> +3V3
- DCDC1 pad 5: (no net) -> Net-(DCDC1-Pad5)
- J1 pad 2: (no net) -> Net-(J1-Pad2)
- J1 pad 3: (no net) -> Net-(J1-Pad3)
- J1 pad 4: (no net) -> Net-(J1-Pad4)
- MCU1 pad 1: (no net) -> Net-(MCU1-Pad1)
- MCU1 pad 12: (no net) -> Net-(MCU1-Pad12)
- MCU1 pad 13: (no net) -> Net-(MCU1-Pad13)
- MCU1 pad 14: (no net) -> Net-(C5-Pad2)
- MCU1 pad 15: (no net) -> Net-(MCU1-Pad15)
- MCU1 pad 16: (no net) -> Net-(MCU1-Pad16)
- MCU1 pad 17: (no net) -> Net-(MCU1-Pad17)
- MCU1 pad 18: (no net) -> Net-(MCU1-Pad18)
- MCU1 pad 2: (no net) -> Net-(MCU1-Pad2)
- MCU1 pad 23: (no net) -> Net-(MCU1-Pad23)
- MCU1 pad 24: (no net) -> Net-(MCU1-Pad24)
- MCU1 pad 25: (no net) -> Net-(MCU1-Pad25)
- MCU1 pad 26: (no net) -> Net-(MCU1-Pad26)
- MCU1 pad 29: (no net) -> Net-(MCU1-Pad29)
- MCU1 pad 3: (no net) -> Net-(MCU1-Pad3)
- MCU1 pad 30: (no net) -> Net-(MCU1-Pad30)
- MCU1 pad 31: (no net) -> Net-(MCU1-Pad31)
- MCU1 pad 32: (no net) -> Net-(MCU1-Pad32)
- MCU1 pad 33: (no net) -> Net-(MCU1-Pad33)
- MCU1 pad 34: (no net) -> Net-(MCU1-Pad34)
- MCU1 pad 35: (no net) -> Net-(MCU1-Pad35)
- MCU1 pad 36: (no net) -> Net-(MCU1-Pad36)
- MCU1 pad 37: (no net) -> Net-(MCU1-Pad37)
- MCU1 pad 38: (no net) -> Net-(MCU1-Pad38)
- MCU1 pad 39: (no net) -> Net-(MCU1-Pad39)
- MCU1 pad 4: (no net) -> Net-(MCU1-Pad4)
- MCU1 pad 40: (no net) -> Net-(MCU1-Pad40)
- MCU1 pad 41: (no net) -> Net-(MCU1-Pad41)
- MCU1 pad 42: (no net) -> Net-(MCU1-Pad42)
- MCU1 pad 43: (no net) -> Net-(MCU1-Pad43)
- MCU1 pad 44: (no net) -> Net-(MCU1-Pad44)
- MCU1 pad 45: (no net) -> Net-(MCU1-Pad45)
- MCU1 pad 46: (no net) -> Net-(MCU1-Pad46)
- MCU1 pad 47: (no net) -> Net-(MCU1-Pad47)
- MCU1 pad 5: (no net) -> Net-(MCU1-Pad5)
- MCU1 pad 51: (no net) -> Net-(MCU1-Pad51)
- MCU1 pad 52: (no net) -> Net-(MCU1-Pad52)
- MCU1 pad 53: (no net) -> Net-(MCU1-Pad53)
- MCU1 pad 54: (no net) -> Net-(MCU1-Pad54)
- MCU1 pad 55: (no net) -> Net-(MCU1-Pad55)
- MCU1 pad 56: (no net) -> Net-(MCU1-Pad56)
- MCU1 pad 57: (no net) -> Net-(MCU1-Pad57)
- MCU1 pad 58: (no net) -> Net-(MCU1-Pad58)
- MCU1 pad 59: (no net) -> Net-(MCU1-Pad59)
- MCU1 pad 6: (no net) -> +3V3
- MCU1 pad 60: (no net) -> Net-(MCU1-Pad60)
- MCU1 pad 61: (no net) -> Net-(MCU1-Pad61)
- MCU1 pad 62: (no net) -> Net-(MCU1-Pad62)
- MCU1 pad 63: (no net) -> Net-(MCU1-Pad63)
- MCU1 pad 64: (no net) -> Net-(MCU1-Pad64)
- MCU1 pad 65: (no net) -> Net-(MCU1-Pad65)
- MCU1 pad 66: (no net) -> Net-(MCU1-Pad66)
- MCU1 pad 67: (no net) -> Net-(MCU1-Pad67)
- MCU1 pad 68: (no net) -> Net-(MCU1-Pad68)
- MCU1 pad 69: (no net) -> Net-(MCU1-Pad69)
- MCU1 pad 7: (no net) -> Net-(MCU1-Pad7)
- MCU1 pad 70: (no net) -> Net-(MCU1-Pad70)
- MCU1 pad 71: (no net) -> Net-(MCU1-Pad71)
- MCU1 pad 72: (no net) -> SWDIO
- MCU1 pad 76: (no net) -> SWCLK
- MCU1 pad 77: (no net) -> Net-(MCU1-Pad77)
- MCU1 pad 78: (no net) -> Net-(MCU1-Pad78)
- MCU1 pad 79: (no net) -> Net-(MCU1-Pad79)
- MCU1 pad 8: (no net) -> Net-(MCU1-Pad8)
- MCU1 pad 80: (no net) -> Net-(MCU1-Pad80)
- MCU1 pad 81: (no net) -> Net-(MCU1-Pad81)
- MCU1 pad 82: (no net) -> Net-(MCU1-Pad82)
- MCU1 pad 83: (no net) -> Net-(MCU1-Pad83)
- MCU1 pad 84: (no net) -> Net-(MCU1-Pad84)
- MCU1 pad 85: (no net) -> Net-(MCU1-Pad85)
- MCU1 pad 86: (no net) -> Net-(MCU1-Pad86)
- MCU1 pad 87: (no net) -> Net-(MCU1-Pad87)
- MCU1 pad 88: (no net) -> Net-(MCU1-Pad88)
- MCU1 pad 89: (no net) -> SWO
- MCU1 pad 9: (no net) -> Net-(MCU1-Pad9)
- MCU1 pad 90: (no net) -> Net-(MCU1-Pad90)
- MCU1 pad 91: (no net) -> Net-(MCU1-Pad91)
- MCU1 pad 92: (no net) -> Net-(MCU1-Pad92)
- MCU1 pad 93: (no net) -> Net-(MCU1-Pad93)
- MCU1 pad 94: (no net) -> Net-(MCU1-Pad94)
- MCU1 pad 95: (no net) -> Net-(MCU1-Pad95)
- MCU1 pad 96: (no net) -> Net-(MCU1-Pad96)
- MCU1 pad 97: (no net) -> Net-(MCU1-Pad97)
- MCU1 pad 98: (no net) -> Net-(MCU1-Pad98)
- R101 pad 2: (no net) -> y1
- R104 pad 2: (no net) -> y2
- R107 pad 2: (no net) -> y3
- R110 pad 2: (no net) -> y4
- R113 pad 2: (no net) -> y5
- R116 pad 2: (no net) -> y6
- R119 pad 2: (no net) -> y7
- R12 pad 2: (no net) -> x3
- R122 pad 2: (no net) -> y8
- R125 pad 2: (no net) -> y9
- R128 pad 2: (no net) -> y10
- R131 pad 2: (no net) -> y11
- R134 pad 2: (no net) -> y12
- R137 pad 2: (no net) -> y13
- R140 pad 2: (no net) -> y14
- R143 pad 2: (no net) -> y15
- R146 pad 2: (no net) -> y16
- R149 pad 2: (no net) -> y17
- R15 pad 2: (no net) -> x4
- R152 pad 2: (no net) -> y18
- R155 pad 2: (no net) -> y19
- R158 pad 2: (no net) -> y20
- R161 pad 2: (no net) -> y21
- R164 pad 2: (no net) -> y22
- R167 pad 2: (no net) -> y23
- R170 pad 2: (no net) -> y24
- R173 pad 2: (no net) -> y25
- R176 pad 2: (no net) -> y26
- R179 pad 2: (no net) -> y27
- R18 pad 2: (no net) -> x5
- R182 pad 2: (no net) -> y28
- R185 pad 2: (no net) -> y29
- R188 pad 2: (no net) -> y30
- R191 pad 2: (no net) -> y31
- R21 pad 2: (no net) -> x6
- R24 pad 2: (no net) -> x7
- R27 pad 2: (no net) -> x8
- R3 pad 2: (no net) -> x0
- R30 pad 2: (no net) -> x9
- R33 pad 2: (no net) -> x10
- R36 pad 2: (no net) -> x11
- R39 pad 2: (no net) -> x12
- R42 pad 2: (no net) -> x13
- R45 pad 2: (no net) -> x14
- R48 pad 2: (no net) -> x15
- R51 pad 2: (no net) -> x16
- R54 pad 2: (no net) -> x17
- R57 pad 2: (no net) -> x18
- R6 pad 2: (no net) -> x1
- R60 pad 2: (no net) -> x19
- R63 pad 2: (no net) -> x20
- R66 pad 2: (no net) -> x21
- R69 pad 2: (no net) -> x22
- R72 pad 2: (no net) -> x23
- R75 pad 2: (no net) -> x24
- R78 pad 2: (no net) -> x25
- R81 pad 2: (no net) -> x26
- R84 pad 2: (no net) -> x27
- R87 pad 2: (no net) -> x28
- R9 pad 2: (no net) -> x2
- R90 pad 2: (no net) -> x29
- R93 pad 2: (no net) -> x30
- R96 pad 2: (no net) -> x31
- R98 pad 2: (no net) -> y0
- U1 pad 4: (no net) -> spi_sclk
- U1 pad 6: (no net) -> spi_mosi
- U1 pad 7: (no net) -> spi_miso
- U1 pad 8: (no net) -> spi_cs_acc
- U2 pad 12: (no net) -> Net-(U2-Pad12)
- U2 pad 13: (no net) -> Net-(U2-Pad13)
- U2 pad 14: (no net) -> Net-(U2-Pad14)
- U2 pad 7: (no net) -> Net-(U2-Pad7)
Routing:
- net +5V: track 0.00 -> 56.8 mm, vias 0 -> 49
- net /led matrix/sheetA575BE91/ANODES: track 41.4 -> 95.2 mm
- net /led matrix/sheetA575BE94/ANODES: track 67.3 -> 92.6 mm
- net /led matrix/sheetA575BE99/ANODES: track 85.3 -> 95.8 mm
- net Net-(M5-Pad1): track 0.00 -> 7.22 mm
- net Net-(M57-Pad1): track 0.00 -> 7.13 mm
- net Net-(M10-Pad3): track 0.00 -> 7.13 mm
- net Net-(M1-Pad1): track 0.00 -> 7.12 mm
- net Net-(M45-Pad1): track 0.00 -> 7.09 mm
- net Net-(M17-Pad1): track 0.00 -> 7.08 mm
- net Net-(M13-Pad1): track 0.00 -> 7.08 mm
- net Net-(M35-Pad1): track 0.00 -> 7.08 mm
- net Net-(M31-Pad1): track 0.00 -> 7.08 mm
- net Net-(M27-Pad1): track 0.00 -> 7.08 mm
- net Net-(M21-Pad1): track 0.00 -> 7.08 mm
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
Commit message: Added All the FETs
All the FETs were Added
And it looks awsome
Parts:
- moved R132 302.6 mm to (66.8, -3.93), turned to 180 degrees
- moved R131 296.0 mm to (69.2, -3.93)
- moved R129 280.9 mm to (66.3, 114.0)
- moved R114 274.8 mm to (48.7, -3.97), turned to 180 degrees
- moved R130 273.2 mm to (68.0, 3.57), turned to 90 degrees
- moved R113 271.9 mm to (51.2, -3.97)
- moved M70 268.6 mm to (50.0, -0.97), turned to 270 degrees
- moved R112 268.2 mm to (50.0, 3.53), turned to 90 degrees
- moved R121 263.3 mm to (59.0, 106.5), turned to 270 degrees
- moved R123 263.1 mm to (60.3, 114.0)
- moved R122 260.7 mm to (57.8, 114.0), turned to 180 degrees
- moved M73 259.9 mm to (59.0, 111.0), turned to 90 degrees
- moved R127 255.5 mm to (65.0, 106.5), turned to 270 degrees
- moved C1 255.0 mm to (74.3, -3.70), turned to 90 degrees
- moved R119 254.0 mm to (57.2, -3.97)
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Routing:
- net GND: track 1.76 -> 33.4 mm, vias 2 -> 33
- net +5V: track 56.8 -> 83.0 mm, vias 49 -> 64
- net Net-(M59-Pad1): track 0.00 -> 7.12 mm
- net Net-(M51-Pad1): track 0.00 -> 7.12 mm
- net Net-(M63-Pad1): track 0.00 -> 7.12 mm
- net Net-(M55-Pad1): track 0.00 -> 7.12 mm
- net Net-(M43-Pad1): track 0.00 -> 7.12 mm
- net Net-(M47-Pad1): track 0.00 -> 7.12 mm
- net Net-(M39-Pad1): track 0.00 -> 7.12 mm
- net /led matrix/sheetDAE5EEF6/CATHODES: track 128.9 -> 134.0 mm, vias 32 -> 33
- net /led matrix/sheetDAE5EEF8/CATHODES: track 128.9 -> 134.0 mm, vias 32 -> 33
- net /led matrix/sheetD95F2321/CATHODES: track 128.9 -> 133.9 mm, vias 32 -> 33
- net /led matrix/sheetDAE5EF02/CATHODES: track 128.9 -> 133.9 mm, vias 32 -> 33
- net /led matrix/sheetDA226153/CATHODES: track 128.9 -> 133.9 mm, vias 32 -> 33
- net /led matrix/sheetDA226151/CATHODES: track 128.9 -> 133.9 mm, vias 32 -> 33
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