File: hard/led_matrix.kicad_pcb (KiCad board)
At the start: 2 copper layers, 160 x 110 mm, 1363 parts, among them J1 MicroXNJ, J2 PJ-3062-CO, J3 Conn_01x06, M1 IRLML6402TRPBF, M10 2N7002,215, M11 IRLML6402TRPBF, M12 2N7002,215, M13 IRLML6402TRPBF, M14 2N7002,215, M15 IRLML6402TRPBF, M16 2N7002,215, M17 IRLML6402TRPBF, M18 2N7002,215, M19 IRLML6402TRPBF, M2 2N7002,215, M20 2N7002,215, M21 IRLML6402TRPBF, M22 2N7002,215, M23 IRLML6402TRPBF, M24 2N7002,215, M25 IRLML6402TRPBF, M26 2N7002,215, M27 IRLML6402TRPBF, M28 2N7002,215, M29 IRLML6402TRPBF, M3 IRLML6402TRPBF, M30 2N7002,215, M31 IRLML6402TRPBF, M32 2N7002,215, M33 IRLML6402TRPBF, M34 2N7002,215, M35 IRLML6402TRPBF, M36 2N7002,215, M37 IRLML6402TRPBF, M38 2N7002,215, M39 IRLML6402TRPBF, M4 2N7002,215, M40 2N7002,215, M41 IRLML6402TRPBF, M42 2N7002,215, M43 IRLML6402TRPBF, M44 2N7002,215, M45 IRLML6402TRPBF, M46 2N7002,215, M47 IRLML6402TRPBF, M48 2N7002,215, M49 IRLML6402TRPBF, M5 IRLML6402TRPBF, M50 2N7002,215, M51 IRLML6402TRPBF, M52 2N7002,215, M53 IRLML6402TRPBF, M54 2N7002,215, M55 IRLML6402TRPBF, M56 2N7002,215, M57 IRLML6402TRPBF, M58 2N7002,215, M59 IRLML6402TRPBF, M6 2N7002,215, M60 2N7002,215, M61 IRLML6402TRPBF, M62 2N7002,215, M63 IRLML6402TRPBF, M64 2N7002,215, M65 IRLML0030TRPBF, M66 IRLML0030TRPBF, M67 IRLML0030TRPBF, M68 IRLML0030TRPBF, M69 IRLML0030TRPBF, M7 IRLML6402TRPBF, M70 IRLML0030TRPBF, M71 IRLML0030TRPBF, M72 IRLML0030TRPBF, M73 IRLML0030TRPBF, M74 IRLML0030TRPBF, M75 IRLML0030TRPBF, M76 IRLML0030TRPBF, M77 IRLML0030TRPBF, M78 IRLML0030TRPBF, M79 IRLML0030TRPBF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

Commit message: added led driver layout by @lukekaese
Parts:
- removed the C5 at (-6.75, 75.5)
- removed the C5 at (340.7, 56.1)
- removed the J3 at (-22.2, 71.8)
- added C5: 0u1/6V3, Capacitor_SMD:C_0402_1005Metric, F.Cu at (23.5, 80.0)
- added D1028: PSM712-LF-T7, Package_TO_SOT_SMD:SOT-23, F.Cu at (185.4, 86.2)
- added G***: LOGO, led_matrix:logo2, F.Cu at (176.2, 36.2)
- added G***: LOGO, led_matrix:logo, F.Cu at (186.0, 36.5)
- added J2: MicroXNJ, led_matrix:Connectors_SHOU HAN_MICRO 4P DIP, F.Cu at (15.0, -0.05)
- added M97: IRLML0030TRPBF, Package_TO_SOT_SMD:SOT-23, F.Cu at (148.0, 6.55)
- added R204: 0R1, Resistor_SMD:R_0805_2012Metric, F.Cu at (7.00, 2.00)
- added R205: 22K/1%, Resistor_SMD:R_0402_1005Metric, F.Cu at (21.2, 95.8)
- added R206: 100R, Resistor_SMD:R_0603_1608Metric, F.Cu at (186.9, 82.0)
- added R207: 100R, Resistor_SMD:R_0603_1608Metric, F.Cu at (184.4, 78.0)
- C14: value 0u1/6V3 -> 1u/6V3; footprint Capacitor_SMD:C_0402_1005Metric -> Capacitor_SMD:C_0805_2012Metric
- C15: value 100n/16V -> 0u1/6V3
- C16: value 22u/16V -> 0u1/6V3; footprint Capacitor_SMD:C_0805_2012Metric -> Capacitor_SMD:C_0402_1005Metric
- C17: value 22u/16V -> 100n/16V; footprint Capacitor_SMD:C_0805_2012Metric -> Capacitor_SMD:C_0402_1005Metric
- C19: value 68p/16V -> 22u/16V; footprint Capacitor_SMD:C_0402_1005Metric -> Capacitor_SMD:C_0805_2012Metric
- C2: value 4u7/6V3 -> 0u1/6V3; footprint Capacitor_SMD:C_0805_2012Metric -> Capacitor_SMD:C_0402_1005Metric
- C21: value 22u/16V -> 68p/16V; footprint Capacitor_SMD:C_0805_2012Metric -> Capacitor_SMD:C_0402_1005Metric
- C22, C23: value 0u1/6V3 -> 22u/16V; footprint Capacitor_SMD:C_0402_1005Metric -> Capacitor_SMD:C_0805_2012Metric
- C24: value 1u/6V3 -> 0u1/6V3; footprint Capacitor_SMD:C_0603_1608Metric -> Capacitor_SMD:C_0402_1005Metric
- C26: footprint Capacitor_SMD:C_0805_2012Metric -> Capacitor_SMD:C_0603_1608Metric
- C4: value 0u1/6V3 -> 4u7/6V3; footprint Capacitor_SMD:C_0402_1005Metric -> Capacitor_SMD:C_0805_2012Metric
- D1025: value D_Zener -> LTST-S270TBKT; footprint Diode_SMD:D_MiniMELF -> led_matrix:LED_LiteOn_LTST-S270TBKT
- D1027: value PSM712-LF-T7 -> D_Zener; footprint Package_TO_SOT_SMD:SOT-23 -> Diode_SMD:D_MiniMELF
- J1: value MicroXNJ -> Conn_01x06; footprint led_matrix:Connectors_SHOU HAN_MICRO 4P DIP -> Connector_PinHeader_2.54mm:PinHeader_1x06_P2.54mm_Vertical
- M1, M11, M13, M15, M17, M19, M21, M23, M25, M27, M29, M3, M31, M33, M35, M37, M39, M41, M43, M45, M47, M49, M5, M51, M53, M55, M57, M59, M61, M63, M7, M9: value IRLML6402TRPBF -> 2N7002,215
- M10, M12, M14, M16, M18, M2, M20, M22, M24, M26, M28, M30, M32, M34, M36, M38, M4, M40, M42, M44, M46, M48, M50, M52, M54, M56, M58, M6, M60, M62, M64, M8: value 2N7002,215 -> IRLML6402TRPBF
- M65: value IRLML0030TRPBF -> 2N7002,215
- R1, R4: value 1K -> 22R
- R10: value 1K -> 1K8
- R100, R103, R106, R97: value 0R -> 120R
- R101, R104, R98: value 1K8 -> 1K
- R102, R105, R108, R111, R114, R117, R120, R123, R126, R129, R132, R135, R138, R141, R144, R147, R150, R153, R156, R159, R162, R165, R168, R171, R174, R177, R180, R183, R186, R189, R192, R99: value 470K -> 1K8
- R107, R110, R113, R116, R119, R122, R125, R128, R131, R134, R137, R140, R143, R146, R149, R152, R155, R158, R161, R164, R167, R170, R173, R176, R179, R182, R185, R188, R191: value 1K8 -> 0R; footprint Resistor_SMD:R_0402_1005Metric -> Resistor_SMD:R_1210_3225Metric
- R109, R112, R115, R118, R121, R124, R127, R130, R133, R136, R139, R142, R145, R148, R151, R154, R157, R160, R163, R166, R169, R172, R175, R178, R181, R184, R187, R190: value 0R -> 470K; footprint Resistor_SMD:R_1210_3225Metric -> Resistor_SMD:R_0402_1005Metric
- R11, R14, R17, R20, R23, R26, R29, R32, R35, R38, R41, R44, R47, R50, R53, R56, R59, R62, R65, R68, R71, R74, R77, R80, R83, R86, R89, R92, R95: value 120R -> 1K; footprint Resistor_SMD:R_1210_3225Metric -> Resistor_SMD:R_0402_1005Metric
- R13, R16, R19, R22, R25, R28, R31, R34, R37, R40, R43, R46, R49, R52, R55, R58, R61, R64, R67, R70, R73, R76, R79, R82, R85, R88, R91, R94: value 1K -> 120R; footprint Resistor_SMD:R_0402_1005Metric -> Resistor_SMD:R_1210_3225Metric
- R193: value 100K/1% -> 470K
- R194: value 0R1 -> 0R; footprint Resistor_SMD:R_0805_2012Metric -> Resistor_SMD:R_1210_3225Metric
- R195: value 22K/1% -> 1K8
- R196: value 100R -> 470K; footprint Resistor_SMD:R_0603_1608Metric -> Resistor_SMD:R_0402_1005Metric
- R197: value 100R -> 0R; footprint Resistor_SMD:R_0603_1608Metric -> Resistor_SMD:R_1210_3225Metric
- R198, R201: value 22R -> 1K8
- R199: value 22R -> 470K
- R2: value 120R -> 22R; footprint Resistor_SMD:R_1210_3225Metric -> Resistor_SMD:R_0402_1005Metric
- R200: value 22R -> 0R; footprint Resistor_SMD:R_0402_1005Metric -> Resistor_SMD:R_1210_3225Metric
- R202: value 470R -> 470K
- R203: value 10K -> 100K/1%
- R3: value 1K8 -> 22R
- R5: value 120R -> 3K3; footprint Resistor_SMD:R_1210_3225Metric -> Resistor_SMD:R_0402_1005Metric
- R6, R9: value 1K8 -> 3K3
- R7: value 1K -> 470R
- R8: value 120R -> 10K; footprint Resistor_SMD:R_1210_3225Metric -> Resistor_SMD:R_0402_1005Metric
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- renumbered J2 to J3
Connections:
- C14 pad 1: +3V3 -> GND
- C14 pad 2: GND -> Net-(C12-Pad2)
- C15 pad 1: Net-(C15-Pad1) -> GND
- C15 pad 2: Net-(C15-Pad2) -> Net-(C12-Pad2)
- C16 pad 1: +5V -> +3V3
- C17 pad 1: GND -> Net-(C17-Pad1)
- C17 pad 2: +5V -> Net-(C17-Pad2)
- C18 pad 1: GND -> +5V
- C18 pad 2: +5V -> GND
- C19 pad 1: Net-(C19-Pad1) -> GND
- C19 pad 2: +3V3 -> +5V
- C20 pad 2: +3V3 -> +5V
- C21 pad 1: GND -> Net-(C21-Pad1)
- C26 pad 2: Net-(C12-Pad2) -> +3V3
- C27 pad 2: Net-(C12-Pad2) -> +3V3
- C4 pad 1: +3V3 -> GND
- C4 pad 2: GND -> Net-(C4-Pad2)
- D1 pad A: /led matrix/common anode/ANODES -> Net-(D1-PadA)
- D1 pad C: /led matrix/common cathode/CATHODES -> Net-(D1-PadC)
- D10 pad C: /led matrix/sheetDA22614E/CATHODES -> /led matrix/sheetDA22614D/CATHODES
- D100 pad C: /led matrix/sheetD89BE98C/CATHODES -> /led matrix/sheetD89BE98B/CATHODES
- D1000 pad C: /led matrix/sheetD95F2324/CATHODES -> /led matrix/sheetD95F2323/CATHODES
- D1001 pad C: /led matrix/sheetDA22614D/CATHODES -> /led matrix/sheetD95F2324/CATHODES
- D1002 pad C: /led matrix/sheetDA22614E/CATHODES -> /led matrix/sheetDA22614D/CATHODES
- D1003 pad C: /led matrix/sheetDA22614F/CATHODES -> /led matrix/sheetDA22614E/CATHODES
- D1004 pad C: /led matrix/sheetDA226150/CATHODES -> /led matrix/sheetDA22614F/CATHODES
- D1005 pad C: /led matrix/sheetDA226151/CATHODES -> /led matrix/sheetDA226150/CATHODES
- D1006 pad C: /led matrix/sheetDA226152/CATHODES -> /led matrix/sheetDA226151/CATHODES
- D1007 pad C: /led matrix/sheetDA226153/CATHODES -> /led matrix/sheetDA226152/CATHODES
- D1008 pad C: /led matrix/sheetDA226154/CATHODES -> /led matrix/sheetDA226153/CATHODES
- D1009 pad C: /led matrix/sheetDAE5EEF6/CATHODES -> /led matrix/sheetDA226154/CATHODES
- D101 pad C: /led matrix/sheetD95F2321/CATHODES -> /led matrix/sheetD89BE98C/CATHODES
- D1010 pad C: /led matrix/sheetDAE5EEF7/CATHODES -> /led matrix/sheetDAE5EEF6/CATHODES
- D1011 pad C: /led matrix/sheetDAE5EEF8/CATHODES -> /led matrix/sheetDAE5EEF7/CATHODES
- D1012 pad C: /led matrix/sheetDAE5EEF9/CATHODES -> /led matrix/sheetDAE5EEF8/CATHODES
- D1013 pad C: /led matrix/sheetDAE5EEFA/CATHODES -> /led matrix/sheetDAE5EEF9/CATHODES
- D1014 pad C: /led matrix/sheetDAE5EEFB/CATHODES -> /led matrix/sheetDAE5EEFA/CATHODES
- D1015 pad C: /led matrix/sheetDAE5EEFC/CATHODES -> /led matrix/sheetDAE5EEFB/CATHODES
- D1016 pad C: /led matrix/sheetDAE5EEFD/CATHODES -> /led matrix/sheetDAE5EEFC/CATHODES
- D1017 pad C: /led matrix/sheetDAE5EEFE/CATHODES -> /led matrix/sheetDAE5EEFD/CATHODES
- D1018 pad C: /led matrix/sheetDAE5EEFF/CATHODES -> /led matrix/sheetDAE5EEFE/CATHODES
- D1019 pad C: /led matrix/sheetDAE5EF00/CATHODES -> /led matrix/sheetDAE5EEFF/CATHODES
- D102 pad C: /led matrix/sheetD95F2322/CATHODES -> /led matrix/sheetD95F2321/CATHODES
- D1020 pad C: /led matrix/sheetDAE5EF01/CATHODES -> /led matrix/sheetDAE5EF00/CATHODES
- D1021 pad C: /led matrix/sheetDAE5EF02/CATHODES -> /led matrix/sheetDAE5EF01/CATHODES
- D1022 pad C: /led matrix/sheetDAE5EF03/CATHODES -> /led matrix/sheetDAE5EF02/CATHODES
- D1023 pad C: /led matrix/sheetDAE5EF04/CATHODES -> /led matrix/sheetDAE5EF03/CATHODES
- D1024 pad C: /led matrix/sheetDAE5EF05/CATHODES -> /led matrix/sheetDAE5EF04/CATHODES
- D1026 pad 1: analog_ring -> analog_tip
- D1027 pad 1: Net-(D1027-Pad1) -> analog_ring
- D1027 pad 2: Net-(D1027-Pad2) -> GND
- D103 pad C: /led matrix/sheetD95F2323/CATHODES -> /led matrix/sheetD95F2322/CATHODES
- D104 pad C: /led matrix/sheetD95F2324/CATHODES -> /led matrix/sheetD95F2323/CATHODES
- D105 pad C: /led matrix/sheetDA22614D/CATHODES -> /led matrix/sheetD95F2324/CATHODES
- D106 pad C: /led matrix/sheetDA22614E/CATHODES -> /led matrix/sheetDA22614D/CATHODES
- D107 pad C: /led matrix/sheetDA22614F/CATHODES -> /led matrix/sheetDA22614E/CATHODES
- D108 pad C: /led matrix/sheetDA226150/CATHODES -> /led matrix/sheetDA22614F/CATHODES
- D109 pad C: /led matrix/sheetDA226151/CATHODES -> /led matrix/sheetDA226150/CATHODES
- D11 pad C: /led matrix/sheetDA22614F/CATHODES -> /led matrix/sheetDA22614E/CATHODES
- D110 pad C: /led matrix/sheetDA226152/CATHODES -> /led matrix/sheetDA226151/CATHODES
- D111 pad C: /led matrix/sheetDA226153/CATHODES -> /led matrix/sheetDA226152/CATHODES
- D112 pad C: /led matrix/sheetDA226154/CATHODES -> /led matrix/sheetDA226153/CATHODES
- D113 pad C: /led matrix/sheetDAE5EEF6/CATHODES -> /led matrix/sheetDA226154/CATHODES
- D114 pad C: /led matrix/sheetDAE5EEF7/CATHODES -> /led matrix/sheetDAE5EEF6/CATHODES
- D115 pad C: /led matrix/sheetDAE5EEF8/CATHODES -> /led matrix/sheetDAE5EEF7/CATHODES
- D116 pad C: /led matrix/sheetDAE5EEF9/CATHODES -> /led matrix/sheetDAE5EEF8/CATHODES
- D117 pad C: /led matrix/sheetDAE5EEFA/CATHODES -> /led matrix/sheetDAE5EEF9/CATHODES
- D118 pad C: /led matrix/sheetDAE5EEFB/CATHODES -> /led matrix/sheetDAE5EEFA/CATHODES
- D119 pad C: /led matrix/sheetDAE5EEFC/CATHODES -> /led matrix/sheetDAE5EEFB/CATHODES
- D12 pad C: /led matrix/sheetDA226150/CATHODES -> /led matrix/sheetDA22614F/CATHODES
- D120 pad C: /led matrix/sheetDAE5EEFD/CATHODES -> /led matrix/sheetDAE5EEFC/CATHODES
- D121 pad C: /led matrix/sheetDAE5EEFE/CATHODES -> /led matrix/sheetDAE5EEFD/CATHODES
- D122 pad C: /led matrix/sheetDAE5EEFF/CATHODES -> /led matrix/sheetDAE5EEFE/CATHODES
- D123 pad C: /led matrix/sheetDAE5EF00/CATHODES -> /led matrix/sheetDAE5EEFF/CATHODES
- D124 pad C: /led matrix/sheetDAE5EF01/CATHODES -> /led matrix/sheetDAE5EF00/CATHODES
- D125 pad C: /led matrix/sheetDAE5EF02/CATHODES -> /led matrix/sheetDAE5EF01/CATHODES
- D126 pad C: /led matrix/sheetDAE5EF03/CATHODES -> /led matrix/sheetDAE5EF02/CATHODES
- D127 pad C: /led matrix/sheetDAE5EF04/CATHODES -> /led matrix/sheetDAE5EF03/CATHODES
- D128 pad C: /led matrix/sheetDAE5EF05/CATHODES -> /led matrix/sheetDAE5EF04/CATHODES
- D129 pad A: /led matrix/sheetA341C37F/ANODES -> /led matrix/sheetA10E8494/ANODES
- D129 pad C: /led matrix/common cathode/CATHODES -> /led matrix/sheetDAE5EF05/CATHODES
- D13 pad C: /led matrix/sheetDA226151/CATHODES -> /led matrix/sheetDA226150/CATHODES
- D130 pad C: /led matrix/sheetD7D8B720/CATHODES -> /led matrix/common cathode/CATHODES
- D131 pad C: /led matrix/sheetD89BE98B/CATHODES -> /led matrix/sheetD7D8B720/CATHODES
- D132 pad C: /led matrix/sheetD89BE98C/CATHODES -> /led matrix/sheetD89BE98B/CATHODES
- D133 pad C: /led matrix/sheetD95F2321/CATHODES -> /led matrix/sheetD89BE98C/CATHODES
- D134 pad C: /led matrix/sheetD95F2322/CATHODES -> /led matrix/sheetD95F2321/CATHODES
- D135 pad C: /led matrix/sheetD95F2323/CATHODES -> /led matrix/sheetD95F2322/CATHODES
- D136 pad C: /led matrix/sheetD95F2324/CATHODES -> /led matrix/sheetD95F2323/CATHODES
- D137 pad C: /led matrix/sheetDA22614D/CATHODES -> /led matrix/sheetD95F2324/CATHODES
- D138 pad C: /led matrix/sheetDA22614E/CATHODES -> /led matrix/sheetDA22614D/CATHODES
- D139 pad C: /led matrix/sheetDA22614F/CATHODES -> /led matrix/sheetDA22614E/CATHODES
- D14 pad C: /led matrix/sheetDA226152/CATHODES -> /led matrix/sheetDA226151/CATHODES
- D140 pad C: /led matrix/sheetDA226150/CATHODES -> /led matrix/sheetDA22614F/CATHODES
- D141 pad C: /led matrix/sheetDA226151/CATHODES -> /led matrix/sheetDA226150/CATHODES
- D142 pad C: /led matrix/sheetDA226152/CATHODES -> /led matrix/sheetDA226151/CATHODES
- D143 pad C: /led matrix/sheetDA226153/CATHODES -> /led matrix/sheetDA226152/CATHODES
- D144 pad C: /led matrix/sheetDA226154/CATHODES -> /led matrix/sheetDA226153/CATHODES
- D145 pad C: /led matrix/sheetDAE5EEF6/CATHODES -> /led matrix/sheetDA226154/CATHODES
- D146 pad C: /led matrix/sheetDAE5EEF7/CATHODES -> /led matrix/sheetDAE5EEF6/CATHODES
- D147 pad C: /led matrix/sheetDAE5EEF8/CATHODES -> /led matrix/sheetDAE5EEF7/CATHODES
- D148 pad C: /led matrix/sheetDAE5EEF9/CATHODES -> /led matrix/sheetDAE5EEF8/CATHODES
- D149 pad C: /led matrix/sheetDAE5EEFA/CATHODES -> /led matrix/sheetDAE5EEF9/CATHODES
- D15 pad C: /led matrix/sheetDA226153/CATHODES -> /led matrix/sheetDA226152/CATHODES
- D150 pad C: /led matrix/sheetDAE5EEFB/CATHODES -> /led matrix/sheetDAE5EEFA/CATHODES
- D151 pad C: /led matrix/sheetDAE5EEFC/CATHODES -> /led matrix/sheetDAE5EEFB/CATHODES
- D152 pad C: /led matrix/sheetDAE5EEFD/CATHODES -> /led matrix/sheetDAE5EEFC/CATHODES
- D153 pad C: /led matrix/sheetDAE5EEFE/CATHODES -> /led matrix/sheetDAE5EEFD/CATHODES
- D154 pad C: /led matrix/sheetDAE5EEFF/CATHODES -> /led matrix/sheetDAE5EEFE/CATHODES
- D155 pad C: /led matrix/sheetDAE5EF00/CATHODES -> /led matrix/sheetDAE5EEFF/CATHODES
- D156 pad C: /led matrix/sheetDAE5EF01/CATHODES -> /led matrix/sheetDAE5EF00/CATHODES
- D157 pad C: /led matrix/sheetDAE5EF02/CATHODES -> /led matrix/sheetDAE5EF01/CATHODES
- D158 pad C: /led matrix/sheetDAE5EF03/CATHODES -> /led matrix/sheetDAE5EF02/CATHODES
- D159 pad C: /led matrix/sheetDAE5EF04/CATHODES -> /led matrix/sheetDAE5EF03/CATHODES
- D16 pad C: /led matrix/sheetDA226154/CATHODES -> /led matrix/sheetDA226153/CATHODES
- D160 pad C: /led matrix/sheetDAE5EF05/CATHODES -> /led matrix/sheetDAE5EF04/CATHODES
- D161 pad A: /led matrix/sheetA341C380/ANODES -> /led matrix/sheetA341C37F/ANODES
- D161 pad C: /led matrix/common cathode/CATHODES -> /led matrix/sheetDAE5EF05/CATHODES
- D162 pad C: /led matrix/sheetD7D8B720/CATHODES -> /led matrix/common cathode/CATHODES
- D163 pad C: /led matrix/sheetD89BE98B/CATHODES -> /led matrix/sheetD7D8B720/CATHODES
- D164 pad C: /led matrix/sheetD89BE98C/CATHODES -> /led matrix/sheetD89BE98B/CATHODES
- D165 pad C: /led matrix/sheetD95F2321/CATHODES -> /led matrix/sheetD89BE98C/CATHODES
- D166 pad C: /led matrix/sheetD95F2322/CATHODES -> /led matrix/sheetD95F2321/CATHODES
- D167 pad C: /led matrix/sheetD95F2323/CATHODES -> /led matrix/sheetD95F2322/CATHODES
- D168 pad C: /led matrix/sheetD95F2324/CATHODES -> /led matrix/sheetD95F2323/CATHODES
- D169 pad C: /led matrix/sheetDA22614D/CATHODES -> /led matrix/sheetD95F2324/CATHODES
- D17 pad C: /led matrix/sheetDAE5EEF6/CATHODES -> /led matrix/sheetDA226154/CATHODES
- D170 pad C: /led matrix/sheetDA22614E/CATHODES -> /led matrix/sheetDA22614D/CATHODES
- D171 pad C: /led matrix/sheetDA22614F/CATHODES -> /led matrix/sheetDA22614E/CATHODES
- D172 pad C: /led matrix/sheetDA226150/CATHODES -> /led matrix/sheetDA22614F/CATHODES
- D173 pad C: /led matrix/sheetDA226151/CATHODES -> /led matrix/sheetDA226150/CATHODES
- D174 pad C: /led matrix/sheetDA226152/CATHODES -> /led matrix/sheetDA226151/CATHODES
- D175 pad C: /led matrix/sheetDA226153/CATHODES -> /led matrix/sheetDA226152/CATHODES
- D176 pad C: /led matrix/sheetDA226154/CATHODES -> /led matrix/sheetDA226153/CATHODES
- D177 pad C: /led matrix/sheetDAE5EEF6/CATHODES -> /led matrix/sheetDA226154/CATHODES
- D178 pad C: /led matrix/sheetDAE5EEF7/CATHODES -> /led matrix/sheetDAE5EEF6/CATHODES
- D179 pad C: /led matrix/sheetDAE5EEF8/CATHODES -> /led matrix/sheetDAE5EEF7/CATHODES
- D18 pad C: /led matrix/sheetDAE5EEF7/CATHODES -> /led matrix/sheetDAE5EEF6/CATHODES
- D180 pad C: /led matrix/sheetDAE5EEF9/CATHODES -> /led matrix/sheetDAE5EEF8/CATHODES
- D181 pad C: /led matrix/sheetDAE5EEFA/CATHODES -> /led matrix/sheetDAE5EEF9/CATHODES
- D182 pad C: /led matrix/sheetDAE5EEFB/CATHODES -> /led matrix/sheetDAE5EEFA/CATHODES
- D183 pad C: /led matrix/sheetDAE5EEFC/CATHODES -> /led matrix/sheetDAE5EEFB/CATHODES
- D184 pad C: /led matrix/sheetDAE5EEFD/CATHODES -> /led matrix/sheetDAE5EEFC/CATHODES
- D185 pad C: /led matrix/sheetDAE5EEFE/CATHODES -> /led matrix/sheetDAE5EEFD/CATHODES
- D186 pad C: /led matrix/sheetDAE5EEFF/CATHODES -> /led matrix/sheetDAE5EEFE/CATHODES
- D187 pad C: /led matrix/sheetDAE5EF00/CATHODES -> /led matrix/sheetDAE5EEFF/CATHODES
- D188 pad C: /led matrix/sheetDAE5EF01/CATHODES -> /led matrix/sheetDAE5EF00/CATHODES
- D189 pad C: /led matrix/sheetDAE5EF02/CATHODES -> /led matrix/sheetDAE5EF01/CATHODES
- D19 pad C: /led matrix/sheetDAE5EEF8/CATHODES -> /led matrix/sheetDAE5EEF7/CATHODES
- D190 pad C: /led matrix/sheetDAE5EF03/CATHODES -> /led matrix/sheetDAE5EF02/CATHODES
- D191 pad C: /led matrix/sheetDAE5EF04/CATHODES -> /led matrix/sheetDAE5EF03/CATHODES
- D192 pad C: /led matrix/sheetDAE5EF05/CATHODES -> /led matrix/sheetDAE5EF04/CATHODES
- D193 pad A: /led matrix/sheetA3FD3BF7/ANODES -> /led matrix/sheetA341C380/ANODES
- D193 pad C: /led matrix/common cathode/CATHODES -> /led matrix/sheetDAE5EF05/CATHODES
- D194 pad C: /led matrix/sheetD7D8B720/CATHODES -> /led matrix/common cathode/CATHODES
- D195 pad C: /led matrix/sheetD89BE98B/CATHODES -> /led matrix/sheetD7D8B720/CATHODES
- D196 pad C: /led matrix/sheetD89BE98C/CATHODES -> /led matrix/sheetD89BE98B/CATHODES
- D197 pad C: /led matrix/sheetD95F2321/CATHODES -> /led matrix/sheetD89BE98C/CATHODES
- D198 pad C: /led matrix/sheetD95F2322/CATHODES -> /led matrix/sheetD95F2321/CATHODES
- D199 pad C: /led matrix/sheetD95F2323/CATHODES -> /led matrix/sheetD95F2322/CATHODES
- D2 pad C: /led matrix/sheetD7D8B720/CATHODES -> /led matrix/common cathode/CATHODES
- D20 pad C: /led matrix/sheetDAE5EEF9/CATHODES -> /led matrix/sheetDAE5EEF8/CATHODES
- D200 pad C: /led matrix/sheetD95F2324/CATHODES -> /led matrix/sheetD95F2323/CATHODES
- D201 pad C: /led matrix/sheetDA22614D/CATHODES -> /led matrix/sheetD95F2324/CATHODES
- D202 pad C: /led matrix/sheetDA22614E/CATHODES -> /led matrix/sheetDA22614D/CATHODES
- D203 pad C: /led matrix/sheetDA22614F/CATHODES -> /led matrix/sheetDA22614E/CATHODES
- D204 pad C: /led matrix/sheetDA226150/CATHODES -> /led matrix/sheetDA22614F/CATHODES
- D205 pad C: /led matrix/sheetDA226151/CATHODES -> /led matrix/sheetDA226150/CATHODES
- D206 pad C: /led matrix/sheetDA226152/CATHODES -> /led matrix/sheetDA226151/CATHODES
- D207 pad C: /led matrix/sheetDA226153/CATHODES -> /led matrix/sheetDA226152/CATHODES
- D208 pad C: /led matrix/sheetDA226154/CATHODES -> /led matrix/sheetDA226153/CATHODES
- D209 pad C: /led matrix/sheetDAE5EEF6/CATHODES -> /led matrix/sheetDA226154/CATHODES
- D21 pad C: /led matrix/sheetDAE5EEFA/CATHODES -> /led matrix/sheetDAE5EEF9/CATHODES
- D210 pad C: /led matrix/sheetDAE5EEF7/CATHODES -> /led matrix/sheetDAE5EEF6/CATHODES
- D211 pad C: /led matrix/sheetDAE5EEF8/CATHODES -> /led matrix/sheetDAE5EEF7/CATHODES
- D212 pad C: /led matrix/sheetDAE5EEF9/CATHODES -> /led matrix/sheetDAE5EEF8/CATHODES
- D213 pad C: /led matrix/sheetDAE5EEFA/CATHODES -> /led matrix/sheetDAE5EEF9/CATHODES
- D214 pad C: /led matrix/sheetDAE5EEFB/CATHODES -> /led matrix/sheetDAE5EEFA/CATHODES
- D215 pad C: /led matrix/sheetDAE5EEFC/CATHODES -> /led matrix/sheetDAE5EEFB/CATHODES
- D216 pad C: /led matrix/sheetDAE5EEFD/CATHODES -> /led matrix/sheetDAE5EEFC/CATHODES
- D217 pad C: /led matrix/sheetDAE5EEFE/CATHODES -> /led matrix/sheetDAE5EEFD/CATHODES
- D218 pad C: /led matrix/sheetDAE5EEFF/CATHODES -> /led matrix/sheetDAE5EEFE/CATHODES
- D219 pad C: /led matrix/sheetDAE5EF00/CATHODES -> /led matrix/sheetDAE5EEFF/CATHODES
- D22 pad C: /led matrix/sheetDAE5EEFB/CATHODES -> /led matrix/sheetDAE5EEFA/CATHODES
- D220 pad C: /led matrix/sheetDAE5EF01/CATHODES -> /led matrix/sheetDAE5EF00/CATHODES
- D221 pad C: /led matrix/sheetDAE5EF02/CATHODES -> /led matrix/sheetDAE5EF01/CATHODES
- D222 pad C: /led matrix/sheetDAE5EF03/CATHODES -> /led matrix/sheetDAE5EF02/CATHODES
- D223 pad C: /led matrix/sheetDAE5EF04/CATHODES -> /led matrix/sheetDAE5EF03/CATHODES
- D224 pad C: /led matrix/sheetDAE5EF05/CATHODES -> /led matrix/sheetDAE5EF04/CATHODES
- D225 pad A: /led matrix/sheetA3FD3BF8/ANODES -> /led matrix/sheetA3FD3BF7/ANODES
- D225 pad C: /led matrix/common cathode/CATHODES -> /led matrix/sheetDAE5EF05/CATHODES
- D226 pad C: /led matrix/sheetD7D8B720/CATHODES -> /led matrix/common cathode/CATHODES
- D227 pad C: /led matrix/sheetD89BE98B/CATHODES -> /led matrix/sheetD7D8B720/CATHODES
- D228 pad C: /led matrix/sheetD89BE98C/CATHODES -> /led matrix/sheetD89BE98B/CATHODES
- D229 pad C: /led matrix/sheetD95F2321/CATHODES -> /led matrix/sheetD89BE98C/CATHODES
- D23 pad C: /led matrix/sheetDAE5EEFC/CATHODES -> /led matrix/sheetDAE5EEFB/CATHODES
- D230 pad C: /led matrix/sheetD95F2322/CATHODES -> /led matrix/sheetD95F2321/CATHODES
- D231 pad C: /led matrix/sheetD95F2323/CATHODES -> /led matrix/sheetD95F2322/CATHODES
- D232 pad C: /led matrix/sheetD95F2324/CATHODES -> /led matrix/sheetD95F2323/CATHODES
- D233 pad C: /led matrix/sheetDA22614D/CATHODES -> /led matrix/sheetD95F2324/CATHODES
- D234 pad C: /led matrix/sheetDA22614E/CATHODES -> /led matrix/sheetDA22614D/CATHODES
- D235 pad C: /led matrix/sheetDA22614F/CATHODES -> /led matrix/sheetDA22614E/CATHODES
- D236 pad C: /led matrix/sheetDA226150/CATHODES -> /led matrix/sheetDA22614F/CATHODES
- D237 pad C: /led matrix/sheetDA226151/CATHODES -> /led matrix/sheetDA226150/CATHODES
- D238 pad C: /led matrix/sheetDA226152/CATHODES -> /led matrix/sheetDA226151/CATHODES
- D239 pad C: /led matrix/sheetDA226153/CATHODES -> /led matrix/sheetDA226152/CATHODES
- D24 pad C: /led matrix/sheetDAE5EEFD/CATHODES -> /led matrix/sheetDAE5EEFC/CATHODES
- D240 pad C: /led matrix/sheetDA226154/CATHODES -> /led matrix/sheetDA226153/CATHODES
- D241 pad C: /led matrix/sheetDAE5EEF6/CATHODES -> /led matrix/sheetDA226154/CATHODES
- D242 pad C: /led matrix/sheetDAE5EEF7/CATHODES -> /led matrix/sheetDAE5EEF6/CATHODES
- D243 pad C: /led matrix/sheetDAE5EEF8/CATHODES -> /led matrix/sheetDAE5EEF7/CATHODES
- D244 pad C: /led matrix/sheetDAE5EEF9/CATHODES -> /led matrix/sheetDAE5EEF8/CATHODES
- D245 pad C: /led matrix/sheetDAE5EEFA/CATHODES -> /led matrix/sheetDAE5EEF9/CATHODES
- D246 pad C: /led matrix/sheetDAE5EEFB/CATHODES -> /led matrix/sheetDAE5EEFA/CATHODES
- D247 pad C: /led matrix/sheetDAE5EEFC/CATHODES -> /led matrix/sheetDAE5EEFB/CATHODES
- D248 pad C: /led matrix/sheetDAE5EEFD/CATHODES -> /led matrix/sheetDAE5EEFC/CATHODES
- D249 pad C: /led matrix/sheetDAE5EEFE/CATHODES -> /led matrix/sheetDAE5EEFD/CATHODES
- D25 pad C: /led matrix/sheetDAE5EEFE/CATHODES -> /led matrix/sheetDAE5EEFD/CATHODES
- D250 pad C: /led matrix/sheetDAE5EEFF/CATHODES -> /led matrix/sheetDAE5EEFE/CATHODES
- D251 pad C: /led matrix/sheetDAE5EF00/CATHODES -> /led matrix/sheetDAE5EEFF/CATHODES
- D252 pad C: /led matrix/sheetDAE5EF01/CATHODES -> /led matrix/sheetDAE5EF00/CATHODES
- D253 pad C: /led matrix/sheetDAE5EF02/CATHODES -> /led matrix/sheetDAE5EF01/CATHODES
- D254 pad C: /led matrix/sheetDAE5EF03/CATHODES -> /led matrix/sheetDAE5EF02/CATHODES
- D255 pad C: /led matrix/sheetDAE5EF04/CATHODES -> /led matrix/sheetDAE5EF03/CATHODES
- D256 pad C: /led matrix/sheetDAE5EF05/CATHODES -> /led matrix/sheetDAE5EF04/CATHODES
- D257 pad A: /led matrix/sheetA4B98B86/ANODES -> /led matrix/sheetA3FD3BF8/ANODES
- D257 pad C: /led matrix/common cathode/CATHODES -> /led matrix/sheetDAE5EF05/CATHODES
- D258 pad C: /led matrix/sheetD7D8B720/CATHODES -> /led matrix/common cathode/CATHODES
- D259 pad C: /led matrix/sheetD89BE98B/CATHODES -> /led matrix/sheetD7D8B720/CATHODES
- D26 pad C: /led matrix/sheetDAE5EEFF/CATHODES -> /led matrix/sheetDAE5EEFE/CATHODES
- D260 pad C: /led matrix/sheetD89BE98C/CATHODES -> /led matrix/sheetD89BE98B/CATHODES
- D261 pad C: /led matrix/sheetD95F2321/CATHODES -> /led matrix/sheetD89BE98C/CATHODES
- D262 pad C: /led matrix/sheetD95F2322/CATHODES -> /led matrix/sheetD95F2321/CATHODES
- D263 pad C: /led matrix/sheetD95F2323/CATHODES -> /led matrix/sheetD95F2322/CATHODES
- D264 pad C: /led matrix/sheetD95F2324/CATHODES -> /led matrix/sheetD95F2323/CATHODES
- D265 pad C: /led matrix/sheetDA22614D/CATHODES -> /led matrix/sheetD95F2324/CATHODES
- D266 pad C: /led matrix/sheetDA22614E/CATHODES -> /led matrix/sheetDA22614D/CATHODES
- D267 pad C: /led matrix/sheetDA22614F/CATHODES -> /led matrix/sheetDA22614E/CATHODES
- D268 pad C: /led matrix/sheetDA226150/CATHODES -> /led matrix/sheetDA22614F/CATHODES
- D269 pad C: /led matrix/sheetDA226151/CATHODES -> /led matrix/sheetDA226150/CATHODES
- D27 pad C: /led matrix/sheetDAE5EF00/CATHODES -> /led matrix/sheetDAE5EEFF/CATHODES
- D270 pad C: /led matrix/sheetDA226152/CATHODES -> /led matrix/sheetDA226151/CATHODES
- D271 pad C: /led matrix/sheetDA226153/CATHODES -> /led matrix/sheetDA226152/CATHODES
- D272 pad C: /led matrix/sheetDA226154/CATHODES -> /led matrix/sheetDA226153/CATHODES
- D273 pad C: /led matrix/sheetDAE5EEF6/CATHODES -> /led matrix/sheetDA226154/CATHODES
- D274 pad C: /led matrix/sheetDAE5EEF7/CATHODES -> /led matrix/sheetDAE5EEF6/CATHODES
- D275 pad C: /led matrix/sheetDAE5EEF8/CATHODES -> /led matrix/sheetDAE5EEF7/CATHODES
- D276 pad C: /led matrix/sheetDAE5EEF9/CATHODES -> /led matrix/sheetDAE5EEF8/CATHODES
- D277 pad C: /led matrix/sheetDAE5EEFA/CATHODES -> /led matrix/sheetDAE5EEF9/CATHODES
- D278 pad C: /led matrix/sheetDAE5EEFB/CATHODES -> /led matrix/sheetDAE5EEFA/CATHODES
- D279 pad C: /led matrix/sheetDAE5EEFC/CATHODES -> /led matrix/sheetDAE5EEFB/CATHODES
- D28 pad C: /led matrix/sheetDAE5EF01/CATHODES -> /led matrix/sheetDAE5EF00/CATHODES
- D280 pad C: /led matrix/sheetDAE5EEFD/CATHODES -> /led matrix/sheetDAE5EEFC/CATHODES
- D281 pad C: /led matrix/sheetDAE5EEFE/CATHODES -> /led matrix/sheetDAE5EEFD/CATHODES
- D282 pad C: /led matrix/sheetDAE5EEFF/CATHODES -> /led matrix/sheetDAE5EEFE/CATHODES
- D283 pad C: /led matrix/sheetDAE5EF00/CATHODES -> /led matrix/sheetDAE5EEFF/CATHODES
- D284 pad C: /led matrix/sheetDAE5EF01/CATHODES -> /led matrix/sheetDAE5EF00/CATHODES
- D285 pad C: /led matrix/sheetDAE5EF02/CATHODES -> /led matrix/sheetDAE5EF01/CATHODES
- D286 pad C: /led matrix/sheetDAE5EF03/CATHODES -> /led matrix/sheetDAE5EF02/CATHODES
- D287 pad C: /led matrix/sheetDAE5EF04/CATHODES -> /led matrix/sheetDAE5EF03/CATHODES
- D288 pad C: /led matrix/sheetDAE5EF05/CATHODES -> /led matrix/sheetDAE5EF04/CATHODES
- D289 pad A: /led matrix/sheetA4B98B87/ANODES -> /led matrix/sheetA4B98B86/ANODES
- D289 pad C: /led matrix/common cathode/CATHODES -> /led matrix/sheetDAE5EF05/CATHODES
- D29 pad C: /led matrix/sheetDAE5EF02/CATHODES -> /led matrix/sheetDAE5EF01/CATHODES
- D290 pad C: /led matrix/sheetD7D8B720/CATHODES -> /led matrix/common cathode/CATHODES
- D291 pad C: /led matrix/sheetD89BE98B/CATHODES -> /led matrix/sheetD7D8B720/CATHODES
- D292 pad C: /led matrix/sheetD89BE98C/CATHODES -> /led matrix/sheetD89BE98B/CATHODES
- D293 pad C: /led matrix/sheetD95F2321/CATHODES -> /led matrix/sheetD89BE98C/CATHODES
- D294 pad C: /led matrix/sheetD95F2322/CATHODES -> /led matrix/sheetD95F2321/CATHODES
- D295 pad C: /led matrix/sheetD95F2323/CATHODES -> /led matrix/sheetD95F2322/CATHODES
- D296 pad C: /led matrix/sheetD95F2324/CATHODES -> /led matrix/sheetD95F2323/CATHODES
- D297 pad C: /led matrix/sheetDA22614D/CATHODES -> /led matrix/sheetD95F2324/CATHODES
- D298 pad C: /led matrix/sheetDA22614E/CATHODES -> /led matrix/sheetDA22614D/CATHODES
- D299 pad C: /led matrix/sheetDA22614F/CATHODES -> /led matrix/sheetDA22614E/CATHODES
- D3 pad C: /led matrix/sheetD89BE98B/CATHODES -> /led matrix/sheetD7D8B720/CATHODES
- D30 pad C: /led matrix/sheetDAE5EF03/CATHODES -> /led matrix/sheetDAE5EF02/CATHODES
- D300 pad C: /led matrix/sheetDA226150/CATHODES -> /led matrix/sheetDA22614F/CATHODES
- D301 pad C: /led matrix/sheetDA226151/CATHODES -> /led matrix/sheetDA226150/CATHODES
- D302 pad C: /led matrix/sheetDA226152/CATHODES -> /led matrix/sheetDA226151/CATHODES
- D303 pad C: /led matrix/sheetDA226153/CATHODES -> /led matrix/sheetDA226152/CATHODES
- D304 pad C: /led matrix/sheetDA226154/CATHODES -> /led matrix/sheetDA226153/CATHODES
- D305 pad C: /led matrix/sheetDAE5EEF6/CATHODES -> /led matrix/sheetDA226154/CATHODES
- D306 pad C: /led matrix/sheetDAE5EEF7/CATHODES -> /led matrix/sheetDAE5EEF6/CATHODES
- D307 pad C: /led matrix/sheetDAE5EEF8/CATHODES -> /led matrix/sheetDAE5EEF7/CATHODES
- D308 pad C: /led matrix/sheetDAE5EEF9/CATHODES -> /led matrix/sheetDAE5EEF8/CATHODES
- D309 pad C: /led matrix/sheetDAE5EEFA/CATHODES -> /led matrix/sheetDAE5EEF9/CATHODES
- D31 pad C: /led matrix/sheetDAE5EF04/CATHODES -> /led matrix/sheetDAE5EF03/CATHODES
- D310 pad C: /led matrix/sheetDAE5EEFB/CATHODES -> /led matrix/sheetDAE5EEFA/CATHODES
- D311 pad C: /led matrix/sheetDAE5EEFC/CATHODES -> /led matrix/sheetDAE5EEFB/CATHODES
- D312 pad C: /led matrix/sheetDAE5EEFD/CATHODES -> /led matrix/sheetDAE5EEFC/CATHODES
- D313 pad C: /led matrix/sheetDAE5EEFE/CATHODES -> /led matrix/sheetDAE5EEFD/CATHODES
- D314 pad C: /led matrix/sheetDAE5EEFF/CATHODES -> /led matrix/sheetDAE5EEFE/CATHODES
- D315 pad C: /led matrix/sheetDAE5EF00/CATHODES -> /led matrix/sheetDAE5EEFF/CATHODES
- D316 pad C: /led matrix/sheetDAE5EF01/CATHODES -> /led matrix/sheetDAE5EF00/CATHODES
- D317 pad C: /led matrix/sheetDAE5EF02/CATHODES -> /led matrix/sheetDAE5EF01/CATHODES
- D318 pad C: /led matrix/sheetDAE5EF03/CATHODES -> /led matrix/sheetDAE5EF02/CATHODES
- D319 pad C: /led matrix/sheetDAE5EF04/CATHODES -> /led matrix/sheetDAE5EF03/CATHODES
- D32 pad C: /led matrix/sheetDAE5EF05/CATHODES -> /led matrix/sheetDAE5EF04/CATHODES
- D320 pad C: /led matrix/sheetDAE5EF05/CATHODES -> /led matrix/sheetDAE5EF04/CATHODES
- D321 pad A: /led matrix/sheetA4B98B88/ANODES -> /led matrix/sheetA4B98B87/ANODES
- D321 pad C: /led matrix/common cathode/CATHODES -> /led matrix/sheetDAE5EF05/CATHODES
- D322 pad C: /led matrix/sheetD7D8B720/CATHODES -> /led matrix/common cathode/CATHODES
- D323 pad C: /led matrix/sheetD89BE98B/CATHODES -> /led matrix/sheetD7D8B720/CATHODES
- D324 pad C: /led matrix/sheetD89BE98C/CATHODES -> /led matrix/sheetD89BE98B/CATHODES
- D325 pad C: /led matrix/sheetD95F2321/CATHODES -> /led matrix/sheetD89BE98C/CATHODES
- D326 pad C: /led matrix/sheetD95F2322/CATHODES -> /led matrix/sheetD95F2321/CATHODES
- D327 pad C: /led matrix/sheetD95F2323/CATHODES -> /led matrix/sheetD95F2322/CATHODES
- D328 pad C: /led matrix/sheetD95F2324/CATHODES -> /led matrix/sheetD95F2323/CATHODES
- D329 pad C: /led matrix/sheetDA22614D/CATHODES -> /led matrix/sheetD95F2324/CATHODES
- D33 pad A: /led matrix/sheet9E2197FD/ANODES -> /led matrix/common anode/ANODES
- D33 pad C: /led matrix/common cathode/CATHODES -> /led matrix/sheetDAE5EF05/CATHODES
- D330 pad C: /led matrix/sheetDA22614E/CATHODES -> /led matrix/sheetDA22614D/CATHODES
- D331 pad C: /led matrix/sheetDA22614F/CATHODES -> /led matrix/sheetDA22614E/CATHODES
- D332 pad C: /led matrix/sheetDA226150/CATHODES -> /led matrix/sheetDA22614F/CATHODES
- D333 pad C: /led matrix/sheetDA226151/CATHODES -> /led matrix/sheetDA226150/CATHODES
- D334 pad C: /led matrix/sheetDA226152/CATHODES -> /led matrix/sheetDA226151/CATHODES
- D335 pad C: /led matrix/sheetDA226153/CATHODES -> /led matrix/sheetDA226152/CATHODES
- D336 pad C: /led matrix/sheetDA226154/CATHODES -> /led matrix/sheetDA226153/CATHODES
- D337 pad C: /led matrix/sheetDAE5EEF6/CATHODES -> /led matrix/sheetDA226154/CATHODES
- D338 pad C: /led matrix/sheetDAE5EEF7/CATHODES -> /led matrix/sheetDAE5EEF6/CATHODES
- D339 pad C: /led matrix/sheetDAE5EEF8/CATHODES -> /led matrix/sheetDAE5EEF7/CATHODES
- D34 pad C: /led matrix/sheetD7D8B720/CATHODES -> /led matrix/common cathode/CATHODES
- D340 pad C: /led matrix/sheetDAE5EEF9/CATHODES -> /led matrix/sheetDAE5EEF8/CATHODES
- D341 pad C: /led matrix/sheetDAE5EEFA/CATHODES -> /led matrix/sheetDAE5EEF9/CATHODES
- D342 pad C: /led matrix/sheetDAE5EEFB/CATHODES -> /led matrix/sheetDAE5EEFA/CATHODES
- D343 pad C: /led matrix/sheetDAE5EEFC/CATHODES -> /led matrix/sheetDAE5EEFB/CATHODES
- D344 pad C: /led matrix/sheetDAE5EEFD/CATHODES -> /led matrix/sheetDAE5EEFC/CATHODES
- D345 pad C: /led matrix/sheetDAE5EEFE/CATHODES -> /led matrix/sheetDAE5EEFD/CATHODES
- D346 pad C: /led matrix/sheetDAE5EEFF/CATHODES -> /led matrix/sheetDAE5EEFE/CATHODES
- D347 pad C: /led matrix/sheetDAE5EF00/CATHODES -> /led matrix/sheetDAE5EEFF/CATHODES
- D348 pad C: /led matrix/sheetDAE5EF01/CATHODES -> /led matrix/sheetDAE5EF00/CATHODES
- D349 pad C: /led matrix/sheetDAE5EF02/CATHODES -> /led matrix/sheetDAE5EF01/CATHODES
- D35 pad C: /led matrix/sheetD89BE98B/CATHODES -> /led matrix/sheetD7D8B720/CATHODES
- D350 pad C: /led matrix/sheetDAE5EF03/CATHODES -> /led matrix/sheetDAE5EF02/CATHODES
- D351 pad C: /led matrix/sheetDAE5EF04/CATHODES -> /led matrix/sheetDAE5EF03/CATHODES
- D352 pad C: /led matrix/sheetDAE5EF05/CATHODES -> /led matrix/sheetDAE5EF04/CATHODES
- D353 pad A: /led matrix/sheetA4B98B89/ANODES -> /led matrix/sheetA4B98B88/ANODES
- D353 pad C: /led matrix/common cathode/CATHODES -> /led matrix/sheetDAE5EF05/CATHODES
- D354 pad C: /led matrix/sheetD7D8B720/CATHODES -> /led matrix/common cathode/CATHODES
- D355 pad C: /led matrix/sheetD89BE98B/CATHODES -> /led matrix/sheetD7D8B720/CATHODES
- D356 pad C: /led matrix/sheetD89BE98C/CATHODES -> /led matrix/sheetD89BE98B/CATHODES
- D357 pad C: /led matrix/sheetD95F2321/CATHODES -> /led matrix/sheetD89BE98C/CATHODES
- D358 pad C: /led matrix/sheetD95F2322/CATHODES -> /led matrix/sheetD95F2321/CATHODES
- D359 pad C: /led matrix/sheetD95F2323/CATHODES -> /led matrix/sheetD95F2322/CATHODES
- D36 pad C: /led matrix/sheetD89BE98C/CATHODES -> /led matrix/sheetD89BE98B/CATHODES
- D360 pad C: /led matrix/sheetD95F2324/CATHODES -> /led matrix/sheetD95F2323/CATHODES
- D361 pad C: /led matrix/sheetDA22614D/CATHODES -> /led matrix/sheetD95F2324/CATHODES
- D362 pad C: /led matrix/sheetDA22614E/CATHODES -> /led matrix/sheetDA22614D/CATHODES
- D363 pad C: /led matrix/sheetDA22614F/CATHODES -> /led matrix/sheetDA22614E/CATHODES
- D364 pad C: /led matrix/sheetDA226150/CATHODES -> /led matrix/sheetDA22614F/CATHODES
- D365 pad C: /led matrix/sheetDA226151/CATHODES -> /led matrix/sheetDA226150/CATHODES
- D366 pad C: /led matrix/sheetDA226152/CATHODES -> /led matrix/sheetDA226151/CATHODES
- D367 pad C: /led matrix/sheetDA226153/CATHODES -> /led matrix/sheetDA226152/CATHODES
- D368 pad C: /led matrix/sheetDA226154/CATHODES -> /led matrix/sheetDA226153/CATHODES
- D369 pad C: /led matrix/sheetDAE5EEF6/CATHODES -> /led matrix/sheetDA226154/CATHODES
- D37 pad C: /led matrix/sheetD95F2321/CATHODES -> /led matrix/sheetD89BE98C/CATHODES
- D370 pad C: /led matrix/sheetDAE5EEF7/CATHODES -> /led matrix/sheetDAE5EEF6/CATHODES
- D371 pad C: /led matrix/sheetDAE5EEF8/CATHODES -> /led matrix/sheetDAE5EEF7/CATHODES
- D372 pad C: /led matrix/sheetDAE5EEF9/CATHODES -> /led matrix/sheetDAE5EEF8/CATHODES
- D373 pad C: /led matrix/sheetDAE5EEFA/CATHODES -> /led matrix/sheetDAE5EEF9/CATHODES
- D374 pad C: /led matrix/sheetDAE5EEFB/CATHODES -> /led matrix/sheetDAE5EEFA/CATHODES
- D375 pad C: /led matrix/sheetDAE5EEFC/CATHODES -> /led matrix/sheetDAE5EEFB/CATHODES
- D376 pad C: /led matrix/sheetDAE5EEFD/CATHODES -> /led matrix/sheetDAE5EEFC/CATHODES
- D377 pad C: /led matrix/sheetDAE5EEFE/CATHODES -> /led matrix/sheetDAE5EEFD/CATHODES
- D378 pad C: /led matrix/sheetDAE5EEFF/CATHODES -> /led matrix/sheetDAE5EEFE/CATHODES
- D379 pad C: /led matrix/sheetDAE5EF00/CATHODES -> /led matrix/sheetDAE5EEFF/CATHODES
- D38 pad C: /led matrix/sheetD95F2322/CATHODES -> /led matrix/sheetD95F2321/CATHODES
- D380 pad C: /led matrix/sheetDAE5EF01/CATHODES -> /led matrix/sheetDAE5EF00/CATHODES
- D381 pad C: /led matrix/sheetDAE5EF02/CATHODES -> /led matrix/sheetDAE5EF01/CATHODES
- D382 pad C: /led matrix/sheetDAE5EF03/CATHODES -> /led matrix/sheetDAE5EF02/CATHODES
- D383 pad C: /led matrix/sheetDAE5EF04/CATHODES -> /led matrix/sheetDAE5EF03/CATHODES
- D384 pad C: /led matrix/sheetDAE5EF05/CATHODES -> /led matrix/sheetDAE5EF04/CATHODES
- D385 pad A: /led matrix/sheetA4B98B8A/ANODES -> /led matrix/sheetA4B98B89/ANODES
- D385 pad C: /led matrix/common cathode/CATHODES -> /led matrix/sheetDAE5EF05/CATHODES
- D386 pad C: /led matrix/sheetD7D8B720/CATHODES -> /led matrix/common cathode/CATHODES
- D387 pad C: /led matrix/sheetD89BE98B/CATHODES -> /led matrix/sheetD7D8B720/CATHODES
- D388 pad C: /led matrix/sheetD89BE98C/CATHODES -> /led matrix/sheetD89BE98B/CATHODES
- D389 pad C: /led matrix/sheetD95F2321/CATHODES -> /led matrix/sheetD89BE98C/CATHODES
- D39 pad C: /led matrix/sheetD95F2323/CATHODES -> /led matrix/sheetD95F2322/CATHODES
- D390 pad C: /led matrix/sheetD95F2322/CATHODES -> /led matrix/sheetD95F2321/CATHODES
- D391 pad C: /led matrix/sheetD95F2323/CATHODES -> /led matrix/sheetD95F2322/CATHODES
- D392 pad C: /led matrix/sheetD95F2324/CATHODES -> /led matrix/sheetD95F2323/CATHODES
- D393 pad C: /led matrix/sheetDA22614D/CATHODES -> /led matrix/sheetD95F2324/CATHODES
- D394 pad C: /led matrix/sheetDA22614E/CATHODES -> /led matrix/sheetDA22614D/CATHODES
- D395 pad C: /led matrix/sheetDA22614F/CATHODES -> /led matrix/sheetDA22614E/CATHODES
- D396 pad C: /led matrix/sheetDA226150/CATHODES -> /led matrix/sheetDA22614F/CATHODES
- D397 pad C: /led matrix/sheetDA226151/CATHODES -> /led matrix/sheetDA226150/CATHODES
- D398 pad C: /led matrix/sheetDA226152/CATHODES -> /led matrix/sheetDA226151/CATHODES
- D399 pad C: /led matrix/sheetDA226153/CATHODES -> /led matrix/sheetDA226152/CATHODES
- D4 pad C: /led matrix/sheetD89BE98C/CATHODES -> /led matrix/sheetD89BE98B/CATHODES
- D40 pad C: /led matrix/sheetD95F2324/CATHODES -> /led matrix/sheetD95F2323/CATHODES
- D400 pad C: /led matrix/sheetDA226154/CATHODES -> /led matrix/sheetDA226153/CATHODES
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Routing:
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- added copper zone on B.Cu, net (none)
- added copper zone on F.Cu, net +3V3
- added copper zone on F.Cu, net +5V
- added copper zone on F.Cu, net Net-(C17-Pad1)
Other:
- board size 160 x 110 mm -> 200 x 125 mm
- copper layers 2 -> 4

Commit message: pcb format refactor
Parts:
- moved C18 187.8 mm to (11.0, 120.0)
- moved C19 187.8 mm to (7.99, 120.0)
- moved D1028 180.0 mm to (14.2, 30.5), turned to 0 degrees
- moved R206 175.8 mm to (18.5, 31.4), turned to 180 degrees
- moved D1027 174.7 mm to (22.0, 33.4), turned to 270 degrees
- moved R207 172.8 mm to (18.5, 29.5), turned to 0 degrees
- moved D1026 171.2 mm to (9.50, 106.8), turned to 180 degrees
- moved D1 153.0 mm to (27.5, 87.0)
- moved M1 153.0 mm to (28.6, 91.2)
- moved R10 153.0 mm to (31.8, 92.0)
- moved R5 153.0 mm to (31.8, 89.1)
- moved R6 153.0 mm to (27.3, 83.2)
- moved R9 153.0 mm to (29.8, 87.6)
- moved J2 18.1 mm to (-0.05, 10.0), turned to 270 degrees
- moved J3 18.0 mm to (11.6, 34.2)
Connections:
- J3 pad R: Net-(D1028-Pad1) -> Net-(D1028-Pad2)
- J3 pad T: Net-(D1028-Pad2) -> Net-(D1028-Pad1)
- R206 pad 2: Net-(D1028-Pad1) -> Net-(D1028-Pad2)
- R207 pad 1: Net-(D1028-Pad2) -> Net-(D1028-Pad1)
Routing:
- net Net-(D1028-Pad2): track 0.00 -> 9.81 mm
- net Net-(D1028-Pad1): track 0.00 -> 9.81 mm
- net GND: vias 39 -> 43
- net (no net): vias 11 -> 10
- added copper zone on B.Cu, net Net-(C17-Pad1)
- removed copper zone on B.Cu, net (none)
