File: hard/leds.sch (KiCad schematic (older format))
At the start: 0 parts

Commit message: signal nmos added
Parts:
- added D1: DIODE, symbol pspice:DIODE
- added D2: LED, symbol Device:LED
- added M1: IRLML6402TRPBF, Package_TO_SOT_SMD:SOT-23, symbol led_matrix:IRLML6402TRPBF
- added R1: 1K8, symbol Device:R
- added R2: 1K, symbol Device:R
- added R3: 120R, symbol Device:R
Connections:
- net labels added: +5V, GND
- wire segments 0 -> 8
Changed lines of the file:
@@
 Comment4 ""
 $EndDescr
+$Comp
+L Device:R R3
+U 1 1 6056B66E
+P 6000 1100
+F 0 "R3" H 6070 1146 50  0000 L CNN
+F 1 "120R" H 6070 1055 50  0000 L CNN
+F 2 "" V 5930 1100 50  0001 C CNN
+F 3 "~" H 6000 1100 50  0001 C CNN
+	1    6000 1100
+	1    0    0    -1
+$EndComp
+$Comp
+L Device:R R2
+U 1 1 6056C15C
+P 5000 1100
+F 0 "R2" H 5070 1146 50  0000 L CNN
+F 1 "1K" H 5070 1055 50  0000 L CNN
+F 2 "" V 4930 1100 50  0001 C CNN
+F 3 "~" H 5000 1100 50  0001 C CNN
+	1    5000 1100
+	1    0    0    -1
+$EndComp
+$Comp
+L power:+5V #PWR03
+U 1 1 6056DAE2
+P 6000 900
+F 0 "#PWR03" H 6000 750 50  0001 C CNN
+F 1 "+5V" H 6015 1073 50  0000 C CNN
+F 2 "" H 6000 900 50  0001 C CNN
+F 3 "" H 6000 900 50  0001 C CNN
+	1    6000 900
+	1    0    0    -1
+$EndComp
+$Comp
+L power:+5V #PWR01
+U 1 1 6056EF1B
+P 5000 900
+F 0 "#PWR01" H 5000 750 50  0001 C CNN
+F 1 "+5V" H 5015 1073 50  0000 C CNN
+F 2 "" H 5000 900 50  0001 C CNN
+F 3 "" H 5000 900 50  0001 C CNN
+	1    5000 900
+	1    0    0    -1
+$EndComp
+Wire Wire Line
+	5000 1250 5000 1500
+Wire Wire Line
+	6000 1300 6000 1250
+Wire Wire Line
+	5700 1500 5000 1500
+$Comp
+L Device:LED D2
+U 1 1 6056FCC6
+P 6000 1950
+F 0 "D2" V 6039 1832 50  0000 R CNN
+F 1 "LED" V 5948 1832 50  0000 R CNN
+F 2 "" H 6000 1950 50  0001 C CNN
+F 3 "~" H 6000 1950 50  0001 C CNN
+	1    6000 1950
+	0    -1   -1   0
+$EndComp
+$Comp
+L power:GND #PWR02
+U 1 1 60570E75
+P 5000 2300
+F 0 "#PWR02" H 5000 2050 50  0001 C CNN
+F 1 "GND" H 5005 2127 50  0000 C CNN
+F 2 "" H 5000 2300 50  0001 C CNN
+F 3 "" H 5000 2300 50  0001 C CNN
+	1    5000 2300
+	1    0    0    -1
+$EndComp
+$Comp
+L power:GND #PWR04
+U 1 1 60571901
+P 6000 2300
+F 0 "#PWR04" H 6000 2050 50  0001 C CNN
+F 1 "GND" H 6005 2127 50  0000 C CNN
+F 2 "" H 6000 2300 50  0001 C CNN
+F 3 "" H 6000 2300 50  0001 C CNN
+	1    6000 2300
+	1    0    0    -1
+$EndComp
+Wire Wire Line
+	5000 2300 5000 2200
+Wire Wire Line
+	6000 2300 6000 2100
+Wire Wire Line
+	6000 1800 6000 1700
+Wire Wire Line
+	6000 950  6000 900
+Wire Wire Line
+	5000 950  5000 900
+$Comp
+L Device:R R1
+U 1 1 60573240
+P 4350 1500
+F 0 "R1" V 4143 1500 50  0000 C CNN
+F 1 "1K8" V 4234 1500 50  0000 C CNN
+F 2 "" V 4280 1500 50  0001 C CNN
+F 3 "~" H 4350 1500 50  0001 C CNN
+	1    4350 1500
+	0    1    1    0
+$EndComp
+$Comp
+L led_matrix:IRLML6402TRPBF M1
+U 1 1 60573F33
+P 5950 1500
+F 0 "M1" H 6105 1454 50  0000 L CNN
+F 1 "IRLML6402TRPBF" H 6105 1545 50  0000 L CNN
+F 2 "Package_TO_SOT_SMD:SOT-23" H 7100 1500 50  0001 C CNN
+F 3 "https://www.infineon.com/dgdl/irlml6402pbf.pdf?fileId=5546d462533600a401535668d5c2263c" H 5950 1500 50  0001 C CNN
+F 4 "IRLML6402PBFTR-ND" H 7100 1500 50  0001 C CNN "DigiKey_Part_Number"
+F 5 "942-IRLML6402TRPBF" H 7100 1500 50  0001 C CNN "Mouser_Part_Number"
+F 6 "C2593" H 6250 1400 50  0001 C CNN "JLCPCB_Part_Number"
+F 7 "Infineon Technologies" H 7100 1500 50  0001 C CNN "MF"
+F 8 "IRLML6402TRPBF" H 7100 1500 50  0001 C CNN "MPN"
+F 9 "MOSFET P-CH 20V 3.7A SOT23" H 7100 1500 50  0001 C CNN "Description"
+	1    5950 1500
+	1    0    0    1
+$EndComp
+$Comp
+L pspice:DIODE D1
+U 1 1 605769EE
+P 4750 1500
+F 0 "D1" H 4750 1765 50  0000 C CNN
+F 1 "DIODE" H 4750 1674 50  0000 C CNN
+F 2 "" H 4750 1500 50  0001 C CNN
+F 3 "~" H 4750 1500 50  0001 C CNN
+	1    4750 1500
+	1    0    0    -1
+$EndComp
 $EndSCHEMATC

Commit message: RIIIIIIIIIIIIIBSSSSSS!!!!
Rib break
Parts:
- removed D1: DIODE, symbol pspice:DIODE
- removed D2: LED, symbol Device:LED
- removed M1: IRLML6402TRPBF, Package_TO_SOT_SMD:SOT-23, symbol led_matrix:IRLML6402TRPBF
- removed R1: 1K8, symbol Device:R
- removed R2: 1K, symbol Device:R
- removed R3: 120R, symbol Device:R
- added D1, D10, D100, D1000, D1001, D1002, D1003, D1004, D1005, D1006, D1007, D1008, D1009, D101, D1010, D1011, D1012, D1013, D1014, D1015, D1016, D1017, D1018, D1019, D102, D1020, D1021, D1022, D1023, D1024, D1025, D1026, D1027, D1028, D1029, D103, D1030, D1031, D1032, D1033, D104, D105, D106, D107, D108, D109, D11, D110, D111, D112, D113, D114, D115, D116, D117, D118, D119, D12, D120, D121, D122, D123, D124, D125, D126, D127, D128, D129, D13, D130, D131, D132, D133, D134, D135, D136, D137, D138, D139, D14, D140, D141, D142, D143, D144, D145, D146, D147, D148, D149, D15, D150, D151, D152, D153, D154, D155, D156, D157, D158, D159, D16, D160, D161, D162, D163, D164, D165, D166, D167, D168, D169, D17, D170, D171, D172, D173, D174, D175, D176, D177, D178, D179, D18, D180, D181, D182, D183, D184, D185, D186, D187, D188, D189, D19, D190, D191, D192, D193, D194, D195, D196, D197, D198, D199, D2, D20, D200, D201, D202, D203, D204, D205, D206, D207, D208, D209, D21, D210, D211, D212, D213, D214, D215, D216, D217, D218, D219, D22, D220, D221, D222, D223, D224, D225, D226, D227, D228, D229, D23, D230, D231, D232, D233, D234, D235, D236, D237, D238, D239, D24, D240, D241, D242, D243, D244, D245, D246, D247, D248, D249, D25, D250, D251, D252, D253, D254, D255, D256, D257, D258, D259, D26, D260, D261, D262, D263, D264, D265, D266, D267, D268, D269, D27, D270, D271, D272, D273, D274, D275, D276, D277, D278, D279, D28, D280, D281, D282, D283, D284, D285, D286, D287, D288, D289, D29, D290, D291, D292, D293, D294, D295, D296, D297, D298, D299, D3, D30, D300, D301, D302, D303, D304, D305, D306, D307, D308, D309, D31, D310, D311, D312, D313, D314, D315, D316, D317, D318, D319, D32, D320, D321, D322, D323, D324, D325, D326, D327, D328, D329, D33, D330, D331, D332, D333, D334, D335, D336, D337, D338, D339, D34, D340, D341, D342, D343, D344, D345, D346, D347, D348, D349, D35, D350, D351, D352, D353, D354, D355, D356, D357, D358, D359, D36, D360, D361, D362, D363, D364, D365, D366, D367, D368, D369, D37, D370, D371, D372, D373, D374, D375, D376, D377, D378, D379, D38, D380, D381, D382, D383, D384, D385, D386, D387, D388, D389, D39, D390, D391, D392, D393, D394, D395, D396, D397, D398, D399, D4, D40, D400, D401, D402, D403, D404, D405, D406, D407, D408, D409, D41, D410, D411, D412, D413, D414, D415, D416, D417, D418, D419, D42, D420, D421, D422, D423, D424, D425, D426, D427, D428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: LTST-S270TBKT, led_matrix:LED_LiteOn_LTST-S270TBKT, symbol led_matrix:LTST-S270TBKT
- added M1, M? (x31): IRLML0030TRPBF, Package_TO_SOT_SMD:SOT-23, symbol led_matrix:IRLML0030TRPBF
- added M? (x21): IRLML6402TRPBF, Package_TO_SOT_SMD:SOT-23, symbol led_matrix:IRLML6402TRPBF
- added M? (x21): 2N7002,215, Package_TO_SOT_SMD:SOT-23, symbol led_matrix:2N7002,215
- added R? (x21): 120R, Resistor_SMD:R_0603_1608Metric, symbol Device:R
- added R? (x21): 1K, Resistor_SMD:R_0603_1608Metric, symbol Device:R
- added R? (x53): 1K8, Resistor_SMD:R_0603_1608Metric, symbol Device:R
- added R? (x32): 470K, Resistor_SMD:R_0603_1608Metric, symbol Device:R
Connections:
- net labels removed: +5V
- wire segments 8 -> 3454

Commit message: 32x32 leds on board
Parts:
- gave numbers to parts that had none: 200
- renumbered D991 to D1000, D992 to D1001, D1025 to D1022, D1026 to D1023, D1027 to D1024, D1028 to D1025, D1029 to D1026, D1030 to D1027, D1031 to D1028, D1032 to D1029, D1033 to D1030, D1022 to D1031, D1023 to D1032, D1024 to D1033, D321 to D318, D318 to D319, D319 to D320, D320 to D321, D353 to D350, D354 to D351, D350 to D352, D351 to D353, D352 to D354, D385 to D382, D386 to D383, D387 to D384, D382 to D385, D383 to D386, D384 to D387, D417 to D414, D418 to D415, D419 to D416, D420 to D417, D414 to D418, D415 to D419, D416 to D420, D449 to D446, D450 to D447, D451 to D448, D452 to D449, D453 to D450, D446 to D451, D447 to D452, D448 to D453, D481 to D478, D482 to D479, D483 to D480, D484 to D481, D485 to D482, D486 to D483, D478 to D484, D479 to D485, D480 to D486, D513 to D510, D514 to D511, D515 to D512, D516 to D513, D517 to D514, D518 to D515, D519 to D516, D510 to D517, D511 to D518, D512 to D519, D545 to D542, D546 to D543, D547 to D544, D548 to D545, D549 to D546, D550 to D547, D551 to D548, D552 to D549, D542 to D550, D543 to D551, D544 to D552, D577 to D574, D578 to D575, D579 to D576, D580 to D577, D581 to D578, D582 to D579, D583 to D580, D584 to D581, D585 to D582, D574 to D583, D575 to D584, D576 to D585, D609 to D606, D610 to D607, D611 to D608, D612 to D609, D613 to D610, D614 to D611, D615 to D612, D616 to D613, D617 to D614, D606 to D615, D607 to D616, D608 to D617, D641 to D638, D642 to D639, D643 to D640, D644 to D641, D645 to D642, D646 to D643, D647 to D644, D648 to D645, D649 to D646, D638 to D647, D639 to D648, D640 to D649, D673 to D670, D674 to D671, D675 to D672, D676 to D673, D677 to D674, D678 to D675, D679 to D676, D680 to D677, D681 to D678, D670 to D679, D671 to D680, D672 to D681, D705 to D702, D706 to D703, D707 to D704, D708 to D705, D709 to D706, D710 to D707, D711 to D708, D712 to D709, D713 to D710, D702 to D711, D703 to D712, D704 to D713, D737 to D734, D738 to D735, D739 to D736, D740 to D737, D741 to D738, D742 to D739, D743 to D740, D744 to D741, D745 to D742, D734 to D743, D735 to D744, D736 to D745, D769 to D766, D770 to D767, D771 to D768, D772 to D769, D773 to D770, D774 to D771, D775 to D772, D776 to D773, D777 to D774, D766 to D775, D767 to D776, D768 to D777, D801 to D798, D802 to D799, D803 to D800, D804 to D801, D805 to D802, D806 to D803, D807 to D804, D808 to D805, D809 to D806, D798 to D807, D799 to D808, D800 to D809, D833 to D830, D834 to D831, D835 to D832, D836 to D833, D837 to D834, D838 to D835, D839 to D836, D840 to D837, D841 to D838, D830 to D839, D831 to D840, D832 to D841, D865 to D862, D866 to D863, D867 to D864, D868 to D865, D869 to D866, D870 to D867, D871 to D868, D872 to D869, D873 to D870, D862 to D871, D863 to D872, D864 to D873, D897 to D894, D898 to D895, D899 to D896, D900 to D897, D901 to D898, D902 to D899, D903 to D900, D904 to D901, D905 to D902, D894 to D903, D895 to D904, D896 to D905, D929 to D926, D930 to D927, D931 to D928, D932 to D929, D933 to D930, D934 to D931, D935 to D932, D936 to D933, D937 to D934, D926 to D935, D927 to D936, D928 to D937, D961 to D958, D962 to D959, D963 to D960, D964 to D961, D965 to D962, D966 to D963, D967 to D964, D968 to D965, D969 to D966, D958 to D967, D959 to D968, D960 to D969, D993 to D990, D994 to D991, D995 to D992, D996 to D993, D997 to D994, D998 to D995, D999 to D996, D1000 to D997, D1001 to D998, D990 to D999, M1 to M43

Commit message: led matrix schematic page completed
Parts:
- removed M1, M15, M16, M17, M18, M19, M2, M20, M21, M29, M3, M30, M31, M32, M33, M34, M35, M4, M5, M6, M7: 2N7002,215, Package_TO_SOT_SMD:SOT-23, symbol led_matrix:2N7002,215
- removed M10, M11, M12, M13, M14, M22, M23, M24, M25, M26, M27, M28, M36, M37, M38, M39, M40, M41, M42, M8, M9: IRLML6402TRPBF, Package_TO_SOT_SMD:SOT-23, symbol led_matrix:IRLML6402TRPBF
- removed M43, M44, M45, M46, M47, M48, M49, M50, M51, M52, M53, M54, M55, M56, M57, M58, M59, M60, M61, M62, M63, M64, M65, M66, M67, M68, M69, M70, M71, M72, M73, M74: IRLML0030TRPBF, Package_TO_SOT_SMD:SOT-23, symbol led_matrix:IRLML0030TRPBF
- removed R1, R100, R102, R104, R106, R108, R110, R112, R114, R116, R118, R120, R122, R124, R126, R2, R22, R23, R24, R25, R26, R27, R28, R3, R4, R43, R44, R45, R46, R47, R48, R49, R5, R57, R6, R66, R68, R7, R70, R72, R74, R76, R78, R80, R82, R84, R86, R88, R90, R92, R94, R96, R98: 1K8, Resistor_SMD:R_0603_1608Metric, symbol Device:R
- removed R10, R11, R12, R13, R14, R29, R30, R31, R32, R33, R34, R35, R50, R51, R52, R53, R54, R55, R56, R8, R9: 1K, Resistor_SMD:R_0603_1608Metric, symbol Device:R
- removed R101, R103, R105, R107, R109, R111, R113, R115, R117, R119, R121, R123, R125, R127, R65, R67, R69, R71, R73, R75, R77, R79, R81, R83, R85, R87, R89, R91, R93, R95, R97, R99: 470K, Resistor_SMD:R_0603_1608Metric, symbol Device:R
- removed R15, R16, R17, R18, R19, R20, R21, R36, R37, R38, R39, R40, R41, R42, R58, R59, R60, R61, R62, R63, R64: 120R, Resistor_SMD:R_0603_1608Metric, symbol Device:R
Connections:
- net sheetA575BE9A/ANODES: now reaches D1031.A, D126.A, D158.A, D190.A, D222.A, D254.A, D286.A, D30.A, D319.A, D352.A, D385.A, D418.A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
- net common cathode/CATHODES: now reaches D1.C, D10.C, D11.C, D12.C, D13.C, D14.C, D15.C, D16.C, D17.C, D18.C, D19.C, D2.C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
- net sheetA575BE9B/ANODES: now reaches D1000.A, D1032.A, D127.A, D159.A, D191.A, D223.A, D255.A, D287.A, D31.A, D320.A, D353.A, D386.A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
- net sheetA575BE9C/ANODES: now reaches D1001.A, D1033.A, D128.A, D160.A, D192.A, D224.A, D256.A, D288.A, D289.A, D32.A, D321.A, D322.A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
- net sheetD7D8B720/CATHODES: now reaches D33.C, D34.C, D35.C, D36.C, D37.C, D38.C, D39.C, D40.C, D41.C, D42.C, D43.C, D44.C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
- net sheetD89BE98B/CATHODES: now reaches D65.C, D66.C, D67.C, D68.C, D69.C, D70.C, D71.C, D72.C, D73.C, D74.C, D75.C, D76.C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
- net sheetD89BE98C/CATHODES: now reaches D100.C, D101.C, D102.C, D103.C, D104.C, D105.C, D106.C, D107.C, D108.C, D109.C, D110.C, D111.C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
- net sheetD95F2321/CATHODES: now reaches D129.C, D130.C, D131.C, D132.C, D133.C, D134.C, D135.C, D136.C, D137.C, D138.C, D139.C, D140.C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
- net sheetD95F2322/CATHODES: now reaches D161.C, D162.C, D163.C, D164.C, D165.C, D166.C, D167.C, D168.C, D169.C, D170.C, D171.C, D172.C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
- net sheetD95F2323/CATHODES: now reaches D193.C, D194.C, D195.C, D196.C, D197.C, D198.C, D199.C, D200.C, D201.C, D202.C, D203.C, D204.C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
- net sheetD95F2324/CATHODES: now reaches D225.C, D226.C, D227.C, D228.C, D229.C, D230.C, D231.C, D232.C, D233.C, D234.C, D235.C, D236.C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
- net sheetDA22614D/CATHODES: now reaches D257.C, D258.C, D259.C, D260.C, D261.C, D262.C, D263.C, D264.C, D265.C, D266.C, D267.C, D268.C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
- net sheetDA22614E/CATHODES: now reaches D290.C, D291.C, D292.C, D293.C, D294.C, D295.C, D296.C, D297.C, D298.C, D299.C, D300.C, D301.C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
- net sheetDA22614F/CATHODES: now reaches D323.C, D324.C, D325.C, D326.C, D327.C, D328.C, D329.C, D330.C, D331.C, D332.C, D333.C, D334.C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
- net sheetDA226150/CATHODES: now reaches D356.C, D357.C, D358.C, D359.C, D360.C, D361.C, D362.C, D363.C, D364.C, D365.C, D366.C, D367.C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
- net sheetDA226151/CATHODES: now reaches D389.C, D390.C, D391.C, D392.C, D393.C, D394.C, D395.C, D396.C, D397.C, D398.C, D399.C, D400.C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
- net sheetDA226152/CATHODES: now reaches D422.C, D423.C, D424.C, D425.C, D426.C, D427.C, D428.C, D429.C, D430.C, D431.C, D432.C, D433.C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
- net sheetDA226153/CATHODES: now reaches D455.C, D456.C, D457.C, D458.C, D459.C, D460.C, D461.C, D462.C, D463.C, D464.C, D465.C, D466.C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
- net sheetDA226154/CATHODES: now reaches D488.C, D489.C, D490.C, D491.C, D492.C, D493.C, D494.C, D495.C, D496.C, D497.C, D498.C, D499.C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
- net sheetDAE5EEF6/CATHODES: now reaches D521.C, D522.C, D523.C, D524.C, D525.C, D526.C, D527.C, D528.C, D529.C, D530.C, D531.C, D532.C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
- net sheetDAE5EEF7/CATHODES: now reaches D554.C, D555.C, D556.C, D557.C, D558.C, D559.C, D560.C, D561.C, D562.C, D563.C, D564.C, D565.C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
- net sheetDAE5EEF8/CATHODES: now reaches D586.C, D587.C, D588.C, D589.C, D590.C, D591.C, D592.C, D593.C, D594.C, D595.C, D596.C, D597.C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
- net sheetDAE5EEF9/CATHODES: now reaches D618.C, D619.C, D620.C, D621.C, D622.C, D623.C, D624.C, D625.C, D626.C, D627.C, D628.C, D629.C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
- net sheetDAE5EEFA/CATHODES: now reaches D650.C, D651.C, D652.C, D653.C, D654.C, D655.C, D656.C, D657.C, D658.C, D659.C, D660.C, D661.C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
- net sheetDAE5EEFB/CATHODES: now reaches D682.C, D683.C, D684.C, D685.C, D686.C, D687.C, D688.C, D689.C, D690.C, D691.C, D692.C, D693.C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
- net sheetDAE5EEFC/CATHODES: now reaches D714.C, D715.C, D716.C, D717.C, D718.C, D719.C, D720.C, D721.C, D722.C, D723.C, D724.C, D725.C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
- net sheetDAE5EEFD/CATHODES: now reaches D746.C, D747.C, D748.C, D749.C, D750.C, D751.C, D752.C, D753.C, D754.C, D755.C, D756.C, D757.C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
- net sheetDAE5EEFE/CATHODES: now reaches D778.C, D779.C, D780.C, D781.C, D782.C, D783.C, D784.C, D785.C, D786.C, D787.C, D788.C, D789.C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
- net sheetDAE5EEFF/CATHODES: now reaches D810.C, D811.C, D812.C, D813.C, D814.C, D815.C, D816.C, D817.C, D818.C, D819.C, D820.C, D821.C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
- net sheetDAE5EF00/CATHODES: now reaches D842.C, D843.C, D844.C, D845.C, D846.C, D847.C, D848.C, D849.C, D850.C, D851.C, D852.C, D853.C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
- net sheetDAE5EF01/CATHODES: now reaches D874.C, D875.C, D876.C, D877.C, D878.C, D879.C, D880.C, D881.C, D882.C, D883.C, D884.C, D885.C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
- net sheetDAE5EF02/CATHODES: now reaches D906.C, D907.C, D908.C, D909.C, D910.C, D911.C, D912.C, D913.C, D914.C, D915.C, D916.C, D917.C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
- net sheetDAE5EF03/CATHODES: now reaches D938.C, D939.C, D940.C, D941.C, D942.C, D943.C, D944.C, D945.C, D946.C, D947.C, D948.C, D949.C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
- net sheetDAE5EF04/CATHODES: now reaches D1000.C, D1001.C, D970.C, D971.C, D972.C, D973.C, D974.C, D975.C, D976.C, D977.C, D978.C, D979.C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
- net sheetDAE5EF05/CATHODES: now reaches D1002.C, D1003.C, D1004.C, D1005.C, D1006.C, D1007.C, D1008.C, D1009.C, D1010.C, D1011.C, D1012.C, D1013.C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
- net sheetA575BE97/ANODES: now reaches D1028.A, D123.A, D155.A, D187.A, D219.A, D251.A, D27.A, D283.A, D316.A, D349.A, D382.A, D415.A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
- net sheetA575BE98/ANODES: now reaches D1029.A, D124.A, D156.A, D188.A, D220.A, D252.A, D28.A, D284.A, D317.A, D350.A, D383.A, D416.A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
- net sheetA575BE99/ANODES: now reaches D1030.A, D125.A, D157.A, D189.A, D221.A, D253.A, D285.A, D29.A, D318.A, D351.A, D384.A, D417.A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
- net sheetA575BE94/ANODES: now reaches D1025.A, D120.A, D152.A, D184.A, D216.A, D24.A, D248.A, D280.A, D313.A, D346.A, D379.A, D412.A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
- net sheetA575BE95/ANODES: now reaches D1026.A, D121.A, D153.A, D185.A, D217.A, D249.A, D25.A, D281.A, D314.A, D347.A, D380.A, D413.A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
- net sheetA575BE96/ANODES: now reaches D1027.A, D122.A, D154.A, D186.A, D218.A, D250.A, D26.A, D282.A, D315.A, D348.A, D381.A, D414.A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
- net sheetA575BE91/ANODES: now reaches D1022.A, D117.A, D149.A, D181.A, D21.A, D213.A, D245.A, D277.A, D310.A, D343.A, D376.A, D409.A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
- net sheetA575BE92/ANODES: now reaches D1023.A, D118.A, D150.A, D182.A, D214.A, D22.A, D246.A, D278.A, D311.A, D344.A, D377.A, D410.A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
- net sheetA575BE93/ANODES: now reaches D1024.A, D119.A, D151.A, D183.A, D215.A, D23.A, D247.A, D279.A, D312.A, D345.A, D378.A, D411.A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
- net sheetA575BE8E/ANODES: now reaches D1019.A, D114.A, D146.A, D178.A, D18.A, D210.A, D242.A, D274.A, D307.A, D340.A, D373.A, D406.A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
- net sheetA575BE8F/ANODES: now reaches D1020.A, D115.A, D147.A, D179.A, D19.A, D211.A, D243.A, D275.A, D308.A, D341.A, D374.A, D407.A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
- net sheetA575BE90/ANODES: now reaches D1021.A, D116.A, D148.A, D180.A, D20.A, D212.A, D244.A, D276.A, D309.A, D342.A, D375.A, D408.A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
- net sheetA575BE8D/ANODES: now reaches D1018.A, D113.A, D145.A, D17.A, D177.A, D209.A, D241.A, D273.A, D306.A, D339.A, D372.A, D405.A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
- net sheetA4B98B8B/ANODES: now reaches D1015.A, D110.A, D14.A, D142.A, D174.A, D206.A, D238.A, D270.A, D303.A, D336.A, D369.A, D402.A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
- net sheetA4B98B8C/ANODES: now reaches D1016.A, D111.A, D143.A, D15.A, D175.A, D207.A, D239.A, D271.A, D304.A, D337.A, D370.A, D403.A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
- net sheetA4B98B8D/ANODES: now reaches D1017.A, D112.A, D144.A, D16.A, D176.A, D208.A, D240.A, D272.A, D305.A, D338.A, D371.A, D404.A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
- net sheetA4B98B88/ANODES: now reaches D1012.A, D107.A, D11.A, D139.A, D171.A, D203.A, D235.A, D267.A, D300.A, D333.A, D366.A, D399.A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
- net sheetA4B98B89/ANODES: now reaches D1013.A, D108.A, D12.A, D140.A, D172.A, D204.A, D236.A, D268.A, D301.A, D334.A, D367.A, D400.A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
- net sheetA4B98B8A/ANODES: now reaches D1014.A, D109.A, D13.A, D141.A, D173.A, D205.A, D237.A, D269.A, D302.A, D335.A, D368.A, D401.A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
- net sheetA3FD3BF8/ANODES: now reaches D1009.A, D104.A, D136.A, D168.A, D200.A, D232.A, D264.A, D297.A, D330.A, D363.A, D396.A, D40.A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
- net sheetA4B98B86/ANODES: now reaches D1010.A, D105.A, D137.A, D169.A, D201.A, D233.A, D265.A, D298.A, D331.A, D364.A, D397.A, D41.A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
- net sheetA4B98B87/ANODES: now reaches D10.A, D1011.A, D106.A, D138.A, D170.A, D202.A, D234.A, D266.A, D299.A, D332.A, D365.A, D398.A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
- net sheetA341C37F/ANODES: now reaches D1006.A, D101.A, D133.A, D165.A, D197.A, D229.A, D261.A, D294.A, D327.A, D360.A, D37.A, D393.A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
- net sheetA341C380/ANODES: now reaches D1007.A, D102.A, D134.A, D166.A, D198.A, D230.A, D262.A, D295.A, D328.A, D361.A, D38.A, D394.A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
- net sheetA3FD3BF7/ANODES: now reaches D1008.A, D103.A, D135.A, D167.A, D199.A, D231.A, D263.A, D296.A, D329.A, D362.A, D39.A, D395.A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
- net sheet9E2197FD/ANODES: now reaches D1003.A, D130.A, D162.A, D194.A, D2.A, D226.A, D258.A, D291.A, D324.A, D34.A, D357.A, D390.A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
- net sheetA10E8493/ANODES: now reaches D1004.A, D131.A, D163.A, D195.A, D227.A, D259.A, D292.A, D3.A, D325.A, D35.A, D358.A, D391.A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
- net sheetA10E8494/ANODES: now reaches D100.A, D1005.A, D132.A, D164.A, D196.A, D228.A, D260.A, D293.A, D326.A, D359.A, D36.A, D392.A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
- net common anode/ANODES: now reaches D1.A, D1002.A, D129.A, D161.A, D193.A, D225.A, D257.A, D290.A, D323.A, D33.A, D356.A, D389.A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
Other:
- note added: "LED Matrix"
- moved on the sheet: D1, D10, D100, D1000, D1001, D1002, D1003, D1004, D1005, D1006, D1007, D1008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

Commit message: mcu progress sync to pcb
Other:
- moved on the sheet: D1, D10, D100, D1000, D1001, D1002, D1003, D1004, D1005, D1006, D1007, D1008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

Commit message: layouting update
Parts:
- removed D288, D321, D354, D387, D420, D453, D486, D519, D552: LTST-S270TBKT, led_matrix:LED_LiteOn_LTST-S270TBKT, symbol led_matrix:LTST-S270TBKT
- renumbered D290 to D10, D256 to D1000, D289 to D1001, D322 to D1002, D355 to D1003, D388 to D1004, D421 to D1005, D454 to D1006, D487 to D1007, D520 to D1008, D553 to D1009, D132 to D101, D585 to D1010, D617 to D1011, D649 to D1012, D681 to D1013, D713 to D1014, D745 to D1015, D777 to D1016, D809 to D1017, D841 to D1018, D873 to D1019, D164 to D102, D905 to D1020, D937 to D1021, D969 to D1022, D1001 to D1023, D1033 to D1024, D196 to D103, D228 to D104, D260 to D105, D293 to D106, D326 to D107, D359 to D108, D392 to D109, D323 to D11, D425 to D110, D458 to D111, D491 to D112, D524 to D113, D557 to D114, D589 to D115, D621 to D116, D653 to D117, D685 to D118, D717 to D119, D356 to D12, D749 to D120, D781 to D121, D813 to D122, D845 to D123, D877 to D124, D909 to D125, D941 to D126, D973 to D127, D1005 to D128, D5 to D129, D389 to D13, D37 to D130, D69 to D131, D101 to D132, D165 to D134, D197 to D135, D229 to D136, D261 to D137, D294 to D138, D327 to D139, D422 to D14, D360 to D140, D393 to D141, D426 to D142, D459 to D143, D492 to D144, D525 to D145, D558 to D146, D590 to D147, D622 to D148, D654 to D149, D455 to D15, D686 to D150, D718 to D151, D750 to D152, D782 to D153, D814 to D154, D846 to D155, D878 to D156, D910 to D157, D942 to D158, D974 to D159, D488 to D16, D1006 to D160, D6 to D161, D38 to D162, D70 to D163, D102 to D164, D134 to D165, D198 to D167, D230 to D168, D262 to D169, D521 to D17, D295 to D170, D328 to D171, D361 to D172, D394 to D173, D427 to D174, D460 to D175, D493 to D176, D526 to D177, D559 to D178, D591 to D179, D554 to D18, D623 to D180, D655 to D181, D687 to D182, D719 to D183, D751 to D184, D783 to D185, D815 to D186, D847 to D187, D879 to D188, D911 to D189, D586 to D19, D943 to D190, D975 to D191, D1007 to D192, D7 to D193, D39 to D194, D71 to D195, D103 to D196, D135 to D197, D167 to D198, D33 to D2, D618 to D20, D231 to D200, D263 to D201, D296 to D202, D329 to D203, D362 to D204, D395 to D205, D428 to D206, D461 to D207, D494 to D208, D527 to D209, D650 to D21, D560 to D210, D592 to D211, D624 to D212, D656 to D213, D688 to D214, D720 to D215, D752 to D216, D784 to D217, D816 to D218, D848 to D219, D682 to D22, D880 to D220, D912 to D221, D944 to D222, D976 to D223, D1008 to D224, D8 to D225, D40 to D226, D72 to D227, D104 to D228, D136 to D229, D714 to D23, D168 to D230, D200 to D231, D264 to D233, D297 to D234, D330 to D235, D363 to D236, D396 to D237, D429 to D238, D462 to D239, D746 to D24, D495 to D240, D528 to D241, D561 to D242, D593 to D243, D625 to D244, D657 to D245, D689 to D246, D721 to D247, D753 to D248, D785 to D249, D778 to D25, D817 to D250, D849 to D251, D881 to D252, D913 to D253, D945 to D254, D977 to D255, D1009 to D256, D9 to D257, D41 to D258, D73 to D259, D810 to D26, D105 to D260, D137 to D261, D169 to D262, D201 to D263, D233 to D264, D298 to D266, D331 to D267, D364 to D268, D397 to D269, D842 to D27, D430 to D270, D463 to D271, D496 to D272, D529 to D273, D562 to D274, D594 to D275, D626 to D276, D658 to D277, D690 to D278, D722 to D279, D874 to D28, D754 to D280, D786 to D281, D818 to D282, D850 to D283, D882 to D284, D914 to D285, D946 to D286, D978 to D287, D1010 to D288, D10 to D289, D906 to D29, D42 to D290, D74 to D291, D106 to D292, D138 to D293, D170 to D294, D202 to D295, D234 to D296, D266 to D297, D299 to D298, D332 to D299, D65 to D3, D938 to D30, D365 to D300, D398 to D301, D431 to D302, D464 to D303, D497 to D304, D530 to D305, D563 to D306, D595 to D307, D627 to D308, D659 to D309, D970 to D31, D691 to D310, D723 to D311, D755 to D312, D787 to D313, D819 to D314, D851 to D315, D883 to D316, D915 to D317, D947 to D318, D979 to D319, D1002 to D32, D1011 to D320, D11 to D321, D43 to D322, D75 to D323, D107 to D324, D139 to D325, D171 to D326, D203 to D327, D235 to D328, D267 to D329, D2 to D33, D300 to D330, D333 to D331, D366 to D332, D399 to D333, D432 to D334, D465 to D335, D498 to D336, D531 to D337, D564 to D338, D596 to D339, D628 to D340, D660 to D341, D692 to D342, D724 to D343, D756 to D344, D788 to D345, D820 to D346, D852 to D347, D884 to D348, D916 to D349, D66 to D35, D948 to D350, D980 to D351, D1012 to D352, D12 to D353, D44 to D354, D76 to D355, D108 to D356, D140 to D357, D172 to D358, D204 to D359, D98 to D36, D236 to D360, D268 to D361, D301 to D362, D334 to D363, D367 to D364, D400 to D365, D433 to D366, D466 to D367, D499 to D368, D532 to D369, D130 to D37, D565 to D370, D597 to D371, D629 to D372, D661 to D373, D693 to D374, D725 to D375, D757 to D376, D789 to D377, D821 to D378, D853 to D379, D162 to D38, D885 to D380, D917 to D381, D949 to D382, D981 to D383, D1013 to D384, D13 to D385, D45 to D386, D77 to D387, D109 to D388, D141 to D389, D194 to D39, D173 to D390, D205 to D391, D237 to D392, D269 to D393, D302 to D394, D335 to D395, D368 to D396, D401 to D397, D434 to D398, D467 to D399, D97 to D4, D226 to D40, D500 to D400, D533 to D401, D566 to D402, D598 to D403, D630 to D404, D662 to D405, D694 to D406, D726 to D407, D758 to D408, D790 to D409, D258 to D41, D822 to D410, D854 to D411, D886 to D412, D918 to D413, D950 to D414, D982 to D415, D1014 to D416, D14 to D417, D46 to D418, D78 to D419, D291 to D42, D110 to D420, D142 to D421, D174 to D422, D206 to D423, D238 to D424, D270 to D425, D303 to D426, D336 to D427, D369 to D428, D402 to D429, D324 to D43, D435 to D430, D468 to D431, D501 to D432, D534 to D433, D567 to D434, D599 to D435, D631 to D436, D663 to D437, D695 to D438, D727 to D439, D357 to D44, D759 to D440, D791 to D441, D823 to D442, D855 to D443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

Commit message: pcb format refactor
Parts:
- renumbered D9 to D10, D99 to D100, D999 to D1000, D1000 to D1001, D1001 to D1002, D1002 to D1003, D1003 to D1004, D1004 to D1005, D1005 to D1006, D1006 to D1007, D1007 to D1008, D1008 to D1009, D100 to D101, D1009 to D1010, D1010 to D1011, D1011 to D1012, D1012 to D1013, D1013 to D1014, D1014 to D1015, D1015 to D1016, D1016 to D1017, D1017 to D1018, D1018 to D1019, D101 to D102, D1019 to D1020, D1020 to D1021, D1021 to D1022, D1022 to D1023, D1023 to D1024, D1024 to D1025, D102 to D103, D103 to D104, D104 to D105, D105 to D106, D106 to D107, D107 to D108, D108 to D109, D10 to D11, D109 to D110, D110 to D111, D111 to D112, D112 to D113, D113 to D114, D114 to D115, D115 to D116, D116 to D117, D117 to D118, D118 to D119, D11 to D12, D119 to D120, D120 to D121, D121 to D122, D122 to D123, D123 to D124, D124 to D125, D125 to D126, D126 to D127, D127 to D128, D128 to D129, D12 to D13, D129 to D130, D130 to D131, D131 to D132, D132 to D133, D133 to D134, D134 to D135, D135 to D136, D136 to D137, D137 to D138, D138 to D139, D13 to D14, D139 to D140, D140 to D141, D141 to D142, D142 to D143, D143 to D144, D144 to D145, D145 to D146, D146 to D147, D147 to D148, D148 to D149, D14 to D15, D149 to D150, D150 to D151, D151 to D152, D152 to D153, D153 to D154, D154 to D155, D155 to D156, D156 to D157, D157 to D158, D158 to D159, D15 to D16, D159 to D160, D160 to D161, D161 to D162, D162 to D163, D163 to D164, D164 to D165, D165 to D166, D166 to D167, D167 to D168, D168 to D169, D16 to D17, D169 to D170, D170 to D171, D171 to D172, D172 to D173, D173 to D174, D174 to D175, D175 to D176, D176 to D177, D177 to D178, D178 to D179, D17 to D18, D179 to D180, D180 to D181, D181 to D182, D182 to D183, D183 to D184, D184 to D185, D185 to D186, D186 to D187, D187 to D188, D188 to D189, D18 to D19, D189 to D190, D190 to D191, D191 to D192, D192 to D193, D193 to D194, D194 to D195, D195 to D196, D196 to D197, D197 to D198, D198 to D199, D1 to D2, D19 to D20, D199 to D200, D200 to D201, D201 to D202, D202 to D203, D203 to D204, D204 to D205, D205 to D206, D206 to D207, D207 to D208, D208 to D209, D20 to D21, D209 to D210, D210 to D211, D211 to D212, D212 to D213, D213 to D214, D214 to D215, D215 to D216, D216 to D217, D217 to D218, D218 to D219, D21 to D22, D219 to D220, D220 to D221, D221 to D222, D222 to D223, D223 to D224, D224 to D225, D225 to D226, D226 to D227, D227 to D228, D228 to D229, D22 to D23, D229 to D230, D230 to D231, D231 to D232, D232 to D233, D233 to D234, D234 to D235, D235 to D236, D236 to D237, D237 to D238, D238 to D239, D23 to D24, D239 to D240, D240 to D241, D241 to D242, D242 to D243, D243 to D244, D244 to D245, D245 to D246, D246 to D247, D247 to D248, D248 to D249, D24 to D25, D249 to D250, D250 to D251, D251 to D252, D252 to D253, D253 to D254, D254 to D255, D255 to D256, D256 to D257, D257 to D258, D258 to D259, D25 to D26, D259 to D260, D260 to D261, D261 to D262, D262 to D263, D263 to D264, D264 to D265, D265 to D266, D266 to D267, D267 to D268, D268 to D269, D26 to D27, D269 to D270, D270 to D271, D271 to D272, D272 to D273, D273 to D274, D274 to D275, D275 to D276, D276 to D277, D277 to D278, D278 to D279, D27 to D28, D279 to D280, D280 to D281, D281 to D282, D282 to D283, D283 to D284, D284 to D285, D285 to D286, D286 to D287, D287 to D288, D288 to D289, D28 to D29, D289 to D290, D290 to D291, D291 to D292, D292 to D293, D293 to D294, D294 to D295, D295 to D296, D296 to D297, D297 to D298, D298 to D299, D2 to D3, D29 to D30, D299 to D300, D300 to D301, D301 to D302, D302 to D303, D303 to D304, D304 to D305, D305 to D306, D306 to D307, D307 to D308, D308 to D309, D30 to D31, D309 to D310, D310 to D311, D311 to D312, D312 to D313, D313 to D314, D314 to D315, D315 to D316, D316 to D317, D317 to D318, D318 to D319, D31 to D32, D319 to D320, D320 to D321, D321 to D322, D322 to D323, D323 to D324, D324 to D325, D325 to D326, D326 to D327, D327 to D328, D328 to D329, D32 to D33, D329 to D330, D330 to D331, D331 to D332, D332 to D333, D333 to D334, D334 to D335, D335 to D336, D336 to D337, D337 to D338, D338 to D339, D33 to D34, D339 to D340, D340 to D341, D341 to D342, D342 to D343, D343 to D344, D344 to D345, D345 to D346, D346 to D347, D347 to D348, D348 to D349, D34 to D35, D349 to D350, D350 to D351, D351 to D352, D352 to D353, D353 to D354, D354 to D355, D355 to D356, D356 to D357, D357 to D358, D358 to D359, D35 to D36, D359 to D360, D360 to D361, D361 to D362, D362 to D363, D363 to D364, D364 to D365, D365 to D366, D366 to D367, D367 to D368, D368 to D369, D36 to D37, D369 to D370, D370 to D371, D371 to D372, D372 to D373, D373 to D374, D374 to D375, D375 to D376, D376 to D377, D377 to D378, D378 to D379, D37 to D38, D379 to D380, D380 to D381, D381 to D382, D382 to D383, D383 to D384, D384 to D385, D385 to D386, D386 to D387, D387 to D388, D388 to D389, D38 to D39, D389 to D390, D390 to D391, D391 to D392, D392 to D393, D393 to D394, D394 to D395, D395 to D396, D396 to D397, D397 to D398, D398 to D399, D3 to D4, D39 to D40, D399 to D400, D400 to D401, D401 to D402, D402 to D403, D403 to D404, D404 to D405, D405 to D406, D406 to D407, D407 to D408, D408 to D409, D40 to D41, D409 to D410, D410 to D411, D411 to D412, D412 to D413, D413 to D414, D414 to D415, D415 to D416, D416 to D417, D417 to D418, D418 to D419, D41 to D42, D419 to D420, D420 to D421, D421 to D422, D422 to D423, D423 to D424, D424 to D425, D425 to D426, D426 to D427, D427 to D428, D428 to D429, D42 to D43, D429 to D430, D430 to D431, D431 to D432, D432 to D433, D433 to D434, D434 to D435, D435 to D436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
