File: hard/leds.sch (KiCad schematic (older format))
At the start: 1024 parts

Commit message: attribute naming update
JLCPCB_Part_Number -> LCSC
DigiKey_Part_Number -> DigiKey
Mouser_Part_Number -> Mouser
Parts:
- D10, D100, D1000, D1001, D1002, D1003, D1004, D1005, D1006, D1007, D1008, D1009, D101, D1010, D1011, D1012, D1013, D1014, D1015, D1016, D1017, D1018, D1019, D102, D1020, D1021, D1022, D1023, D1024, D1025, D103, D104, D105, D106, D107, D108, D109, D11, D110, D111, D112, D113, D114, D115, D116, D117, D118, D119, D12, D120, D121, D122, D123, D124, D125, D126, D127, D128, D129, D13, D130, D131, D132, D133, D134, D135, D136, D137, D138, D139, D14, D140, D141, D142, D143, D144, D145, D146, D147, D148, D149, D15, D150, D151, D152, D153, D154, D155, D156, D157, D158, D159, D16, D160, D161, D162, D163, D164, D165, D166, D167, D168, D169, D17, D170, D171, D172, D173, D174, D175, D176, D177, D178, D179, D18, D180, D181, D182, D183, D184, D185, D186, D187, D188, D189, D19, D190, D191, D192, D193, D194, D195, D196, D197, D198, D199, D2, D20, D200, D201, D202, D203, D204, D205, D206, D207, D208, D209, D21, D210, D211, D212, D213, D214, D215, D216, D217, D218, D219, D22, D220, D221, D222, D223, D224, D225, D226, D227, D228, D229, D23, D230, D231, D232, D233, D234, D235, D236, D237, D238, D239, D24, D240, D241, D242, D243, D244, D245, D246, D247, D248, D249, D25, D250, D251, D252, D253, D254, D255, D256, D257, D258, D259, D26, D260, D261, D262, D263, D264, D265, D266, D267, D268, D269, D27, D270, D271, D272, D273, D274, D275, D276, D277, D278, D279, D28, D280, D281, D282, D283, D284, D285, D286, D287, D288, D289, D29, D290, D291, D292, D293, D294, D295, D296, D297, D298, D299, D3, D30, D300, D301, D302, D303, D304, D305, D306, D307, D308, D309, D31, D310, D311, D312, D313, D314, D315, D316, D317, D318, D319, D32, D320, D321, D322, D323, D324, D325, D326, D327, D328, D329, D33, D330, D331, D332, D333, D334, D335, D336, D337, D338, D339, D34, D340, D341, D342, D343, D344, D345, D346, D347, D348, D349, D35, D350, D351, D352, D353, D354, D355, D356, D357, D358, D359, D36, D360, D361, D362, D363, D364, D365, D366, D367, D368, D369, D37, D370, D371, D372, D373, D374, D375, D376, D377, D378, D379, D38, D380, D381, D382, D383, D384, D385, D386, D387, D388, D389, D39, D390, D391, D392, D393, D394, D395, D396, D397, D398, D399, D4, D40, D400, D401, D402, D403, D404, D405, D406, D407, D408, D409, D41, D410, D411, D412, D413, D414, D415, D416, D417, D418, D419, D42, D420, D421, D422, D423, D424, D425, D426, D427, D428, D429, D43, D430, D431, D432, D433, D434, D435, D436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: DigiKey (none) -> LTST-S270TBKT-5A-ND; DigiKey_Part_Number LTST-S270TBKT-5A-ND -> (none); JLCPCB_Part_Number C125115 -> (none); LCSC (none) -> C125115; Mouser (none) -> 859-LTST-S270TBKT; Mouser_Part_Number 859-LTST-S270TBKT -> (none)

Commit message: re-connect footprints
Parts:
- renumbered D2 to D1, D11 to D10, D101 to D100, D1001 to D1000, D1002 to D1001, D1003 to D1002, D1004 to D1003, D1005 to D1004, D1006 to D1005, D1007 to D1006, D1008 to D1007, D1009 to D1008, D1010 to D1009, D102 to D101, D1011 to D1010, D1012 to D1011, D1013 to D1012, D1014 to D1013, D1015 to D1014, D1016 to D1015, D1017 to D1016, D1018 to D1017, D1019 to D1018, D1020 to D1019, D103 to D102, D1021 to D1020, D1022 to D1021, D1023 to D1022, D1024 to D1023, D1025 to D1024, D104 to D103, D105 to D104, D106 to D105, D107 to D106, D108 to D107, D109 to D108, D110 to D109, D12 to D11, D111 to D110, D112 to D111, D113 to D112, D114 to D113, D115 to D114, D116 to D115, D117 to D116, D118 to D117, D119 to D118, D120 to D119, D13 to D12, D121 to D120, D122 to D121, D123 to D122, D124 to D123, D125 to D124, D126 to D125, D127 to D126, D128 to D127, D129 to D128, D130 to D129, D14 to D13, D131 to D130, D132 to D131, D133 to D132, D134 to D133, D135 to D134, D136 to D135, D137 to D136, D138 to D137, D139 to D138, D140 to D139, D15 to D14, D141 to D140, D142 to D141, D143 to D142, D144 to D143, D145 to D144, D146 to D145, D147 to D146, D148 to D147, D149 to D148, D150 to D149, D16 to D15, D151 to D150, D152 to D151, D153 to D152, D154 to D153, D155 to D154, D156 to D155, D157 to D156, D158 to D157, D159 to D158, D160 to D159, D17 to D16, D161 to D160, D162 to D161, D163 to D162, D164 to D163, D165 to D164, D166 to D165, D167 to D166, D168 to D167, D169 to D168, D170 to D169, D18 to D17, D171 to D170, D172 to D171, D173 to D172, D174 to D173, D175 to D174, D176 to D175, D177 to D176, D178 to D177, D179 to D178, D180 to D179, D19 to D18, D181 to D180, D182 to D181, D183 to D182, D184 to D183, D185 to D184, D186 to D185, D187 to D186, D188 to D187, D189 to D188, D190 to D189, D20 to D19, D191 to D190, D192 to D191, D193 to D192, D194 to D193, D195 to D194, D196 to D195, D197 to D196, D198 to D197, D199 to D198, D200 to D199, D3 to D2, D21 to D20, D201 to D200, D202 to D201, D203 to D202, D204 to D203, D205 to D204, D206 to D205, D207 to D206, D208 to D207, D209 to D208, D210 to D209, D22 to D21, D211 to D210, D212 to D211, D213 to D212, D214 to D213, D215 to D214, D216 to D215, D217 to D216, D218 to D217, D219 to D218, D220 to D219, D23 to D22, D221 to D220, D222 to D221, D223 to D222, D224 to D223, D225 to D224, D226 to D225, D227 to D226, D228 to D227, D229 to D228, D230 to D229, D24 to D23, D231 to D230, D232 to D231, D233 to D232, D234 to D233, D235 to D234, D236 to D235, D237 to D236, D238 to D237, D239 to D238, D240 to D239, D25 to D24, D241 to D240, D242 to D241, D243 to D242, D244 to D243, D245 to D244, D246 to D245, D247 to D246, D248 to D247, D249 to D248, D250 to D249, D26 to D25, D251 to D250, D252 to D251, D253 to D252, D254 to D253, D255 to D254, D256 to D255, D257 to D256, D258 to D257, D259 to D258, D260 to D259, D27 to D26, D261 to D260, D262 to D261, D263 to D262, D264 to D263, D265 to D264, D266 to D265, D267 to D266, D268 to D267, D269 to D268, D270 to D269, D28 to D27, D271 to D270, D272 to D271, D273 to D272, D274 to D273, D275 to D274, D276 to D275, D277 to D276, D278 to D277, D279 to D278, D280 to D279, D29 to D28, D281 to D280, D282 to D281, D283 to D282, D284 to D283, D285 to D284, D286 to D285, D287 to D286, D288 to D287, D289 to D288, D290 to D289, D30 to D29, D291 to D290, D292 to D291, D293 to D292, D294 to D293, D295 to D294, D296 to D295, D297 to D296, D298 to D297, D299 to D298, D300 to D299, D4 to D3, D31 to D30, D301 to D300, D302 to D301, D303 to D302, D304 to D303, D305 to D304, D306 to D305, D307 to D306, D308 to D307, D309 to D308, D310 to D309, D32 to D31, D311 to D310, D312 to D311, D313 to D312, D314 to D313, D315 to D314, D316 to D315, D317 to D316, D318 to D317, D319 to D318, D320 to D319, D33 to D32, D321 to D320, D322 to D321, D323 to D322, D324 to D323, D325 to D324, D326 to D325, D327 to D326, D328 to D327, D329 to D328, D330 to D329, D34 to D33, D331 to D330, D332 to D331, D333 to D332, D334 to D333, D335 to D334, D336 to D335, D337 to D336, D338 to D337, D339 to D338, D340 to D339, D35 to D34, D341 to D340, D342 to D341, D343 to D342, D344 to D343, D345 to D344, D346 to D345, D347 to D346, D348 to D347, D349 to D348, D350 to D349, D36 to D35, D351 to D350, D352 to D351, D353 to D352, D354 to D353, D355 to D354, D356 to D355, D357 to D356, D358 to D357, D359 to D358, D360 to D359, D37 to D36, D361 to D360, D362 to D361, D363 to D362, D364 to D363, D365 to D364, D366 to D365, D367 to D366, D368 to D367, D369 to D368, D370 to D369, D38 to D37, D371 to D370, D372 to D371, D373 to D372, D374 to D373, D375 to D374, D376 to D375, D377 to D376, D378 to D377, D379 to D378, D380 to D379, D39 to D38, D381 to D380, D382 to D381, D383 to D382, D384 to D383, D385 to D384, D386 to D385, D387 to D386, D388 to D387, D389 to D388, D390 to D389, D40 to D39, D391 to D390, D392 to D391, D393 to D392, D394 to D393, D395 to D394, D396 to D395, D397 to D396, D398 to D397, D399 to D398, D400 to D399, D5 to D4, D41 to D40, D401 to D400, D402 to D401, D403 to D402, D404 to D403, D405 to D404, D406 to D405, D407 to D406, D408 to D407, D409 to D408, D410 to D409, D42 to D41, D411 to D410, D412 to D411, D413 to D412, D414 to D413, D415 to D414, D416 to D415, D417 to D416, D418 to D417, D419 to D418, D420 to D419, D43 to D42, D421 to D420, D422 to D421, D423 to D422, D424 to D423, D425 to D424, D426 to D425, D427 to D426, D428 to D427, D429 to D428, D430 to D429, D44 to D43, D431 to D430, D432 to D431, D433 to D432, D434 to D433, D435 to D434, D436 to D435, D437 to D436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
