File: hard/uc.sch (KiCad schematic (older format))
At the start: 29 parts, among them J1 Conn_01x06, M1 2N7002,215

Commit message: layout progress
Connections:
- net y22 is gone; now on net x20: MCU1.5 (PE6(TRACED3,TIM9_CH2,SPI4_MOSI,SAI1_SD_A,FMC_A22,DCMI_D7))
- net LED_STATUS: now also MCU1.1 (PE2(TRACECLK,SPI4_SCK,SAI1_MCLK_A,QUADSPI_BK1_IO2,FMC_A23)); no longer MCU1.37 (PB2(TIM2_CH4,SAI1_SD_A,SPI3_MOSI/I2S3_SD,QUADSPI_CLK,OTG_HS_ULPI_D4,SDIO_CK,BOOT1))
- net x10: now also MCU1.72 (PA13(JTMS-SWDIO)), R2.1; no longer MCU1.69 (PA10(TIM1_CH3,USART1_RX,OTG_FS_ID,DCMI_D1))
- net x13: now also MCU1.67 (PA8(MCO1,TIM1_CH1,I2C3_SCL,USART1_CK,OTG_FS_SOF)); no longer MCU1.72 (PA13(JTMS-SWDIO)), R2.1
- net x14: now also MCU1.69 (PA10(TIM1_CH3,USART1_RX,OTG_FS_ID,DCMI_D1)); no longer MCU1.76 (PA14(JTCK-SWCLK)), R1.1
- net x16: now also MCU1.37 (PB2(TIM2_CH4,SAI1_SD_A,SPI3_MOSI/I2S3_SD,QUADSPI_CLK,OTG_HS_ULPI_D4,SDIO_CK,BOOT1)); no longer MCU1.15 (PC0(SAI1_MCLK_B,OTG_HS_ULPI_STP,FMC_SDNWE))
- net x17: now also MCU1.2 (PE3(TRACED0,SAI1_SD_B,FMC_A19)); no longer MCU1.16 (PC1(SPI3_MOSI/I2S3_SD,SAI1_SD_A,SPI2_MOSI/I2S2_SD,ADC123_IN11))
- net x18: now also MCU1.3 (PE4(TRACED1,SPI4_NSS,SAI1_FS_A,FMC_A20,DCMI_D4)); no longer MCU1.17 (PC2(SPI2_MISO,OTG_HS_ULPI_DIR,FMC_SDNE0,ADC123_IN12))
- net x19: now also MCU1.4 (PE5(TRACED2,TIM9_CH1,SPI4_MISO,SAI1_SCK_A,FMC_A21,DCMI_D6)); no longer MCU1.18 (PC3(SPI2_MOSI/I2S2_SD,OTG_HS_ULPI_NXT,FMC_SDCKE0,ADC123_IN13))
- net x20: no longer MCU1.33 (PC4(I2S1_MCK,SPDIFRX_IN2,FMC_SDNE0,ADC12_IN14))
- net x21: now also MCU1.38 (PE7(TIM1_ETR,UART5_RX,QUADSPI_BK2_IO0,FMC_D4)); no longer MCU1.34 (PC5(USART3_RX,SPDIFRX_IN3,FMC_SDCKE0,ADC12_IN15))
- net x22: now also MCU1.96 (PB9(TIM2_CH2,TIM4_CH4,TIM11_CH1,I2C1_SDA,SPI2_NSS/I2S2_WS,SAI1_FS_B,CAN1_TX,SDIO_D5,DCMI_D7)); no longer MCU1.64 (PC7(TIM3_CH2,TIM8_CH2,FMPI2C1_SDA,SPI2_SCK/I2S2_CK,I2S3_MCK,SPDIFRX_IN1,USART6_RX,SDIO_D7,DCMI_D1))
- net x23: now also MCU1.95 (PB8(TIM2_CH1/TIM2_ETR,TIM4_CH3,TIM10_CH1,I2C1_SCL,CAN1_RX,SDIO_D4,DCMI_D6)); no longer MCU1.63 (PC6(TIM3_CH1,TIM8_CH1,FMPI2C1_SCL,I2S2_MCK,USART6_TX,SDIO_D6,DCMI_D0))
- net x24: now also MCU1.39 (PE8(TIM1_CH1N,UART5_TX,QUADSPI_BK2_IO1,FMC_D5)); no longer MCU1.65 (PC8(TRACED0,TIM3_CH3,TIM8_CH3,UART5_RTS,USART6_CK,SDIO_D0,DCMI_D2))
- net x25: now also MCU1.40 (PE9(TIM1_CH1,QUADSPI_BK2_IO2,FMC_D6)); no longer MCU1.66 (PC9(MCO2,TIM3_CH4,TIM8_CH4,I2C3_SDA,I2S_CKIN,UART5_CTS,QUADSPI_BK1_IO0,SDIO_D1,DCMI_D3))
- net x26: now also MCU1.41 (PE10(TIM1_CH2N,QUADSPI_BK2_IO3,FMC_D7)); no longer MCU1.78 (PC10(SPI3_SCK/I2S3_CK,USART3_TX,UART4_TX,QUADSPI_BK1_IO1,SDIO_D2,DCMI_D8))
- net x27: now also MCU1.42 (PE11(TIM1_CH2,SPI4_NSS,SAI2_SD_B,FMC_D8)); no longer MCU1.79 (PC11(SPI3_MISO,USART3_RX,UART4_RX,QUADSPI_BK2_NCS,SDIO_D3,DCMI_D4))
- net x28: now also MCU1.43 (PE12(TIM1_CH3N,SPI4_SCK,SAI2_SCK_B,FMC_D9)); no longer MCU1.80 (PC12(I2C2_SDA,SPI3_MOSI/I2S3_SD,USART3_CK,UART5_TX,SDIO_CK,DCMI_D9))
- net x29: now also MCU1.44 (PE13(TIM1_CH3,SPI4_MISO,SAI2_FS_B,FMC_D10)); no longer MCU1.7 (PC13(TAMP_1/WKUP1))
- net x30: now also MCU1.45 (PE14(TIM1_CH4,SPI4_MOSI,SAI2_MCLK_B,FMC_D11)); no longer MCU1.8 (PC14(OSC32_IN))
- net x31: now also MCU1.46 (PE15(TIM1_BKIN,FMC_D12)); no longer MCU1.9 (PC15(OSC32_OUT))
- net x8: now also MCU1.76 (PA14(JTCK-SWCLK)), R1.1; no longer MCU1.67 (PA8(MCO1,TIM1_CH1,I2C3_SCL,USART1_CK,OTG_FS_SOF))
- net y0: now also MCU1.56 (PD9(USART3_RX,FMC_D14)); no longer MCU1.81 (PD0(SPI4_MISO,SPI3_MOSI/I2S3_SD,CAN1_RX,FMC_D2))
- net y1: now also MCU1.88 (PD7(USART2_CK,SPDIFRX_IN0,FMC_NE1)); no longer MCU1.82 (PD1(SPI2_NSS/I2S2_WS,CAN1_TX,FMC_D3))
- net y11: now also MCU1.81 (PD0(SPI4_MISO,SPI3_MOSI/I2S3_SD,CAN1_RX,FMC_D2)); no longer MCU1.58 (PD11(FMPI2C1_SMBA,USART3_CTS,QUADSPI_BK1_IO0,SAI2_SD_A,FMC_A16))
- net y13: now also MCU1.80 (PC12(I2C2_SDA,SPI3_MOSI/I2S3_SD,USART3_CK,UART5_TX,SDIO_CK,DCMI_D9)); no longer MCU1.60 (PD13(TIM4_CH2,FMPI2C1_SDA,QUADSPI_BK1_IO3,SAI2_SCK_A,FMC_A18))
- net y15: now also MCU1.86 (PD5(USART2_TX,FMC_NWE)); no longer MCU1.62 (PD15(TIM4_CH4,FMPI2C1_SDA,FMC_D1))
- net y16: now also MCU1.18 (PC3(SPI2_MOSI/I2S2_SD,OTG_HS_ULPI_NXT,FMC_SDCKE0,ADC123_IN13))
- net y17: now also MCU1.83 (PD2(TIM3_ETR,UART5_RX,SDIO_CMD,DCMI_D11))
- net y18: now also MCU1.33 (PC4(I2S1_MCK,SPDIFRX_IN2,FMC_SDNE0,ADC12_IN14)); no longer MCU1.1 (PE2(TRACECLK,SPI4_SCK,SAI1_MCLK_A,QUADSPI_BK1_IO2,FMC_A23))
- net y19: now also MCU1.79 (PC11(SPI3_MISO,USART3_RX,UART4_RX,QUADSPI_BK2_NCS,SDIO_D3,DCMI_D4)); no longer MCU1.2 (PE3(TRACED0,SAI1_SD_B,FMC_A19))
- net y2: now also MCU1.58 (PD11(FMPI2C1_SMBA,USART3_CTS,QUADSPI_BK1_IO0,SAI2_SD_A,FMC_A16)); no longer MCU1.83 (PD2(TIM3_ETR,UART5_RX,SDIO_CMD,DCMI_D11))
- net y20: now also MCU1.64 (PC7(TIM3_CH2,TIM8_CH2,FMPI2C1_SDA,SPI2_SCK/I2S2_CK,I2S3_MCK,SPDIFRX_IN1,USART6_RX,SDIO_D7,DCMI_D1)); no longer MCU1.3 (PE4(TRACED1,SPI4_NSS,SAI1_FS_A,FMC_A20,DCMI_D4))
- net y21: now also MCU1.78 (PC10(SPI3_SCK/I2S3_CK,USART3_TX,UART4_TX,QUADSPI_BK1_IO1,SDIO_D2,DCMI_D8)); no longer MCU1.4 (PE5(TRACED2,TIM9_CH1,SPI4_MISO,SAI1_SCK_A,FMC_A21,DCMI_D6))
- net y23: now also MCU1.7 (PC13(TAMP_1/WKUP1)); no longer MCU1.38 (PE7(TIM1_ETR,UART5_RX,QUADSPI_BK2_IO0,FMC_D4))
- net y24: now also MCU1.34 (PC5(USART3_RX,SPDIFRX_IN3,FMC_SDCKE0,ADC12_IN15)); no longer MCU1.39 (PE8(TIM1_CH1N,UART5_TX,QUADSPI_BK2_IO1,FMC_D5))
- net y25: now also MCU1.8 (PC14(OSC32_IN)); no longer MCU1.40 (PE9(TIM1_CH1,QUADSPI_BK2_IO2,FMC_D6))
- net y26: now also MCU1.63 (PC6(TIM3_CH1,TIM8_CH1,FMPI2C1_SCL,I2S2_MCK,USART6_TX,SDIO_D6,DCMI_D0)); no longer MCU1.41 (PE10(TIM1_CH2N,QUADSPI_BK2_IO3,FMC_D7))
- net y27: now also MCU1.15 (PC0(SAI1_MCLK_B,OTG_HS_ULPI_STP,FMC_SDNWE)); no longer MCU1.42 (PE11(TIM1_CH2,SPI4_NSS,SAI2_SD_B,FMC_D8))
- net y28: now also MCU1.66 (PC9(MCO2,TIM3_CH4,TIM8_CH4,I2C3_SDA,I2S_CKIN,UART5_CTS,QUADSPI_BK1_IO0,SDIO_D1,DCMI_D3)); no longer MCU1.43 (PE12(TIM1_CH3N,SPI4_SCK,SAI2_SCK_B,FMC_D9))
- net y29: now also MCU1.16 (PC1(SPI3_MOSI/I2S3_SD,SAI1_SD_A,SPI2_MOSI/I2S2_SD,ADC123_IN11)); no longer MCU1.44 (PE13(TIM1_CH3,SPI4_MISO,SAI2_FS_B,FMC_D10))
- net y3: now also MCU1.87 (PD6(SPI3_MOSI/I2S3_SD,SAI1_SD_A,USART2_RX,FMC_NWAIT,DCMI_D10)); no longer MCU1.84 (PD3(TRACED1,SPI2_SCK/I2S2_CK,USART2_CTS,QUADSPI_CLK,FMC_CLK,DCMI_D5))
- net y30: now also MCU1.9 (PC15(OSC32_OUT)); no longer MCU1.45 (PE14(TIM1_CH4,SPI4_MOSI,SAI2_MCLK_B,FMC_D11))
- net y31: now also MCU1.17 (PC2(SPI2_MISO,OTG_HS_ULPI_DIR,FMC_SDNE0,ADC123_IN12)); no longer MCU1.46 (PE15(TIM1_BKIN,FMC_D12))
- net y4: now also MCU1.60 (PD13(TIM4_CH2,FMPI2C1_SDA,QUADSPI_BK1_IO3,SAI2_SCK_A,FMC_A18)); no longer MCU1.85 (PD4(USART2_RTS,FMC_NOE))
- net y5: now also MCU1.85 (PD4(USART2_RTS,FMC_NOE)); no longer MCU1.86 (PD5(USART2_TX,FMC_NWE))
- net y6: now also MCU1.62 (PD15(TIM4_CH4,FMPI2C1_SDA,FMC_D1)); no longer MCU1.87 (PD6(SPI3_MOSI/I2S3_SD,SAI1_SD_A,USART2_RX,FMC_NWAIT,DCMI_D10))
- net y7: now also MCU1.84 (PD3(TRACED1,SPI2_SCK/I2S2_CK,USART2_CTS,QUADSPI_CLK,FMC_CLK,DCMI_D5)); no longer MCU1.88 (PD7(USART2_CK,SPDIFRX_IN0,FMC_NE1))
- net y9: now also MCU1.82 (PD1(SPI2_NSS/I2S2_WS,CAN1_TX,FMC_D3)); no longer MCU1.56 (PD9(USART3_RX,FMC_D14))
Changed lines of the file:
@@
 Wire Wire Line
 	11950 6550 12000 6550
-Text GLabel 9950 5500 2    50   Input ~ 0
+Text GLabel 3550 6000 0    50   Input ~ 0
 y15
 Text GLabel 9950 5600 2    50   Input ~ 0
 y14
-Text GLabel 10850 6200 0    50   Input ~ 0
-nRST
 $Comp
 L Device:R R7
@@
 	11200 6200 11250 6200
 Text GLabel 13950 1900 2    50   Input ~ 0
-x14
+x8
 Text GLabel 13950 2300 2    50   Input ~ 0
-x13
+x10
 $Comp
 L power:GND #PWR02
@@
 	0    1    1    0
 $EndComp
-Text GLabel 3550 7000 0    50   Input ~ 0
+Text GLabel 11850 4700 2    50   Input ~ 0
 y19
 Text GLabel 13950 2900 2    50   Input ~ 0
@@
 Wire Wire Line
 	15950 7500 15950 7550
-Text GLabel 3550 3350 0    50   Input ~ 0
-LED_STATUS
 Wire Wire Line
 	13500 2300 13600 2300
@@
 Text GLabel 3550 2700 0    50   Input ~ 0
 x7
-Text GLabel 11050 2700 2    50   Input ~ 0
+Text GLabel 11050 2100 2    50   Input ~ 0
 x8
 Text GLabel 11050 2600 2    50   Input ~ 0
 x9
-Text GLabel 11050 2500 2    50   Input ~ 0
+Text GLabel 11050 2200 2    50   Input ~ 0
 x10
 Text GLabel 11050 2400 2    50   Input ~ 0
@@
 Text GLabel 11050 2300 2    50   Input ~ 0
 x12
-Text GLabel 11050 2200 2    50   Input ~ 0
+Text GLabel 11050 2700 2    50   Input ~ 0
 x13
-Text GLabel 11050 2100 2    50   Input ~ 0
+Text GLabel 11050 2500 2    50   Input ~ 0
 x14
 Text GLabel 11050 2000 2    50   Input ~ 0
 x15
-Text GLabel 3550 4300 0    50   Input ~ 0
-x16
-Text GLabel 3550 4400 0    50   Input ~ 0
-x17
-Text GLabel 3550 4500 0    50   Input ~ 0
-x18
-Text GLabel 3550 4600 0    50   Input ~ 0
-x19
-Text GLabel 3550 4700 0    50   Input ~ 0
-x20
 $Comp
 L led_matrix:STM32F446VE MCU1
@@
 	1    0    0    -1
 $EndComp
-Text GLabel 3550 4800 0    50   Input ~ 0
-x21
-Text GLabel 3550 4900 0    50   Input ~ 0
-x22
-Text GLabel 3550 5000 0    50   Input ~ 0
-x23
-Text GLabel 11850 5000 2    50   Input ~ 0
+Text GLabel 8250 7400 2    50   Input ~ 0
 x24
-Text GLabel 11850 4900 2    50   Input ~ 0
+Text GLabel 8250 7300 2    50   Input ~ 0
 x25
-Text GLabel 11850 4800 2    50   Input ~ 0
+Text GLabel 8250 7200 2    50   Input ~ 0
 x26
-Text GLabel 11850 4700 2    50   Input ~ 0
+Text GLabel 8250 7100 2    50   Input ~ 0
 x27
-Text GLabel 11850 4600 2    50   Input ~ 0
+Text GLabel 8250 7000 2    50   Input ~ 0
 x28
-Text GLabel 11850 4500 2    50   Input ~ 0
+Text GLabel 8250 6900 2    50   Input ~ 0
 x29
-Text GLabel 11850 4400 2    50   Input ~ 0
+Text GLabel 8250 6800 2    50   Input ~ 0
 x30
-Text GLabel 11850 4300 2    50   Input ~ 0
+Text GLabel 8250 6700 2    50   Input ~ 0
 x31
 Text GLabel 9950 6200 2    50   Input ~ 0
 y8
-Text GLabel 9950 6100 2    50   Input ~ 0
+Text GLabel 3550 5600 0    50   Input ~ 0
 y9
 Text GLabel 9950 6000 2    50   Input ~ 0
 y10
-Text GLabel 9950 5900 2    50   Input ~ 0
+Text GLabel 3550 5500 0    50   Input ~ 0
 y11
 Text GLabel 9950 5800 2    50   Input ~ 0
 y12
-Text GLabel 9950 5700 2    50   Input ~ 0
+Text GLabel 11850 4600 2    50   Input ~ 0
 y13
 Wire Wire Line
@@
 Wire Wire Line
 	13050 2300 13400 2300
-Text GLabel 2950 6700 0    50   Input ~ 0
-y16
-Text GLabel 2950 6800 0    50   Input ~ 0
+Text GLabel 3550 5700 0    50   Input ~ 0
 y17
-Text GLabel 3550 6900 0    50   Input ~ 0
+Text GLabel 3550 4700 0    50   Input ~ 0
 y18
 Text GLabel 3550 3450 0    50   Input ~ 0
 SWO
-Text GLabel 3550 7100 0    50   Input ~ 0
+Text GLabel 3550 4900 0    50   Input ~ 0
 y20
-Text GLabel 3550 7200 0    50   Input ~ 0
+Text GLabel 11850 4800 2    50   Input ~ 0
 y21
-Text GLabel 3550 7300 0    50   Input ~ 0
-y22
-Text GLabel 3550 7400 0    50   Input ~ 0
+Text GLabel 11850 4500 2    50   Input ~ 0
 y23
-Text GLabel 8250 7400 2    50   Input ~ 0
+Text GLabel 3550 4800 0    50   Input ~ 0
 y24
-Text GLabel 8250 7300 2    50   Input ~ 0
+Text GLabel 11850 4400 2    50   Input ~ 0
 y25
-Text GLabel 8250 7200 2    50   Input ~ 0
+Text GLabel 3550 5000 0    50   Input ~ 0
 y26
-Text GLabel 8250 7100 2    50   Input ~ 0
+Text GLabel 3550 4300 0    50   Input ~ 0
 y27
-Text GLabel 8250 7000 2    50   Input ~ 0
+Text GLabel 11850 4900 2    50   Input ~ 0
 y28
-Text GLabel 8250 6900 2    50   Input ~ 0
+Text GLabel 3550 4400 0    50   Input ~ 0
 y29
-Text GLabel 8250 6800 2    50   Input ~ 0
+Text GLabel 11850 4300 2    50   Input ~ 0
 y30
-Text GLabel 8250 6700 2    50   Input ~ 0
+Text GLabel 3550 4500 0    50   Input ~ 0
 y31
-Text GLabel 3550 5700 0    50   Input ~ 0
+Text GLabel 9950 5900 2    50   Input ~ 0
 y2
+Text GLabel 3550 5800 0    50   Input ~ 0
+y7
+Text GLabel 9950 5500 2    50   Input ~ 0
+y6
+Text GLabel 3550 5900 0    50   Input ~ 0
+y5
+Text GLabel 9950 5700 2    50   Input ~ 0
+y4
+Text GLabel 3550 6100 0    50   Input ~ 0
+y3
 Text GLabel 3550 6200 0    50   Input ~ 0
-y7
-Text GLabel 3550 6100 0    50   Input ~ 0
-y6
-Text GLabel 3550 6000 0    50   Input ~ 0
-y5
-Text GLabel 3550 5900 0    50   Input ~ 0
-y4
-Text GLabel 3550 5800 0    50   Input ~ 0
-y3
-Text GLabel 3550 5600 0    50   Input ~ 0
 y1
-Text GLabel 3550 5500 0    50   Input ~ 0
+Text GLabel 9950 6100 2    50   Input ~ 0
 y0
 Text GLabel 3550 3150 0    50   Input ~ 0
@@
 Text GLabel 3550 6800 0    50   Input ~ 0
 ACC_INT2
+Text GLabel 11650 3850 2    50   Input ~ 0
+x23
+Text GLabel 11650 3750 2    50   Input ~ 0
+x22
+Text GLabel 3550 7400 0    50   Input ~ 0
+x21
+Text GLabel 3550 7300 0    50   Input ~ 0
+x20
+Text GLabel 3550 7200 0    50   Input ~ 0
+x19
+Text GLabel 3550 7100 0    50   Input ~ 0
+x18
+Text GLabel 3550 7000 0    50   Input ~ 0
+x17
+Text GLabel 3550 3350 0    50   Input ~ 0
+x16
+Text GLabel 3550 6900 0    50   Input ~ 0
+LED_STATUS
+Text GLabel 3550 4600 0    50   Input ~ 0
+y16
+Text GLabel 10850 6200 0    50   Input ~ 0
+nRST
 $EndSCHEMATC

Commit message: layout progress
Connections:
- net x13 is gone; now on net x5: MCU1.67 (PA8(MCO1,TIM1_CH1,I2C3_SCL,USART1_CK,OTG_FS_SOF))
- net x25 is gone; now on net x14: MCU1.40 (PE9(TIM1_CH1,QUADSPI_BK2_IO2,FMC_D6))
- net x26 is gone; now on net x15: MCU1.41 (PE10(TIM1_CH2N,QUADSPI_BK2_IO3,FMC_D7))
- net x28 is gone; now on net x7: MCU1.43 (PE12(TIM1_CH3N,SPI4_SCK,SAI2_SCK_B,FMC_D9))
- net x29 is gone; now on net x9: MCU1.44 (PE13(TIM1_CH3,SPI4_MISO,SAI2_FS_B,FMC_D10))
- net x30 is gone; now on net x11: MCU1.45 (PE14(TIM1_CH4,SPI4_MOSI,SAI2_MCLK_B,FMC_D11))
- net x31 is gone; now on net x12: MCU1.46 (PE15(TIM1_BKIN,FMC_D12))
- net x0: now also MCU1.77 (PA15(JTDI,TIM2_CH1/TIM2_ETR,HDMI_CEC,SPI1_NSS/I2S1_WS,SPI3_NSS/I2S3_WS,UART4_RTS))
- net x1: now also MCU1.70 (PA11(TIM1_CH4,USART1_CTS,CAN1_RX,OTG_FS_DM))
- net x10: now also MCU1.76 (PA14(JTCK-SWCLK)), R1.1; no longer MCU1.72 (PA13(JTMS-SWDIO)), R2.1
- net x11: no longer MCU1.70 (PA11(TIM1_CH4,USART1_CTS,CAN1_RX,OTG_FS_DM))
- net x12: no longer MCU1.71 (PA12(TIM1_ETR,USART1_RTS,SAI2_FS_B,CAN1_TX,OTG_FS_DP))
- net x14: no longer MCU1.69 (PA10(TIM1_CH3,USART1_RX,OTG_FS_ID,DCMI_D1))
- net x15: no longer MCU1.77 (PA15(JTDI,TIM2_CH1/TIM2_ETR,HDMI_CEC,SPI1_NSS/I2S1_WS,SPI3_NSS/I2S3_WS,UART4_RTS))
- net x2: now also MCU1.71 (PA12(TIM1_ETR,USART1_RTS,SAI2_FS_B,CAN1_TX,OTG_FS_DP))
- net x3: now also MCU1.69 (PA10(TIM1_CH3,USART1_RX,OTG_FS_ID,DCMI_D1))
- net x4: now also MCU1.68 (PA9(TIM1_CH2,I2C3_SMBA,SPI2_SCK/I2S2_CK,SAI1_SD_B,USART1_TX,DCMI_D0,OTG_FS_VBUS))
- net x6: now also MCU1.90 (PB4(NJTRST,TIM3_CH1,I2C3_SDA,SPI1_MISO,SPI3_MISO,SPI2_NSS/I2S2_WS))
- net x8: now also MCU1.72 (PA13(JTMS-SWDIO)), R2.1; no longer MCU1.76 (PA14(JTCK-SWCLK)), R1.1
- net x9: no longer MCU1.68 (PA9(TIM1_CH2,I2C3_SMBA,SPI2_SCK/I2S2_CK,SAI1_SD_B,USART1_TX,DCMI_D0,OTG_FS_VBUS))
- net y0: now also MCU1.33 (PC4(I2S1_MCK,SPDIFRX_IN2,FMC_SDNE0,ADC12_IN14)); no longer MCU1.56 (PD9(USART3_RX,FMC_D14))
- net y10: now also MCU1.64 (PC7(TIM3_CH2,TIM8_CH2,FMPI2C1_SDA,SPI2_SCK/I2S2_CK,I2S3_MCK,SPDIFRX_IN1,USART6_RX,SDIO_D7,DCMI_D1)); no longer MCU1.57 (PD10(USART3_CK,FMC_D15))
- net y12: now also MCU1.63 (PC6(TIM3_CH1,TIM8_CH1,FMPI2C1_SCL,I2S2_MCK,USART6_TX,SDIO_D6,DCMI_D0)); no longer MCU1.59 (PD12(TIM4_CH1,FMPI2C1_SCL,USART3_RTS,QUADSPI_BK1_IO1,SAI2_FS_A,FMC_A17))
- net y14: now also MCU1.60 (PD13(TIM4_CH2,FMPI2C1_SDA,QUADSPI_BK1_IO3,SAI2_SCK_A,FMC_A18)); no longer MCU1.61 (PD14(TIM4_CH3,FMPI2C1_SCL,SAI2_SCK_A,FMC_D0))
- net y16: now also MCU1.55 (PD8(USART3_TX,SPDIFRX_IN1,FMC_D13)); no longer MCU1.18 (PC3(SPI2_MOSI/I2S2_SD,OTG_HS_ULPI_NXT,FMC_SDCKE0,ADC123_IN13))
- net y18: now also MCU1.56 (PD9(USART3_RX,FMC_D14)); no longer MCU1.33 (PC4(I2S1_MCK,SPDIFRX_IN2,FMC_SDNE0,ADC12_IN14))
- net y2: now also MCU1.34 (PC5(USART3_RX,SPDIFRX_IN3,FMC_SDCKE0,ADC12_IN15)); no longer MCU1.58 (PD11(FMPI2C1_SMBA,USART3_CTS,QUADSPI_BK1_IO0,SAI2_SD_A,FMC_A16))
- net y20: now also MCU1.59 (PD12(TIM4_CH1,FMPI2C1_SCL,USART3_RTS,QUADSPI_BK1_IO1,SAI2_FS_A,FMC_A17)); no longer MCU1.64 (PC7(TIM3_CH2,TIM8_CH2,FMPI2C1_SDA,SPI2_SCK/I2S2_CK,I2S3_MCK,SPDIFRX_IN1,USART6_RX,SDIO_D7,DCMI_D1))
- net y24: now also MCU1.58 (PD11(FMPI2C1_SMBA,USART3_CTS,QUADSPI_BK1_IO0,SAI2_SD_A,FMC_A16)); no longer MCU1.34 (PC5(USART3_RX,SPDIFRX_IN3,FMC_SDCKE0,ADC12_IN15))
- net y26: now also MCU1.61 (PD14(TIM4_CH3,FMPI2C1_SCL,SAI2_SCK_A,FMC_D0)); no longer MCU1.63 (PC6(TIM3_CH1,TIM8_CH1,FMPI2C1_SCL,I2S2_MCK,USART6_TX,SDIO_D6,DCMI_D0))
- net y27: now also MCU1.9 (PC15(OSC32_OUT)); no longer MCU1.15 (PC0(SAI1_MCLK_B,OTG_HS_ULPI_STP,FMC_SDNWE))
- net y28: now also MCU1.62 (PD15(TIM4_CH4,FMPI2C1_SDA,FMC_D1)); no longer MCU1.66 (PC9(MCO2,TIM3_CH4,TIM8_CH4,I2C3_SDA,I2S_CKIN,UART5_CTS,QUADSPI_BK1_IO0,SDIO_D1,DCMI_D3))
- net y29: now also MCU1.15 (PC0(SAI1_MCLK_B,OTG_HS_ULPI_STP,FMC_SDNWE)); no longer MCU1.16 (PC1(SPI3_MOSI/I2S3_SD,SAI1_SD_A,SPI2_MOSI/I2S2_SD,ADC123_IN11))
- net y30: now also MCU1.65 (PC8(TRACED0,TIM3_CH3,TIM8_CH3,UART5_RTS,USART6_CK,SDIO_D0,DCMI_D2)); no longer MCU1.9 (PC15(OSC32_OUT))
- net y31: now also MCU1.16 (PC1(SPI3_MOSI/I2S3_SD,SAI1_SD_A,SPI2_MOSI/I2S2_SD,ADC123_IN11)); no longer MCU1.17 (PC2(SPI2_MISO,OTG_HS_ULPI_DIR,FMC_SDNE0,ADC123_IN12))
- net y4: now also MCU1.18 (PC3(SPI2_MOSI/I2S2_SD,OTG_HS_ULPI_NXT,FMC_SDCKE0,ADC123_IN13)); no longer MCU1.60 (PD13(TIM4_CH2,FMPI2C1_SDA,QUADSPI_BK1_IO3,SAI2_SCK_A,FMC_A18))
- net y6: now also MCU1.17 (PC2(SPI2_MISO,OTG_HS_ULPI_DIR,FMC_SDNE0,ADC123_IN12)); no longer MCU1.62 (PD15(TIM4_CH4,FMPI2C1_SDA,FMC_D1))
- net y8: now also MCU1.66 (PC9(MCO2,TIM3_CH4,TIM8_CH4,I2C3_SDA,I2S_CKIN,UART5_CTS,QUADSPI_BK1_IO0,SDIO_D1,DCMI_D3)); no longer MCU1.55 (PD8(USART3_TX,SPDIFRX_IN1,FMC_D13))
- new net y22: MCU1.57 (PD10(USART3_CK,FMC_D15))
Changed lines of the file:
@@
-$Comp
-L led_matrix:STM32F446VE MCU1
-U 2 1 605A0D1E
-P 7600 3050
-F 0 "MCU1" H 7600 3215 50  0000 C CNN
-F 1 "STM32F446VE" H 7600 3124 50  0000 C CNN
-F 2 "led_matrix:LQFP-100_14x14mm_P0.5mm" H 8150 3400 50  0001 C CNN
-F 3 "https://www.st.com/resource/en/datasheet/stm32f446ve.pdf" H 8150 3400 50  0001 C CNN
-F 4 "C91929" H 7600 3050 50  0001 C CNN "JLCPCB_Part_Number"
-F 5 "STMicroelectronics" H 7600 3050 50  0001 C CNN "MF"
-F 6 "STM32F446VET6" H 7600 3050 50  0001 C CNN "MPN"
-F 7 "ST MICROELECTRONICS LQFP-100_14X14X05P ROHS" H 7600 3050 50  0001 C CNN "Description"
-	2    7600 3050
-	1    0    0    -1
-$EndComp
 $Comp
 L led_matrix:STM32F446VE MCU1
@@
 y15
 Text GLabel 9950 5600 2    50   Input ~ 0
-y14
+y26
 $Comp
 L Device:R R7
@@
 	11200 6200 11250 6200
 Text GLabel 13950 1900 2    50   Input ~ 0
+x10
+Text GLabel 13950 2300 2    50   Input ~ 0
 x8
-Text GLabel 13950 2300 2    50   Input ~ 0
-x10
 $Comp
 L power:GND #PWR02
@@
 x7
 Text GLabel 11050 2100 2    50   Input ~ 0
+x10
+Text GLabel 11050 2600 2    50   Input ~ 0
+x4
+Text GLabel 11050 2200 2    50   Input ~ 0
 x8
-Text GLabel 11050 2600 2    50   Input ~ 0
-x9
-Text GLabel 11050 2200 2    50   Input ~ 0
-x10
 Text GLabel 11050 2400 2    50   Input ~ 0
-x11
+x1
 Text GLabel 11050 2300 2    50   Input ~ 0
-x12
+x2
 Text GLabel 11050 2700 2    50   Input ~ 0
-x13
+x5
 Text GLabel 11050 2500 2    50   Input ~ 0
-x14
+x3
 Text GLabel 11050 2000 2    50   Input ~ 0
-x15
+x0
 $Comp
 L led_matrix:STM32F446VE MCU1
@@
 x24
 Text GLabel 8250 7300 2    50   Input ~ 0
-x25
+x14
 Text GLabel 8250 7200 2    50   Input ~ 0
-x26
+x15
 Text GLabel 8250 7100 2    50   Input ~ 0
 x27
 Text GLabel 8250 7000 2    50   Input ~ 0
-x28
-Text GLabel 8250 6900 2    50   Input ~ 0
-x29
+x7
 Text GLabel 8250 6800 2    50   Input ~ 0
-x30
+x11
 Text GLabel 8250 6700 2    50   Input ~ 0
-x31
+x12
 Text GLabel 9950 6200 2    50   Input ~ 0
-y8
+y16
 Text GLabel 3550 5600 0    50   Input ~ 0
 y9
 Text GLabel 9950 6000 2    50   Input ~ 0
-y10
+y22
 Text GLabel 3550 5500 0    50   Input ~ 0
 y11
 Text GLabel 9950 5800 2    50   Input ~ 0
-y12
+y20
 Text GLabel 11850 4600 2    50   Input ~ 0
 y13
@@
 y17
 Text GLabel 3550 4700 0    50   Input ~ 0
-y18
+y0
 Text GLabel 3550 3450 0    50   Input ~ 0
 SWO
 Text GLabel 3550 4900 0    50   Input ~ 0
-y20
+y10
 Text GLabel 11850 4800 2    50   Input ~ 0
 y21
@@
 y23
 Text GLabel 3550 4800 0    50   Input ~ 0
-y24
+y2
 Text GLabel 11850 4400 2    50   Input ~ 0
 y25
 Text GLabel 3550 5000 0    50   Input ~ 0
-y26
+y12
 Text GLabel 3550 4300 0    50   Input ~ 0
-y27
-Text GLabel 11850 4900 2    50   Input ~ 0
-y28
+y29
 Text GLabel 3550 4400 0    50   Input ~ 0
-y29
-Text GLabel 11850 4300 2    50   Input ~ 0
-y30
+y31
 Text GLabel 3550 4500 0    50   Input ~ 0
-y31
+y6
 Text GLabel 9950 5900 2    50   Input ~ 0
-y2
+y24
 Text GLabel 3550 5800 0    50   Input ~ 0
 y7
 Text GLabel 9950 5500 2    50   Input ~ 0
-y6
+y28
 Text GLabel 3550 5900 0    50   Input ~ 0
 y5
 Text GLabel 9950 5700 2    50   Input ~ 0
-y4
+y14
 Text GLabel 3550 6100 0    50   Input ~ 0
 y3
@@
 y1
 Text GLabel 9950 6100 2    50   Input ~ 0
-y0
+y18
 Text GLabel 3550 3150 0    50   Input ~ 0
 3MM5_TIP
@@
 Text GLabel 3550 7100 0    50   Input ~ 0
 x18
+Text GLabel 3550 6900 0    50   Input ~ 0
+LED_STATUS
+Text GLabel 3550 4600 0    50   Input ~ 0
+y4
+Text GLabel 10850 6200 0    50   Input ~ 0
+nRST
+Text GLabel 11850 4300 2    50   Input ~ 0
+y27
+Text GLabel 11850 5000 2    50   Input ~ 0
+y30
+Text GLabel 11850 4900 2    50   Input ~ 0
+y8
+$Comp
+L led_matrix:STM32F446VE MCU1
+U 2 1 605A0D1E
+P 7600 3050
+F 0 "MCU1" H 7600 3215 50  0000 C CNN
+F 1 "STM32F446VE" H 7600 3124 50  0000 C CNN
+F 2 "led_matrix:LQFP-100_14x14mm_P0.5mm" H 8150 3400 50  0001 C CNN
+F 3 "https://www.st.com/resource/en/datasheet/stm32f446ve.pdf" H 8150 3400 50  0001 C CNN
+F 4 "C91929" H 7600 3050 50  0001 C CNN "JLCPCB_Part_Number"
+F 5 "STMicroelectronics" H 7600 3050 50  0001 C CNN "MF"
+F 6 "STM32F446VET6" H 7600 3050 50  0001 C CNN "MPN"
+F 7 "ST MICROELECTRONICS LQFP-100_14X14X05P ROHS" H 7600 3050 50  0001 C CNN "Description"
+	2    7600 3050
+	1    0    0    -1
+$EndComp
+Text GLabel 3550 3550 0    50   Input ~ 0
+x6
+Text GLabel 8250 6900 2    50   Input ~ 0
+x9
 Text GLabel 3550 7000 0    50   Input ~ 0
 x17
 Text GLabel 3550 3350 0    50   Input ~ 0
 x16
-Text GLabel 3550 6900 0    50   Input ~ 0
-LED_STATUS
-Text GLabel 3550 4600 0    50   Input ~ 0
-y16
-Text GLabel 10850 6200 0    50   Input ~ 0
-nRST
 $EndSCHEMATC
