File: hard/uc.sch (KiCad schematic (older format))
At the start: 29 parts, among them J1 Conn_01x06, M1 2N7002,215

Commit message: release candidate. ready for review by @lukekaese
Parts:
- removed C1, C10, C11, C13, C15, C16, C2, C5, C6, C7: 0u1/6V3, Capacitor_SMD:C_0402_1005Metric, symbol Device:C
- removed C12, C14: 1u/6V3, Capacitor_SMD:C_0805_2012Metric, symbol Device:C
- removed C3, C4: 4u7/6V3, Capacitor_SMD:C_0805_2012Metric, symbol Device:C
- removed C8, C9: 10u/6V3, Capacitor_SMD:C_0805_2012Metric, symbol Device:C
- removed D1: LTST-S270TBKT, led_matrix:LED_LiteOn_LTST-S270TBKT, symbol led_matrix:LTST-S270TBKT
- removed L1: 0R, Resistor_SMD:R_1206_3216Metric, symbol Device:L
- removed M1: 2N7002,215, Package_TO_SOT_SMD:SOT-23, symbol led_matrix:2N7002,215
- removed unit 7 of MCU1
- removed R10: 1K8, Resistor_SMD:R_0402_1005Metric, symbol Device:R
- removed R7: 470R, Resistor_SMD:R_0402_1005Metric, symbol Device:R
- removed R8: 10K, Resistor_SMD:R_0402_1005Metric, symbol Device:R
- removed R9: 3K3, Resistor_SMD:R_0402_1005Metric, symbol Device:R
Connections:
- net LED_STATUS: no longer MCU1.1 (PE2(TRACECLK,SPI4_SCK,SAI1_MCLK_A,QUADSPI_BK1_IO2,FMC_A23))
- net x0: no longer MCU1.23 (PA0(TIM2_CH1/TIM2_ETR,TIM5_CH1,TIM8_ETR,USART2_CTS,UART4_TX,ADC123_IN0,WKUP0/TAMP_2))
- net x1: no longer MCU1.24 (PA1(TIM2_CH2,TIM5_CH2,USART2_RTS,UART4_RX,QUADSPI_BK1_IO3,SAI2_MCLK_B,ADC123_IN1))
- net x15: now also MCU1.31 (PA6(TIM1_BKIN,TIM3_CH1,TIM8_BKIN,SPI1_MISO,I2S2_MCK,TIM13_CH1,DCMI_PIXCLK,ADC12_IN6)); no longer MCU1.41 (PE10(TIM1_CH2N,QUADSPI_BK2_IO3,FMC_D7))
- net x17: now also MCU1.26 (PA3(TIM2_CH4,TIM5_CH4,TIM9_CH2,SAI1_FS_A,USART2_RX,OTG_HS_ULPI_D0,ADC123_IN3)); no longer MCU1.2 (PE3(TRACED0,SAI1_SD_B,FMC_A19))
- net x18: now also MCU1.32 (PA7(TIM1_CH1N,TIM3_CH2,TIM8_CH1N,SPI1_MOSI/I2S1_SD,TIM14_CH1,FMC_SDNWE,ADC12_IN7)); no longer MCU1.3 (PE4(TRACED1,SPI4_NSS,SAI1_FS_A,FMC_A20,DCMI_D4))
- net x19: now also MCU1.30 (PA5(TIM2_CH1/TIM2_ETR,TIM8_CH1N,SPI1_SCK/I2S1_CK,OTG_HS_ULPI_CK,ADC12_IN5,DAC_OUT2)); no longer MCU1.4 (PE5(TRACED2,TIM9_CH1,SPI4_MISO,SAI1_SCK_A,FMC_A21,DCMI_D6))
- net x2: no longer MCU1.25 (PA2(TIM2_CH3,TIM5_CH3,TIM9_CH1,USART2_TX,SAI2_SCK_B,ADC123_IN2))
- net x20: now also MCU1.29 (PA4(SPI1_NSS/I2S1_WS,SPI3_NSS/I2S3_WS,USART2_CK,OTG_HS_SOF,DCMI_HSYNC,ADC12_IN4,DAC_OUT1)); no longer MCU1.5 (PE6(TRACED3,TIM9_CH2,SPI4_MOSI,SAI1_SD_A,FMC_A22,DCMI_D7))
- net x21: now also MCU1.24 (PA1(TIM2_CH2,TIM5_CH2,USART2_RTS,UART4_RX,QUADSPI_BK1_IO3,SAI2_MCLK_B,ADC123_IN1)); no longer MCU1.38 (PE7(TIM1_ETR,UART5_RX,QUADSPI_BK2_IO0,FMC_D4))
- net x22: now also MCU1.23 (PA0(TIM2_CH1/TIM2_ETR,TIM5_CH1,TIM8_ETR,USART2_CTS,UART4_TX,ADC123_IN0,WKUP0/TAMP_2)); no longer MCU1.96 (PB9(TIM2_CH2,TIM4_CH4,TIM11_CH1,I2C1_SDA,SPI2_NSS/I2S2_WS,SAI1_FS_B,CAN1_TX,SDIO_D5,DCMI_D7))
- net x23: now also MCU1.38 (PE7(TIM1_ETR,UART5_RX,QUADSPI_BK2_IO0,FMC_D4)); no longer MCU1.95 (PB8(TIM2_CH1/TIM2_ETR,TIM4_CH3,TIM10_CH1,I2C1_SCL,CAN1_RX,SDIO_D4,DCMI_D6))
- net x24: now also MCU1.95 (PB8(TIM2_CH1/TIM2_ETR,TIM4_CH3,TIM10_CH1,I2C1_SCL,CAN1_RX,SDIO_D4,DCMI_D6)); no longer MCU1.39 (PE8(TIM1_CH1N,UART5_TX,QUADSPI_BK2_IO1,FMC_D5))
- net x27: now also MCU1.5 (PE6(TRACED3,TIM9_CH2,SPI4_MOSI,SAI1_SD_A,FMC_A22,DCMI_D7)); no longer MCU1.42 (PE11(TIM1_CH2,SPI4_NSS,SAI2_SD_B,FMC_D8))
- net x3: no longer MCU1.26 (PA3(TIM2_CH4,TIM5_CH4,TIM9_CH2,SAI1_FS_A,USART2_RX,OTG_HS_ULPI_D0,ADC123_IN3))
- net x4: no longer MCU1.29 (PA4(SPI1_NSS/I2S1_WS,SPI3_NSS/I2S3_WS,USART2_CK,OTG_HS_SOF,DCMI_HSYNC,ADC12_IN4,DAC_OUT1))
- net x5: no longer MCU1.30 (PA5(TIM2_CH1/TIM2_ETR,TIM8_CH1N,SPI1_SCK/I2S1_CK,OTG_HS_ULPI_CK,ADC12_IN5,DAC_OUT2))
- net x6: no longer MCU1.31 (PA6(TIM1_BKIN,TIM3_CH1,TIM8_BKIN,SPI1_MISO,I2S2_MCK,TIM13_CH1,DCMI_PIXCLK,ADC12_IN6))
- net x7: no longer MCU1.32 (PA7(TIM1_CH1N,TIM3_CH2,TIM8_CH1N,SPI1_MOSI/I2S1_SD,TIM14_CH1,FMC_SDNWE,ADC12_IN7))
- new net x13: MCU1.41 (PE10(TIM1_CH2N,QUADSPI_BK2_IO3,FMC_D7))
- new net x25: MCU1.96 (PB9(TIM2_CH2,TIM4_CH4,TIM11_CH1,I2C1_SDA,SPI2_NSS/I2S2_WS,SAI1_FS_B,CAN1_TX,SDIO_D5,DCMI_D7))
- new net x26: MCU1.25 (PA2(TIM2_CH3,TIM5_CH3,TIM9_CH1,USART2_TX,SAI2_SCK_B,ADC123_IN2))
- new net x28: MCU1.3 (PE4(TRACED1,SPI4_NSS,SAI1_FS_A,FMC_A20,DCMI_D4))
- new net x29: MCU1.2 (PE3(TRACED0,SAI1_SD_B,FMC_A19))
- new net x30: MCU1.1 (PE2(TRACECLK,SPI4_SCK,SAI1_MCLK_A,QUADSPI_BK1_IO2,FMC_A23))
- new net x31: MCU1.4 (PE5(TRACED2,TIM9_CH1,SPI4_MISO,SAI1_SCK_A,FMC_A21,DCMI_D6))
Other:
- note removed: "power led / status led"
- note removed: "todo: recheck pins\n"
- moved on the sheet: J1, MCU1A, MCU1B, MCU1C, MCU1D, MCU1E, R1, R2, R3, R4
