File: hard/supply.sch (KiCad schematic (older format))
At the start: 13 parts, among them J1 MicroXNJ

Commit message: layouting update
Parts:
- renumbered C4 to C15, C1 to C16, C2 to C17, C3 to C18, C5 to C19, C6 to C20, C7 to C21, L1 to L2, R194 to R193, R193 to R194
Changed lines of the file:
@@
 $EndComp
 $Comp
-L Device:C C3
+L Device:C C18
 U 1 1 6055E066
 P 5450 3650
-F 0 "C3" H 5336 3604 50  0000 R CNN
+F 0 "C18" H 5336 3604 50  0000 R CNN
 F 1 "22u/16V" H 5336 3695 50  0000 R CNN
 F 2 "Capacitor_SMD:C_0805_2012Metric" H 5488 3500 50  0001 C CNN
@@
 $EndComp
 $Comp
-L Device:C C4
+L Device:C C15
 U 1 1 60562941
 P 6750 3400
-F 0 "C4" V 6498 3400 50  0000 C CNN
+F 0 "C15" V 6498 3400 50  0000 C CNN
 F 1 "100n/16V" V 6589 3400 50  0000 C CNN
 F 2 "Capacitor_SMD:C_0402_1005Metric" H 6788 3250 50  0001 C CNN
@@
 $EndComp
 $Comp
-L Device:C C5
+L Device:C C19
 U 1 1 60563587
 P 7450 4150
-F 0 "C5" H 7335 4104 50  0000 R CNN
+F 0 "C19" H 7335 4104 50  0000 R CNN
 F 1 "68p/16V" H 7335 4195 50  0000 R CNN
 F 2 "Capacitor_SMD:C_0402_1005Metric" H 7488 4000 50  0001 C CNN
@@
 $EndComp
 $Comp
-L Device:R R194
+L Device:R R193
 U 1 1 6056BF47
 P 8000 4150
-F 0 "R194" H 8070 4196 50  0000 L CNN
+F 0 "R193" H 8070 4196 50  0000 L CNN
 F 1 "100K/1%" H 8070 4105 50  0000 L CNN
 F 2 "Resistor_SMD:R_0402_1005Metric" V 7930 4150 50  0001 C CNN
@@
 $EndComp
 $Comp
-L Device:C C6
+L Device:C C20
 U 1 1 60572E18
 P 8600 4150
-F 0 "C6" H 8485 4104 50  0000 R CNN
+F 0 "C20" H 8485 4104 50  0000 R CNN
 F 1 "22u/16V" H 8485 4195 50  0000 R CNN
 F 2 "Capacitor_SMD:C_0805_2012Metric" H 8638 4000 50  0001 C CNN
@@
 $EndComp
 $Comp
-L Device:C C7
+L Device:C C21
 U 1 1 60574B19
 P 9200 4150
-F 0 "C7" H 9085 4104 50  0000 R CNN
+F 0 "C21" H 9085 4104 50  0000 R CNN
 F 1 "22u/16V" H 9085 4195 50  0000 R CNN
 F 2 "Capacitor_SMD:C_0805_2012Metric" H 9238 4000 50  0001 C CNN
@@
 $EndComp
 $Comp
-L power:+3V3 #PWR0173
+L power:+3V3 #PWR0182
 U 1 1 60578BC3
 P 9250 3850
-F 0 "#PWR0173" H 9250 3700 50  0001 C CNN
+F 0 "#PWR0182" H 9250 3700 50  0001 C CNN
 F 1 "+3V3" H 9265 4023 50  0000 C CNN
 F 2 "" H 9250 3850 50  0001 C CNN
@@
 	6950 3900 6550 3900
 $Comp
-L power:+5V #PWR0168
+L power:+5V #PWR0179
 U 1 1 6057B855
 P 5350 3350
-F 0 "#PWR0168" H 5350 3200 50  0001 C CNN
+F 0 "#PWR0179" H 5350 3200 50  0001 C CNN
 F 1 "+5V" H 5365 3523 50  0000 C CNN
 F 2 "" H 5350 3350 50  0001 C CNN
@@
 	5450 3900 5450 3800
 $Comp
-L power:GND #PWR0169
+L power:GND #PWR0183
 U 1 1 60575673
 P 5450 4050
-F 0 "#PWR0169" H 5450 3800 50  0001 C CNN
+F 0 "#PWR0183" H 5450 3800 50  0001 C CNN
 F 1 "GND" H 5455 3877 50  0000 C CNN
 F 2 "" H 5450 4050 50  0001 C CNN
@@
 	6550 4400 7450 4400
 $Comp
-L power:GND #PWR0171
+L power:GND #PWR0189
 U 1 1 605811D8
 P 8600 4850
-F 0 "#PWR0171" H 8600 4600 50  0001 C CNN
+F 0 "#PWR0189" H 8600 4600 50  0001 C CNN
 F 1 "GND" H 8605 4677 50  0000 C CNN
 F 2 "" H 8600 4850 50  0001 C CNN
@@
 Connection ~ 8600 3900
 $Comp
-L power:GND #PWR0172
+L power:GND #PWR0190
 U 1 1 605828FA
 P 9200 4850
-F 0 "#PWR0172" H 9200 4600 50  0001 C CNN
+F 0 "#PWR0190" H 9200 4600 50  0001 C CNN
 F 1 "GND" H 9205 4677 50  0000 C CNN
 F 2 "" H 9200 4850 50  0001 C CNN
@@
 $EndComp
 $Comp
-L power:GND #PWR0170
+L power:GND #PWR0188
 U 1 1 6057A1D3
 P 8000 4850
-F 0 "#PWR0170" H 8000 4600 50  0001 C CNN
+F 0 "#PWR0188" H 8000 4600 50  0001 C CNN
 F 1 "GND" H 8005 4677 50  0000 C CNN
 F 2 "" H 8000 4850 50  0001 C CNN
@@
 	9200 4850 9200 4300
 $Comp
-L led_matrix:8u2 L1
+L led_matrix:8u2 L2
 U 1 1 605A5BBD
 P 7150 3900
-F 0 "L1" V 7431 3900 50  0000 C CNN
+F 0 "L2" V 7431 3900 50  0000 C CNN
 F 1 "8u2" V 7340 3900 50  0000 C CNN
 F 2 "led_matrix:L_Sunking_MWSA0603S" H 7150 3900 50  0001 C CNN
@@
 $EndComp
 $Comp
-L power:+5V #PWR0167
+L power:+5V #PWR0178
 U 1 1 6056C9AF
 P 4150 3350
-F 0 "#PWR0167" H 4150 3200 50  0001 C CNN
+F 0 "#PWR0178" H 4150 3200 50  0001 C CNN
 F 1 "+5V" H 4165 3523 50  0000 C CNN
 F 2 "" H 4150 3350 50  0001 C CNN
@@
 $EndComp
 $Comp
-L power:GND #PWR0162
+L power:GND #PWR0185
 U 1 1 6056D447
 P 2950 4100
-F 0 "#PWR0162" H 2950 3850 50  0001 C CNN
+F 0 "#PWR0185" H 2950 3850 50  0001 C CNN
 F 1 "GND" H 2955 3927 50  0000 C CNN
 F 2 "" H 2950 4100 50  0001 C CNN
@@
 $EndComp
 $Comp
-L Device:R R193
+L Device:R R194
 U 1 1 6056E34B
 P 3600 4450
-F 0 "R193" H 3670 4496 50  0000 L CNN
+F 0 "R194" H 3670 4496 50  0000 L CNN
 F 1 "0R1" H 3670 4405 50  0000 L CNN
 F 2 "Resistor_SMD:R_0805_2012Metric" V 3530 4450 50  0001 C CNN
@@
 $EndComp
 $Comp
-L Device:C C1
+L Device:C C16
 U 1 1 60578754
 P 3500 3600
-F 0 "C1" H 3385 3554 50  0000 R CNN
+F 0 "C16" H 3385 3554 50  0000 R CNN
 F 1 "22u/16V" H 3385 3645 50  0000 R CNN
 F 2 "Capacitor_SMD:C_0805_2012Metric" H 3538 3450 50  0001 C CNN
@@
 $EndComp
 $Comp
-L Device:C C2
+L Device:C C17
 U 1 1 6057A690
 P 4100 3600
-F 0 "C2" H 3985 3554 50  0000 R CNN
+F 0 "C17" H 3985 3554 50  0000 R CNN
 F 1 "22u/16V" H 3985 3645 50  0000 R CNN
 F 2 "Capacitor_SMD:C_0805_2012Metric" H 4138 3450 50  0001 C CNN
@@
 	3500 3400 4100 3400
 $Comp
-L power:GND #PWR0164
+L power:GND #PWR0180
 U 1 1 6057E614
 P 3500 3800
-F 0 "#PWR0164" H 3500 3550 50  0001 C CNN
+F 0 "#PWR0180" H 3500 3550 50  0001 C CNN
 F 1 "GND" H 3505 3627 50  0000 C CNN
 F 2 "" H 3500 3800 50  0001 C CNN
@@
 $EndComp
 $Comp
-L power:GND #PWR0166
+L power:GND #PWR0181
 U 1 1 6057ED88
 P 4100 3800
-F 0 "#PWR0166" H 4100 3550 50  0001 C CNN
+F 0 "#PWR0181" H 4100 3550 50  0001 C CNN
 F 1 "GND" H 4105 3627 50  0000 C CNN
 F 2 "" H 4100 3800 50  0001 C CNN
@@
 	4100 3800 4100 3750
 $Comp
-L power:Earth #PWR0165
+L power:Earth #PWR0187
 U 1 1 614EE00A
 P 3800 4500
-F 0 "#PWR0165" H 3800 4250 50  0001 C CNN
+F 0 "#PWR0187" H 3800 4250 50  0001 C CNN
 F 1 "Earth" H 3800 4350 50  0001 C CNN
 F 2 "" H 3800 4500 50  0001 C CNN
@@
 	2900 4000 2900 4050
 $Comp
-L power:GND #PWR0163
+L power:GND #PWR0186
 U 1 1 614F0A85
 P 3400 4500
-F 0 "#PWR0163" H 3400 4250 50  0001 C CNN
+F 0 "#PWR0186" H 3400 4250 50  0001 C CNN
 F 1 "GND" H 3405 4327 50  0000 C CNN
 F 2 "" H 3400 4500 50  0001 C CNN
@@
 $EndComp
 $Comp
-L power:Earth #PWR0161
+L power:Earth #PWR0184
 U 1 1 614F2C5D
 P 2750 4100
-F 0 "#PWR0161" H 2750 3850 50  0001 C CNN
+F 0 "#PWR0184" H 2750 3850 50  0001 C CNN
 F 1 "Earth" H 2750 3950 50  0001 C CNN
 F 2 "" H 2750 4100 50  0001 C CNN

Commit message: pcb format refactor
Parts:
- renumbered C15 to C17, C16 to C18, C17 to C19, C18 to C20, C19 to C21, C20 to C22, C21 to C23, J1 to J2, R193 to R203, R194 to R204, R195 to R205
Changed lines of the file:
@@
 $EndComp
 $Comp
-L Device:C C18
+L Device:C C20
 U 1 1 6055E066
 P 5450 3650
-F 0 "C18" H 5336 3604 50  0000 R CNN
+F 0 "C20" H 5336 3604 50  0000 R CNN
 F 1 "22u/16V" H 5336 3695 50  0000 R CNN
 F 2 "Capacitor_SMD:C_0805_2012Metric" H 5488 3500 50  0001 C CNN
@@
 $EndComp
 $Comp
-L Device:C C15
+L Device:C C17
 U 1 1 60562941
 P 6750 3400
-F 0 "C15" V 6498 3400 50  0000 C CNN
+F 0 "C17" V 6498 3400 50  0000 C CNN
 F 1 "100n/16V" V 6589 3400 50  0000 C CNN
 F 2 "Capacitor_SMD:C_0402_1005Metric" H 6788 3250 50  0001 C CNN
@@
 $EndComp
 $Comp
-L Device:C C19
+L Device:C C21
 U 1 1 60563587
 P 7450 4150
-F 0 "C19" H 7335 4104 50  0000 R CNN
+F 0 "C21" H 7335 4104 50  0000 R CNN
 F 1 "68p/16V" H 7335 4195 50  0000 R CNN
 F 2 "Capacitor_SMD:C_0402_1005Metric" H 7488 4000 50  0001 C CNN
@@
 $EndComp
 $Comp
-L Device:R R193
+L Device:R R203
 U 1 1 6056BF47
 P 8000 4150
-F 0 "R193" H 8070 4196 50  0000 L CNN
+F 0 "R203" H 8070 4196 50  0000 L CNN
 F 1 "100K/1%" H 8070 4105 50  0000 L CNN
 F 2 "Resistor_SMD:R_0402_1005Metric" V 7930 4150 50  0001 C CNN
@@
 $EndComp
 $Comp
-L Device:R R195
+L Device:R R205
 U 1 1 6056F7CE
 P 8000 4650
-F 0 "R195" H 8070 4696 50  0000 L CNN
+F 0 "R205" H 8070 4696 50  0000 L CNN
 F 1 "22K/1%" H 8070 4605 50  0000 L CNN
 F 2 "Resistor_SMD:R_0402_1005Metric" V 7930 4650 50  0001 C CNN
@@
 $EndComp
 $Comp
-L Device:C C20
+L Device:C C22
 U 1 1 60572E18
 P 8600 4150
-F 0 "C20" H 8485 4104 50  0000 R CNN
+F 0 "C22" H 8485 4104 50  0000 R CNN
 F 1 "22u/16V" H 8485 4195 50  0000 R CNN
 F 2 "Capacitor_SMD:C_0805_2012Metric" H 8638 4000 50  0001 C CNN
@@
 $EndComp
 $Comp
-L Device:C C21
+L Device:C C23
 U 1 1 60574B19
 P 9200 4150
-F 0 "C21" H 9085 4104 50  0000 R CNN
+F 0 "C23" H 9085 4104 50  0000 R CNN
 F 1 "22u/16V" H 9085 4195 50  0000 R CNN
 F 2 "Capacitor_SMD:C_0805_2012Metric" H 9238 4000 50  0001 C CNN
@@
 $EndComp
 $Comp
-L power:+3V3 #PWR0182
+L power:+3V3 #PWR0191
 U 1 1 60578BC3
 P 9250 3850
-F 0 "#PWR0182" H 9250 3700 50  0001 C CNN
+F 0 "#PWR0191" H 9250 3700 50  0001 C CNN
 F 1 "+3V3" H 9265 4023 50  0000 C CNN
 F 2 "" H 9250 3850 50  0001 C CNN
@@
 	6950 3900 6550 3900
 $Comp
-L power:+5V #PWR0179
+L power:+5V #PWR0188
 U 1 1 6057B855
 P 5350 3350
-F 0 "#PWR0179" H 5350 3200 50  0001 C CNN
+F 0 "#PWR0188" H 5350 3200 50  0001 C CNN
 F 1 "+5V" H 5365 3523 50  0000 C CNN
 F 2 "" H 5350 3350 50  0001 C CNN
@@
 	5450 3900 5450 3800
 $Comp
-L power:GND #PWR0183
+L power:GND #PWR0192
 U 1 1 60575673
 P 5450 4050
-F 0 "#PWR0183" H 5450 3800 50  0001 C CNN
+F 0 "#PWR0192" H 5450 3800 50  0001 C CNN
 F 1 "GND" H 5455 3877 50  0000 C CNN
 F 2 "" H 5450 4050 50  0001 C CNN
@@
 	6550 4400 7450 4400
 $Comp
-L power:GND #PWR0189
+L power:GND #PWR0198
 U 1 1 605811D8
 P 8600 4850
-F 0 "#PWR0189" H 8600 4600 50  0001 C CNN
+F 0 "#PWR0198" H 8600 4600 50  0001 C CNN
 F 1 "GND" H 8605 4677 50  0000 C CNN
 F 2 "" H 8600 4850 50  0001 C CNN
@@
 Connection ~ 8600 3900
 $Comp
-L power:GND #PWR0190
+L power:GND #PWR0199
 U 1 1 605828FA
 P 9200 4850
-F 0 "#PWR0190" H 9200 4600 50  0001 C CNN
+F 0 "#PWR0199" H 9200 4600 50  0001 C CNN
 F 1 "GND" H 9205 4677 50  0000 C CNN
 F 2 "" H 9200 4850 50  0001 C CNN
@@
 $EndComp
 $Comp
-L power:GND #PWR0188
+L power:GND #PWR0197
 U 1 1 6057A1D3
 P 8000 4850
-F 0 "#PWR0188" H 8000 4600 50  0001 C CNN
+F 0 "#PWR0197" H 8000 4600 50  0001 C CNN
 F 1 "GND" H 8005 4677 50  0000 C CNN
 F 2 "" H 8000 4850 50  0001 C CNN
@@
 $EndComp
 $Comp
-L Connector:USB_B_Micro J1
+L Connector:USB_B_Micro J2
 U 1 1 60567F22
 P 2900 3600
-F 0 "J1" H 2957 4067 50  0000 C CNN
+F 0 "J2" H 2957 4067 50  0000 C CNN
 F 1 "MicroXNJ" H 2957 3976 50  0000 C CNN
 F 2 "led_matrix:Connectors_SHOU HAN_MICRO 4P DIP" H 3050 3550 50  0001 C CNN
@@
 $EndComp
 $Comp
-L power:+5V #PWR0178
+L power:+5V #PWR0187
 U 1 1 6056C9AF
 P 4150 3350
-F 0 "#PWR0178" H 4150 3200 50  0001 C CNN
+F 0 "#PWR0187" H 4150 3200 50  0001 C CNN
 F 1 "+5V" H 4165 3523 50  0000 C CNN
 F 2 "" H 4150 3350 50  0001 C CNN
@@
 $EndComp
 $Comp
-L power:GND #PWR0185
+L power:GND #PWR0194
 U 1 1 6056D447
 P 2950 4100
-F 0 "#PWR0185" H 2950 3850 50  0001 C CNN
+F 0 "#PWR0194" H 2950 3850 50  0001 C CNN
 F 1 "GND" H 2955 3927 50  0000 C CNN
 F 2 "" H 2950 4100 50  0001 C CNN
@@
 $EndComp
 $Comp
-L Device:R R194
+L Device:R R204
 U 1 1 6056E34B
 P 3600 4450
-F 0 "R194" H 3670 4496 50  0000 L CNN
+F 0 "R204" H 3670 4496 50  0000 L CNN
 F 1 "0R1" H 3670 4405 50  0000 L CNN
 F 2 "Resistor_SMD:R_0805_2012Metric" V 3530 4450 50  0001 C CNN
@@
 $EndComp
 $Comp
-L Device:C C16
+L Device:C C18
 U 1 1 60578754
 P 3500 3600
-F 0 "C16" H 3385 3554 50  0000 R CNN
+F 0 "C18" H 3385 3554 50  0000 R CNN
 F 1 "22u/16V" H 3385 3645 50  0000 R CNN
 F 2 "Capacitor_SMD:C_0805_2012Metric" H 3538 3450 50  0001 C CNN
@@
 $EndComp
 $Comp
-L Device:C C17
+L Device:C C19
 U 1 1 6057A690
 P 4100 3600
-F 0 "C17" H 3985 3554 50  0000 R CNN
+F 0 "C19" H 3985 3554 50  0000 R CNN
 F 1 "22u/16V" H 3985 3645 50  0000 R CNN
 F 2 "Capacitor_SMD:C_0805_2012Metric" H 4138 3450 50  0001 C CNN
@@
 	3500 3400 4100 3400
 $Comp
-L power:GND #PWR0180
+L power:GND #PWR0189
 U 1 1 6057E614
 P 3500 3800
-F 0 "#PWR0180" H 3500 3550 50  0001 C CNN
+F 0 "#PWR0189" H 3500 3550 50  0001 C CNN
 F 1 "GND" H 3505 3627 50  0000 C CNN
 F 2 "" H 3500 3800 50  0001 C CNN
@@
 $EndComp
 $Comp
-L power:GND #PWR0181
+L power:GND #PWR0190
 U 1 1 6057ED88
 P 4100 3800
-F 0 "#PWR0181" H 4100 3550 50  0001 C CNN
+F 0 "#PWR0190" H 4100 3550 50  0001 C CNN
 F 1 "GND" H 4105 3627 50  0000 C CNN
 F 2 "" H 4100 3800 50  0001 C CNN
@@
 	4100 3800 4100 3750
 $Comp
-L power:Earth #PWR0187
+L power:Earth #PWR0196
 U 1 1 614EE00A
 P 3800 4500
-F 0 "#PWR0187" H 3800 4250 50  0001 C CNN
+F 0 "#PWR0196" H 3800 4250 50  0001 C CNN
 F 1 "Earth" H 3800 4350 50  0001 C CNN
 F 2 "" H 3800 4500 50  0001 C CNN
@@
 	2900 4000 2900 4050
 $Comp
-L power:GND #PWR0186
+L power:GND #PWR0195
 U 1 1 614F0A85
 P 3400 4500
-F 0 "#PWR0186" H 3400 4250 50  0001 C CNN
+F 0 "#PWR0195" H 3400 4250 50  0001 C CNN
 F 1 "GND" H 3405 4327 50  0000 C CNN
 F 2 "" H 3400 4500 50  0001 C CNN
@@
 $EndComp
 $Comp
-L power:Earth #PWR0184
+L power:Earth #PWR0193
 U 1 1 614F2C5D
 P 2750 4100
-F 0 "#PWR0184" H 2750 3850 50  0001 C CNN
+F 0 "#PWR0193" H 2750 3850 50  0001 C CNN
 F 1 "Earth" H 2750 3950 50  0001 C CNN
 F 2 "" H 2750 4100 50  0001 C CNN
